Commit message: Add LinkPose Gazebo plugin.

File: r3mcell_gazebo/urdf/irb120_macro.urdf.xacro (robot description, xacro)
@@ -527,4 +527,10 @@
     </joint>
     <!-- === SCHUNK EGP-64 GRIPPER === -->
+    <!-- LOAD LinkPose Gazebo (ROS2) PLUGIN: -->
+    <gazebo>
+      <plugin name="ros2_linkpose_plugin" filename="libros2_linkpose_plugin.so" >
+        <link>EE_egp64</link>
+      </plugin>
+    </gazebo>
   </xacro:macro>
 </robot>

Commit message: Update R3M_Cell (28Jun).

File: r3mcell_gazebo/urdf/irb120_macro.urdf.xacro (robot description, xacro)
@@ -520,9 +520,9 @@
     </link>
     <joint name="EE_egp64_joint" type="prismatic" >
-      <parent link="egp64_gripper_base_link" />
+      <parent link="tool0" />
       <child link="EE_egp64" />
       <limit effort="10000" lower="0.0" upper="0.0" velocity="0.0"/>
       <axis xyz="1 0 0" />
-      <origin xyz="0.033 -0.018 0.15" rpy="0 0 0"/>
+      <origin xyz="0.0 0.0 0.17" rpy="0 0 0"/>
     </joint>
     <!-- === SCHUNK EGP-64 GRIPPER === -->

Commit message: Update R3M_Cell (Pick&Place).

File: r3mcell_gazebo/urdf/irb120_macro.urdf.xacro (robot description, xacro)
@@ -524,5 +524,5 @@
       <limit effort="10000" lower="0.0" upper="0.0" velocity="0.0"/>
       <axis xyz="1 0 0" />
-      <origin xyz="0.0 0.0 0.17" rpy="0 0 0"/>
+      <origin xyz="0.0 0.0 0.19" rpy="0 0 0"/>
     </joint>
     <!-- === SCHUNK EGP-64 GRIPPER === -->
