Commit message: Fix warnings on ros2_control node.

File: r3mcell_gazebo/urdf/irb120_ros2control.xacro (robot description, xacro)
@@ -208,4 +208,28 @@
       </xacro:unless>
       <!-- === SCHUNK EGP-64 GRIPPER === -->
+      <!-- AVOIDING WARNING MSG in Gazebo: -->
+      <xacro:unless value="${bringup}">
+        <joint name="BASE_TF_joint">
+          <command_interface name="position"/>
+          <command_interface name="velocity"/>
+          <state_interface name="position"/>
+          <state_interface name="velocity"/>
+          <state_interface name="effort"/>
+        </joint>
+        <joint name="TCP_joint">
+          <command_interface name="position"/>
+          <command_interface name="velocity"/>
+          <state_interface name="position"/>
+          <state_interface name="velocity"/>
+          <state_interface name="effort"/>
+        </joint>
+        <joint name="EE_egp64_joint">
+          <command_interface name="position"/>
+          <command_interface name="velocity"/>
+          <state_interface name="position"/>
+          <state_interface name="velocity"/>
+          <state_interface name="effort"/>
+        </joint>
+      </xacro:unless>
     </ros2_control>
     <xacro:unless value="${bringup}">
