Commit message: Modify coordinate origin (+HomePose) and upload MegaPose6D testing script.

File: r3mcell_gazebo/urdf/irb120.urdf.xacro (robot description, xacro)
@@ -82,4 +82,5 @@
     <parent link="world"/>
     <child link="cell"/>
+    <origin xyz="0.926 -0.124 0.0" rpy="0.0 0.0 0.0" />
   </joint>
   <joint name="cell-base_link-fixed" type="fixed">
@@ -88,4 +89,5 @@
     <origin xyz="-0.6506 0.6489 0.8605" rpy="0.0 0.0 0.0" />
   </joint>
+  <!-- Hide for M6D Testing:
   <link name="ergobox">
     <visual>
@@ -111,4 +113,5 @@
     <origin xyz="-0.3 0.32 0.8605" rpy="0.0 0.0 0.0" />
   </joint>
+  -->
   <!-- CAMERA -->
   <xacro:unless value="${bringup}">
@@ -133,5 +136,5 @@
     </link>
     <joint name="camera_joint" type="fixed">
-      <origin xyz="-0.15 0.65 1.90" rpy="0 1.23 3.1416"/>
+      <origin xyz="0.776 0.526 1.90" rpy="0 1.23 3.1416"/>
       <parent link="world"/>
       <child link="camera_link"/>

File: r3mcell_gazebo/urdf/irb120_ros2control.xacro (robot description, xacro)
@@ -110,5 +110,5 @@
         </command_interface>
         <state_interface name="position">
-          <param name="initial_value">0.0</param>
+          <param name="initial_value">-0.5236</param>
         </state_interface>
         <state_interface name="velocity"/>
@@ -125,5 +125,5 @@
         </command_interface>
         <state_interface name="position">
-          <param name="initial_value">0.0</param>
+          <param name="initial_value">0.5236</param>
         </state_interface>
         <state_interface name="velocity"/>
