Commit message: Migration of R3M to new HMI Format.

File: CranfieldUniversity/r3mcell_cu_gazebo/urdf/abb_resources/common_materials.xacro (robot description, xacro)
@@ -1,5 +1,5 @@
 <?xml version="1.0"?>
 <robot xmlns:xacro="http://ros.org/wiki/xacro">
-  <xacro:include filename="$(find r3mcell_gazebo)/urdf/abb_resources/common_colours.xacro"/>
+  <xacro:include filename="$(find r3mcell_cu_gazebo)/urdf/abb_resources/common_colours.xacro"/>
   <xacro:macro name="material_abb_orange">
     <material name="">

File: CranfieldUniversity/r3mcell_cu_gazebo/urdf/irb120.urdf.xacro (robot description, xacro)
@@ -54,5 +54,5 @@
   <xacro:property name="robot_ip" value="$(arg robot_ip)"/>
   <!-- Include XACRO-MACRO file of the IRB120: -->
-  <xacro:include filename="$(find r3mcell_gazebo)/urdf/irb120_macro.urdf.xacro"/>
+  <xacro:include filename="$(find r3mcell_cu_gazebo)/urdf/irb120_macro.urdf.xacro"/>
   <xacro:irb120
     prefix=""
@@ -65,5 +65,5 @@
       <origin xyz="0.0 0.0 0.0" rpy="0 0 0" />
       <geometry>
-        <mesh filename="file://$(find r3mcell_gazebo)/meshes/IALab/IRB120enclosure.dae" scale="1 1 1" />
+        <mesh filename="file://$(find r3mcell_cu_gazebo)/meshes/IALab/IRB120enclosure.dae" scale="1 1 1" />
       </geometry>
     </visual>
@@ -71,5 +71,5 @@
       <origin xyz="0.0 0.0 0.0" rpy="0 0 0" />
       <geometry>
-        <mesh filename="file://$(find r3mcell_gazebo)/meshes/IALab/IRB120enclosure.dae" scale="1 1 1" />
+        <mesh filename="file://$(find r3mcell_cu_gazebo)/meshes/IALab/IRB120enclosure.dae" scale="1 1 1" />
       </geometry>
     </collision>
@@ -94,5 +94,5 @@
       <origin xyz="0.0 0.0 0.0" rpy="0 0 0" />
       <geometry>
-        <mesh filename="file://$(find r3mcell_gazebo)/meshes/IALab/ergobox.dae" scale="1 1 1" />
+        <mesh filename="file://$(find r3mcell_cu_gazebo)/meshes/IALab/ergobox.dae" scale="1 1 1" />
       </geometry>
     </visual>
@@ -100,5 +100,5 @@
       <origin xyz="0.0 0.0 0.0" rpy="0 0 0" />
       <geometry>
-        <mesh filename="file://$(find r3mcell_gazebo)/meshes/IALab/ergobox.dae" scale="1 1 1" />
+        <mesh filename="file://$(find r3mcell_cu_gazebo)/meshes/IALab/ergobox.dae" scale="1 1 1" />
       </geometry>
     </collision>

File: CranfieldUniversity/r3mcell_cu_gazebo/urdf/irb120_macro.urdf.xacro (robot description, xacro)
@@ -49,15 +49,15 @@
 <robot xmlns:xacro="http://ros.org/wiki/xacro">
   <!-- Include additional ABB-Resources/MATERIALS+COLOUR xacro files: -->
-  <xacro:include filename="$(find r3mcell_gazebo)/urdf/abb_resources/common_materials.xacro"/>
+  <xacro:include filename="$(find r3mcell_cu_gazebo)/urdf/abb_resources/common_materials.xacro"/>
   <!-- XACRO-MACRO of ABB-IRB120: -->
   <xacro:macro name="irb120" params="prefix bringup robot_ip">
     <!-- ABB-IRB120 + EGP64 TRANSMISSION: -->
     <xacro:unless value="${bringup}">
-      <xacro:include filename="$(find r3mcell_gazebo)/urdf/irb120_transmission.xacro" />
+      <xacro:include filename="$(find r3mcell_cu_gazebo)/urdf/irb120_transmission.xacro" />
       <xacro:irb120_transmission
         prefix="" />
     </xacro:unless>
     <!-- ABB-IRB120 + EGP64 GAZEBO - ROS2_CONTROL: -->
-    <xacro:include filename="$(find r3mcell_gazebo)/urdf/irb120_ros2control.xacro" />
+    <xacro:include filename="$(find r3mcell_cu_gazebo)/urdf/irb120_ros2control.xacro" />
     <xacro:irb120_ros2control
       prefix=""
@@ -76,5 +76,5 @@
         <origin xyz="0 0 0" rpy="0 0 0"/>
         <geometry>
-          <mesh filename="file://$(find r3mcell_gazebo)/meshes/visual/base_link.dae"/>
+          <mesh filename="file://$(find r3mcell_cu_gazebo)/meshes/visual/base_link.dae"/>
         </geometry>
         <xacro:material_abb_orange />
@@ -83,5 +83,5 @@
         <origin xyz="0 0 0" rpy="0 0 0"/>
         <geometry>
-          <mesh filename="file://$(find r3mcell_gazebo)/meshes/collision/base_link.stl"/>
+          <mesh filename="file://$(find r3mcell_cu_gazebo)/meshes/collision/base_link.stl"/>
         </geometry>
         <xacro:material_abb_yellow />
@@ -98,5 +98,5 @@
         <origin xyz="0 0 0" rpy="0 0 0"/>
         <geometry>
-          <mesh filename="file://$(find r3mcell_gazebo)/meshes/visual/link_1.dae"/>
+          <mesh filename="file://$(find r3mcell_cu_gazebo)/meshes/visual/link_1.dae"/>
         </geometry>
         <xacro:material_abb_orange />
@@ -105,5 +105,5 @@
         <origin xyz="0 0 0" rpy="0 0 0"/>
         <geometry>
-          <mesh filename="file://$(find r3mcell_gazebo)/meshes/collision/link_1.stl"/>
+          <mesh filename="file://$(find r3mcell_cu_gazebo)/meshes/collision/link_1.stl"/>
         </geometry>
         <xacro:material_abb_yellow />
@@ -120,5 +120,5 @@
         <origin xyz="0 0 0" rpy="0 0 0"/>
         <geometry>
-          <mesh filename="file://$(find r3mcell_gazebo)/meshes/visual/link_2.dae"/>
+          <mesh filename="file://$(find r3mcell_cu_gazebo)/meshes/visual/link_2.dae"/>
         </geometry>
         <xacro:material_abb_orange />
@@ -127,5 +127,5 @@
         <origin xyz="0 0 0" rpy="0 0 0"/>
         <geometry>
-          <mesh filename="file://$(find r3mcell_gazebo)/meshes/collision/link_2.stl"/>
+          <mesh filename="file://$(find r3mcell_cu_gazebo)/meshes/collision/link_2.stl"/>
         </geometry>
         <xacro:material_abb_yellow />
@@ -142,5 +142,5 @@
         <origin xyz="0 0 0" rpy="0 0 0"/>
         <geometry>
-          <mesh filename="file://$(find r3mcell_gazebo)/meshes/visual/link_3.dae"/>
+          <mesh filename="file://$(find r3mcell_cu_gazebo)/meshes/visual/link_3.dae"/>
         </geometry>
         <xacro:material_abb_orange />
@@ -149,5 +149,5 @@
         <origin xyz="0 0 0" rpy="0 0 0"/>
         <geometry>
-          <mesh filename="file://$(find r3mcell_gazebo)/meshes/collision/link_3.stl"/>
+          <mesh filename="file://$(find r3mcell_cu_gazebo)/meshes/collision/link_3.stl"/>
         </geometry>
         <xacro:material_abb_yellow />
@@ -164,5 +164,5 @@
         <origin xyz="0 0 0" rpy="0 0 0"/>
         <geometry>
-          <mesh filename="file://$(find r3mcell_gazebo)/meshes/visual/link_4.dae"/>
+          <mesh filename="file://$(find r3mcell_cu_gazebo)/meshes/visual/link_4.dae"/>
         </geometry>
         <xacro:material_abb_orange />
@@ -171,5 +171,5 @@
         <origin xyz="0 0 0" rpy="0 0 0"/>
         <geometry>
-          <mesh filename="file://$(find r3mcell_gazebo)/meshes/collision/link_4.stl"/>
+          <mesh filename="file://$(find r3mcell_cu_gazebo)/meshes/collision/link_4.stl"/>
         </geometry>
         <xacro:material_abb_yellow />
@@ -186,5 +186,5 @@
         <origin xyz="0 0 0" rpy="0 0 0"/>
         <geometry>
-          <mesh filename="file://$(find r3mcell_gazebo)/meshes/visual/link_5.dae"/>
+          <mesh filename="file://$(find r3mcell_cu_gazebo)/meshes/visual/link_5.dae"/>
         </geometry>
         <xacro:material_abb_orange />
@@ -193,5 +193,5 @@
         <origin xyz="0 0 0" rpy="0 0 0"/>
         <geometry>
-          <mesh filename="file://$(find r3mcell_gazebo)/meshes/collision/link_5.stl"/>
+          <mesh filename="file://$(find r3mcell_cu_gazebo)/meshes/collision/link_5.stl"/>
         </geometry>
         <xacro:material_abb_yellow />
@@ -208,5 +208,5 @@
         <origin xyz="0 0 0" rpy="0 0 0"/>
         <geometry>
-          <mesh filename="file://$(find r3mcell_gazebo)/meshes/visual/link_6.dae"/>
+          <mesh filename="file://$(find r3mcell_cu_gazebo)/meshes/visual/link_6.dae"/>
         </geometry>
         <xacro:material_abb_black />
@@ -215,5 +215,5 @@
         <origin xyz="0 0 0" rpy="0 0 0"/>
         <geometry>
-          <mesh filename="file://$(find r3mcell_gazebo)/meshes/collision/link_6.stl"/>
+          <mesh filename="file://$(find r3mcell_cu_gazebo)/meshes/collision/link_6.stl"/>
         </geometry>
         <xacro:material_abb_yellow />
@@ -345,10 +345,10 @@
       <visual>
         <geometry>
-          <mesh filename="file://$(find r3mcell_gazebo)/meshes/egp64/egp64_Adapter.dae" />
-        </geometry>
-      </visual>
-      <collision>
-        <geometry>
-          <mesh filename="file://$(find r3mcell_gazebo)/meshes/egp64/egp64_Adapter.dae" />
+          <mesh filename="file://$(find r3mcell_cu_gazebo)/meshes/egp64/egp64_Adapter.dae" />
+        </geometry>
+      </visual>
+      <collision>
+        <geometry>
+          <mesh filename="file://$(find r3mcell_cu_gazebo)/meshes/egp64/egp64_Adapter.dae" />
         </geometry>
       </collision>
@@ -378,5 +378,5 @@
       <visual>
         <geometry>
-          <mesh filename="file://$(find r3mcell_gazebo)/meshes/egp64/egp64_BaseNoAdapter.dae" />
+          <mesh filename="file://$(find r3mcell_cu_gazebo)/meshes/egp64/egp64_BaseNoAdapter.dae" />
         </geometry>
         <material name="blue">
@@ -386,5 +386,5 @@
       <collision>
         <geometry>
-          <mesh filename="file://$(find r3mcell_gazebo)/meshes/egp64/egp64_BaseNoAdapter.dae" />
+          <mesh filename="file://$(find r3mcell_cu_gazebo)/meshes/egp64/egp64_BaseNoAdapter.dae" />
         </geometry>
         <material name="blue"/>
@@ -405,5 +405,5 @@
       <visual>
         <geometry>
-          <mesh filename="file://$(find r3mcell_gazebo)/meshes/egp64/egp64_LeftFingerBase.dae" />
+          <mesh filename="file://$(find r3mcell_cu_gazebo)/meshes/egp64/egp64_LeftFingerBase.dae" />
         </geometry>
         <material name="black">
@@ -413,5 +413,5 @@
       <collision>
         <geometry>
-          <mesh filename="file://$(find r3mcell_gazebo)/meshes/egp64/egp64_LeftFingerBase.dae" />
+          <mesh filename="file://$(find r3mcell_cu_gazebo)/meshes/egp64/egp64_LeftFingerBase.dae" />
         </geometry>
         <material name="black" />
@@ -435,5 +435,5 @@
       <visual>
         <geometry>
-          <mesh filename="file://$(find r3mcell_gazebo)/meshes/egp64/egp64_LeftFinger.dae" />
+          <mesh filename="file://$(find r3mcell_cu_gazebo)/meshes/egp64/egp64_LeftFinger.dae" />
         </geometry>
         <material name="silver">
@@ -443,5 +443,5 @@
       <collision>
         <geometry>
-          <mesh filename="file://$(find r3mcell_gazebo)/meshes/egp64/egp64_LeftFinger.dae" />
+          <mesh filename="file://$(find r3mcell_cu_gazebo)/meshes/egp64/egp64_LeftFinger.dae" />
         </geometry>
         <material name="black"/>
@@ -462,5 +462,5 @@
       <visual>
         <geometry>
-          <mesh filename="file://$(find r3mcell_gazebo)/meshes/egp64/egp64_RightFingerBase.dae" />
+          <mesh filename="file://$(find r3mcell_cu_gazebo)/meshes/egp64/egp64_RightFingerBase.dae" />
         </geometry>
         <material name="black"/>
@@ -468,5 +468,5 @@
       <collision>
         <geometry>
-          <mesh filename="file://$(find r3mcell_gazebo)/meshes/egp64/egp64_RightFingerBase.dae" />
+          <mesh filename="file://$(find r3mcell_cu_gazebo)/meshes/egp64/egp64_RightFingerBase.dae" />
         </geometry>
         <material name="black"/>
@@ -490,5 +490,5 @@
       <visual>
         <geometry>
-          <mesh filename="file://$(find r3mcell_gazebo)/meshes/egp64/egp64_RightFinger.dae" />
+          <mesh filename="file://$(find r3mcell_cu_gazebo)/meshes/egp64/egp64_RightFinger.dae" />
         </geometry>
         <material name="silver" />
@@ -496,5 +496,5 @@
       <collision>
         <geometry>
-          <mesh filename="file://$(find r3mcell_gazebo)/meshes/egp64/egp64_RightFinger.dae" />
+          <mesh filename="file://$(find r3mcell_cu_gazebo)/meshes/egp64/egp64_RightFinger.dae" />
         </geometry>
         <material name="black"/>

File: CranfieldUniversity/r3mcell_cu_gazebo/urdf/irb120_ros2control.xacro (robot description, xacro)
@@ -63,5 +63,5 @@
         <plugin filename="libgazebo_ros2_control.so" name="gazebo_ros2_control">
           <robot_sim_type>gazebo_ros2_control/GazeboSystem</robot_sim_type>
-          <parameters>$(find r3mcell_gazebo)/config/irb120egp64_controller.yaml</parameters>
+          <parameters>$(find r3mcell_cu_gazebo)/config/irb120egp64_controller.yaml</parameters>
         </plugin>
       </gazebo>
