Commit message: Adapt r3mcell_cu_gazebo to new HMI (layouts format)(LamStack layout components missing).

File: CranfieldUniversity/r3mcell_cu_gazebo/urdf/irb120.urdf.xacro (robot description, xacro)
@@ -49,6 +49,13 @@
 <robot name="irb120" xmlns:xacro="http://ros.org/wiki/xacro">
   <!-- PASS ARGUMENTS: -->
+  <!-- layout -->
+  <xacro:arg name="r3mcell_cu_1" default="false"/>
+  <xacro:property name="r3mcell_cu_1" value="$(arg r3mcell_cu_1)"/>
+  <xacro:arg name="r3mcell_cu_2" default="false"/>
+  <xacro:property name="r3mcell_cu_2" value="$(arg r3mcell_cu_2)"/>
+  <!-- bringup -->
   <xacro:arg name="bringup" default="false"/>
   <xacro:property name="bringup" value="$(arg bringup)"/>
+  <!-- robot_ip -->
   <xacro:arg name="robot_ip" default="0.0.0.0"/>
   <xacro:property name="robot_ip" value="$(arg robot_ip)"/>
@@ -57,4 +64,6 @@
   <xacro:irb120
     prefix=""
+    r3mcell_cu_1="${r3mcell_cu_1}"
+    r3mcell_cu_2="${r3mcell_cu_2}"
     bringup="${bringup}"
     robot_ip="${robot_ip}"/>
@@ -89,29 +98,34 @@
     <origin xyz="-0.6506 0.6489 0.8605" rpy="0.0 0.0 0.0" />
   </joint>
-  <!-- Hide for M6D Testing:
-  <link name="ergobox">
-    <visual>
-      <origin xyz="0.0 0.0 0.0" rpy="0 0 0" />
-      <geometry>
-        <mesh filename="file://$(find r3mcell_cu_gazebo)/meshes/IALab/ergobox.dae" scale="1 1 1" />
-      </geometry>
-    </visual>
-    <collision>
-      <origin xyz="0.0 0.0 0.0" rpy="0 0 0" />
-      <geometry>
-        <mesh filename="file://$(find r3mcell_cu_gazebo)/meshes/IALab/ergobox.dae" scale="1 1 1" />
-      </geometry>
-    </collision>
-    <inertial>
-      <mass value="10.0"/>
-      <inertia ixx="0.0002" ixy="0.0002" ixz="0.0002" iyy="0.0" iyz="0.0" izz="0.0" />
-    </inertial>
-  </link>
-  <joint name="cell-ergobox-fixed" type="fixed">
-    <parent link="cell"/>
-    <child link="ergobox"/>
-    <origin xyz="-0.3 0.32 0.8605" rpy="0.0 0.0 0.0" />
-  </joint>
-  -->
+  <xacro:if value="${r3mcell_cu_1}">
+    <!-- MUST MODIFY: We need a cirular box rather than a square box to avoid conflict with box detections.
+    <link name="ergobox">
+      <visual>
+        <origin xyz="0.0 0.0 0.0" rpy="0 0 0" />
+        <geometry>
+          <mesh filename="file://$(find r3mcell_cu_gazebo)/meshes/IALab/ergobox.dae" scale="1 1 1" />
+        </geometry>
+      </visual>
+      <collision>
+        <origin xyz="0.0 0.0 0.0" rpy="0 0 0" />
+        <geometry>
+          <mesh filename="file://$(find r3mcell_cu_gazebo)/meshes/IALab/ergobox.dae" scale="1 1 1" />
+        </geometry>
+      </collision>
+      <inertial>
+        <mass value="10.0"/>
+        <inertia ixx="0.0002" ixy="0.0002" ixz="0.0002" iyy="0.0" iyz="0.0" izz="0.0" />
+      </inertial>
+    </link>
+    <joint name="cell-ergobox-fixed" type="fixed">
+      <parent link="cell"/>
+      <child link="ergobox"/>
+      <origin xyz="-0.3 0.32 0.8605" rpy="0.0 0.0 0.0" />
+    </joint>
+    -->
+  </xacro:if>
+  <xacro:if value="${r3mcell_cu_2}">
+    <!-- Must add the LamStack layout here! -->
+  </xacro:if>
   <!-- CAMERA -->
   <xacro:unless value="${bringup}">

File: CranfieldUniversity/r3mcell_cu_gazebo/urdf/irb120_macro.urdf.xacro (robot description, xacro)
@@ -51,10 +51,12 @@
   <xacro:include filename="$(find r3mcell_cu_gazebo)/urdf/abb_resources/common_materials.xacro"/>
   <!-- XACRO-MACRO of ABB-IRB120: -->
-  <xacro:macro name="irb120" params="prefix bringup robot_ip">
+  <xacro:macro name="irb120" params="prefix r3mcell_cu_1 r3mcell_cu_2 bringup robot_ip">
     <!-- ABB-IRB120 + EGP64 TRANSMISSION: -->
     <xacro:unless value="${bringup}">
       <xacro:include filename="$(find r3mcell_cu_gazebo)/urdf/irb120_transmission.xacro" />
       <xacro:irb120_transmission
-        prefix="" />
+        prefix=""
+        r3mcell_cu_1="${r3mcell_cu_1}"
+        r3mcell_cu_2="${r3mcell_cu_2}"/>
     </xacro:unless>
     <!-- ABB-IRB120 + EGP64 GAZEBO - ROS2_CONTROL: -->
@@ -62,4 +64,6 @@
     <xacro:irb120_ros2control
       prefix=""
+      r3mcell_cu_1="${r3mcell_cu_1}"
+      r3mcell_cu_2="${r3mcell_cu_2}"
       bringup="${bringup}"
       robot_ip="${robot_ip}"/>
@@ -341,196 +345,250 @@
     <!-- ========== END-EFFECTORS ========== -->
     <!-- === SCHUNK EGP-64 GRIPPER === -->
-    <!-- Schunk coupler (LINK): -->
-    <link name="schunk_coupler">
-      <visual>
-        <geometry>
-          <mesh filename="file://$(find r3mcell_cu_gazebo)/meshes/egp64/egp64_Adapter.dae" />
-        </geometry>
-      </visual>
-      <collision>
-        <geometry>
-          <mesh filename="file://$(find r3mcell_cu_gazebo)/meshes/egp64/egp64_Adapter.dae" />
-        </geometry>
-      </collision>
-      <inertial>
-        <origin xyz="0 0 0" rpy="0 0 ${pi/2}" />
-        <mass value="0.001" />
-        <inertia ixx="0.001" ixy="0.0" ixz="0.0" iyy="0.001" iyz="0.0" izz="0.001"/>
-      </inertial>
-    </link>
-    <!-- Schunk coupler (JOINT): -->
-    <joint name="schunk_coupler_joint" type="fixed">
-      <origin xyz="0 0 0.001" rpy="0 0 ${pi/2}" />
-      <parent link="tool0"/>
-      <child link="schunk_coupler"/>
-    </joint>
-    <gazebo reference="schunk_coupler">
-      <mu1>0.9</mu1>
-      <mu2>0.9</mu2>
-      <material>Gazebo/Black</material>
-    </gazebo>
-    <link name="egp64_gripper_base_link">
-      <inertial>
-        <origin xyz="0 0 0" rpy="0 0 0" />
-        <mass value="0.005" />
-        <inertia ixx="0.001" ixy="0.0" ixz="0.0" iyy="0.001" iyz="0.0" izz="0.001"/>
-      </inertial>
-      <visual>
-        <geometry>
-          <mesh filename="file://$(find r3mcell_cu_gazebo)/meshes/egp64/egp64_BaseNoAdapter.dae" />
-        </geometry>
-        <material name="blue">
-          <color rgba="0 0 1 1"/>
-        </material>
-      </visual>
-      <collision>
-        <geometry>
-          <mesh filename="file://$(find r3mcell_cu_gazebo)/meshes/egp64/egp64_BaseNoAdapter.dae" />
-        </geometry>
-        <material name="blue"/>
-      </collision>
-    </link>
-    <joint name="egp64_coupler" type="fixed">
-      <parent link="schunk_coupler"/>
-      <child link="egp64_gripper_base_link"/>
-      <origin xyz="-0.03205 0.01812 0.02047" rpy="0 0 0" />
-    </joint>
-    <!-- LEFT FINGER BASE -->
-    <link name="egp64_finger_left_link">
-      <inertial>
+    <xacro:if value="${r3mcell_cu_1}">
+      <!-- Schunk coupler (LINK): -->
+      <link name="schunk_coupler">
+        <visual>
+          <geometry>
+            <mesh filename="file://$(find r3mcell_cu_gazebo)/meshes/egp64/egp64_Adapter.dae" />
+          </geometry>
+        </visual>
+        <collision>
+          <geometry>
+            <mesh filename="file://$(find r3mcell_cu_gazebo)/meshes/egp64/egp64_Adapter.dae" />
+          </geometry>
+        </collision>
+        <inertial>
+          <origin xyz="0 0 0" rpy="0 0 ${pi/2}" />
+          <mass value="0.001" />
+          <inertia ixx="0.001" ixy="0.0" ixz="0.0" iyy="0.001" iyz="0.0" izz="0.001"/>
+        </inertial>
+      </link>
+      <!-- Schunk coupler (JOINT): -->
+      <joint name="schunk_coupler_joint" type="fixed">
+        <origin xyz="0 0 0.001" rpy="0 0 ${pi/2}" />
+        <parent link="tool0"/>
+        <child link="schunk_coupler"/>
+      </joint>
+      <gazebo reference="schunk_coupler">
+        <mu1>0.9</mu1>
+        <mu2>0.9</mu2>
+        <material>Gazebo/Black</material>
+      </gazebo>
+      <link name="egp64_gripper_base_link">
+        <inertial>
+          <origin xyz="0 0 0" rpy="0 0 0" />
+          <mass value="0.005" />
+          <inertia ixx="0.001" ixy="0.0" ixz="0.0" iyy="0.001" iyz="0.0" izz="0.001"/>
+        </inertial>
+        <visual>
+          <geometry>
+            <mesh filename="file://$(find r3mcell_cu_gazebo)/meshes/egp64/egp64_BaseNoAdapter.dae" />
+          </geometry>
+          <material name="blue">
+            <color rgba="0 0 1 1"/>
+          </material>
+        </visual>
+        <collision>
+          <geometry>
+            <mesh filename="file://$(find r3mcell_cu_gazebo)/meshes/egp64/egp64_BaseNoAdapter.dae" />
+          </geometry>
+          <material name="blue"/>
+        </collision>
+      </link>
+      <joint name="egp64_coupler" type="fixed">
+        <parent link="schunk_coupler"/>
+        <child link="egp64_gripper_base_link"/>
+        <origin xyz="-0.03205 0.01812 0.02047" rpy="0 0 0" />
+      </joint>
+      <!-- LEFT FINGER BASE -->
+      <link name="egp64_finger_left_link">
+        <inertial>
+          <origin xyz="0.01483 -0.00782 0" rpy="0 0 0" />
+          <mass value="0.002" />
+          <inertia ixx="0.001" ixy="0.0" ixz="0.0" iyy="0.001" iyz="0.0" izz="0.001"/>
+        </inertial>
+        <visual>
+          <geometry>
+            <mesh filename="file://$(find r3mcell_cu_gazebo)/meshes/egp64/egp64_LeftFingerBase.dae" />
+          </geometry>
+          <material name="black">
+            <color rgba="0 0 0 1"/>
+          </material>
+        </visual>
+        <collision>
+          <geometry>
+            <mesh filename="file://$(find r3mcell_cu_gazebo)/meshes/egp64/egp64_LeftFingerBase.dae" />
+          </geometry>
+          <material name="black" />
+        </collision>
+      </link>
+      <joint name="egp64_finger_left_joint" type="prismatic" >
+        <parent link="egp64_gripper_base_link" />
+        <child link="egp64_finger_left_link" />
+        <limit effort="1000" lower="-0.001" upper="0.04" velocity="0.2"/>
         <origin xyz="0.01483 -0.00782 0" rpy="0 0 0" />
-        <mass value="0.002" />
-        <inertia ixx="0.001" ixy="0.0" ixz="0.0" iyy="0.001" iyz="0.0" izz="0.001"/>
-      </inertial>
-      <visual>
-        <geometry>
-          <mesh filename="file://$(find r3mcell_cu_gazebo)/meshes/egp64/egp64_LeftFingerBase.dae" />
-        </geometry>
-        <material name="black">
-          <color rgba="0 0 0 1"/>
-        </material>
-      </visual>
-      <collision>
-        <geometry>
-          <mesh filename="file://$(find r3mcell_cu_gazebo)/meshes/egp64/egp64_LeftFingerBase.dae" />
-        </geometry>
-        <material name="black" />
-      </collision>
-    </link>
-    <joint name="egp64_finger_left_joint" type="prismatic" >
-      <parent link="egp64_gripper_base_link" />
-      <child link="egp64_finger_left_link" />
-      <limit effort="1000" lower="-0.001" upper="0.04" velocity="0.2"/>
-      <origin xyz="0.01483 -0.00782 0" rpy="0 0 0" />
-      <axis xyz="-1 0 0" />
-      <dynamics damping="1.0" friction="1.0"/>
-    </joint>
-    <!-- LEFT FINGERTIP -->
-    <link name="egp64_fingertip_left_link">
-      <inertial>
-        <origin xyz="0.03869 -0.0005 0.00093" rpy="0 0 0" />
-        <mass value="0.001" />
-        <inertia ixx="0.001" ixy="0.0" ixz="0.0" iyy="0.001" iyz="0.0" izz="0.001"/>
-      </inertial>
-      <visual>
-        <geometry>
-          <mesh filename="file://$(find r3mcell_cu_gazebo)/meshes/egp64/egp64_LeftFinger.dae" />
-        </geometry>
-        <material name="silver">
-          <color rgba="0.8 0.8 0.8 1"/>
-        </material>
-      </visual>
-      <collision>
-        <geometry>
-          <mesh filename="file://$(find r3mcell_cu_gazebo)/meshes/egp64/egp64_LeftFinger.dae" />
-        </geometry>
-        <material name="black"/>
-      </collision>
-    </link>
-    <joint name="egp64_fingertip_left_joint" type="fixed" >
-      <parent link="egp64_finger_left_link" />
-      <child link="egp64_fingertip_left_link" />
-      <origin xyz="0.03869 -0.0005 0.00093" rpy="0 0 0"/>
-    </joint>
-    <!-- RIGHT FINGER BASE -->
-    <link name="egp64_finger_right_link">
-      <inertial>
+        <axis xyz="-1 0 0" />
+        <dynamics damping="1.0" friction="1.0"/>
+      </joint>
+      <!-- LEFT FINGERTIP -->
+      <link name="egp64_fingertip_left_link">
+        <inertial>
+          <origin xyz="0.03869 -0.0005 0.00093" rpy="0 0 0" />
+          <mass value="0.001" />
+          <inertia ixx="0.001" ixy="0.0" ixz="0.0" iyy="0.001" iyz="0.0" izz="0.001"/>
+        </inertial>
+        <visual>
+          <geometry>
+            <mesh filename="file://$(find r3mcell_cu_gazebo)/meshes/egp64/egp64_LeftFinger.dae" />
+          </geometry>
+          <material name="silver">
+            <color rgba="0.8 0.8 0.8 1"/>
+          </material>
+        </visual>
+        <collision>
+          <geometry>
+            <mesh filename="file://$(find r3mcell_cu_gazebo)/meshes/egp64/egp64_LeftFinger.dae" />
+          </geometry>
+          <material name="black"/>
+        </collision>
+      </link>
+      <joint name="egp64_fingertip_left_joint" type="fixed" >
+        <parent link="egp64_finger_left_link" />
+        <child link="egp64_fingertip_left_link" />
+        <origin xyz="0.03869 -0.0005 0.00093" rpy="0 0 0"/>
+      </joint>
+      <!-- RIGHT FINGER BASE -->
+      <link name="egp64_finger_right_link">
+        <inertial>
+          <origin xyz="-0.0153 -0.00602 0" rpy="0 0 0" />
+          <mass value="0.002" />
+          <inertia ixx="0.001" ixy="0.0" ixz="0.0" iyy="0.001" iyz="0.0" izz="0.001"/>
+        </inertial>
+        <visual>
+          <geometry>
+            <mesh filename="file://$(find r3mcell_cu_gazebo)/meshes/egp64/egp64_RightFingerBase.dae" />
+          </geometry>
+          <material name="black"/>
+        </visual>
+        <collision>
+          <geometry>
+            <mesh filename="file://$(find r3mcell_cu_gazebo)/meshes/egp64/egp64_RightFingerBase.dae" />
+          </geometry>
+          <material name="black"/>
+        </collision>
+      </link>
+      <joint name="egp64_finger_right_joint" type="prismatic" >
+        <parent link="egp64_gripper_base_link" />
+        <child link="egp64_finger_right_link" />
+        <limit effort="1000" lower="-0.001" upper="0.04" velocity="0.2"/>
         <origin xyz="-0.0153 -0.00602 0" rpy="0 0 0" />
-        <mass value="0.002" />
-        <inertia ixx="0.001" ixy="0.0" ixz="0.0" iyy="0.001" iyz="0.0" izz="0.001"/>
-      </inertial>
-      <visual>
-        <geometry>
-          <mesh filename="file://$(find r3mcell_cu_gazebo)/meshes/egp64/egp64_RightFingerBase.dae" />
-        </geometry>
-        <material name="black"/>
-      </visual>
-      <collision>
-        <geometry>
-          <mesh filename="file://$(find r3mcell_cu_gazebo)/meshes/egp64/egp64_RightFingerBase.dae" />
-        </geometry>
-        <material name="black"/>
-      </collision>
-    </link>
-    <joint name="egp64_finger_right_joint" type="prismatic" >
-      <parent link="egp64_gripper_base_link" />
-      <child link="egp64_finger_right_link" />
-      <limit effort="1000" lower="-0.001" upper="0.04" velocity="0.2"/>
-      <origin xyz="-0.0153 -0.00602 0" rpy="0 0 0" />
-      <axis xyz="1 0 0" />
-      <dynamics damping="1.0" friction="1.0"/>
-    </joint>
-    <!-- RIGHT FINGERTIP -->
-    <link name="egp64_fingertip_right_link">
-      <inertial>
-        <origin xyz="-0.01211 -0.00197 0.00093" rpy="0 0 0" />
-        <mass value="0.001" />
-        <inertia ixx="0.001" ixy="0.0" ixz="0.0" iyy="0.001" iyz="0.0" izz="0.001"/>
-      </inertial>
-      <visual>
-        <geometry>
-          <mesh filename="file://$(find r3mcell_cu_gazebo)/meshes/egp64/egp64_RightFinger.dae" />
-        </geometry>
-        <material name="silver" />
-      </visual>
-      <collision>
-        <geometry>
-          <mesh filename="file://$(find r3mcell_cu_gazebo)/meshes/egp64/egp64_RightFinger.dae" />
-        </geometry>
-        <material name="black"/>
-      </collision>
-    </link>
-    <joint name="egp64_fingertip_right_joint" type="fixed" >
-      <parent link="egp64_finger_right_link" />
-      <child link="egp64_fingertip_right_link" />
-      <origin xyz="-0.01211 -0.00197 0.00093" rpy="0 0 0"/>
-    </joint>
-    <!-- SMALL CUBE FOR GRIPPER PLUGIN -->
-    <link name="EE_egp64">
-      <inertial>
-        <origin xyz="0 0 0" rpy="0 0 0" />
-        <mass value="0.00001" />
-        <inertia ixx="0.001" ixy="0.0" ixz="0.0" iyy="0.001" iyz="0.0" izz="0.001"/>
-      </inertial>
-      <visual>
-        <geometry>
-          <box size= "0.001 0.001 0.001" />
-        </geometry>
-      </visual>
-    </link>
-    <joint name="EE_egp64_joint" type="prismatic" >
-      <parent link="tool0" />
-      <child link="EE_egp64" />
-      <limit effort="10000" lower="0.0" upper="0.0" velocity="0.0"/>
-      <axis xyz="1 0 0" />
-      <origin xyz="0.0 0.0 0.19" rpy="0 0 0"/>
-    </joint>
-    <!-- === SCHUNK EGP-64 GRIPPER === -->
-    <!-- LOAD LinkPose Gazebo (ROS2) PLUGIN: -->
-    <gazebo>
-      <plugin name="ros2_linkpose_plugin" filename="libros2_linkpose_plugin.so" >
-        <link>EE_egp64</link>
-      </plugin>
-    </gazebo>
+        <axis xyz="1 0 0" />
+        <dynamics damping="1.0" friction="1.0"/>
+      </joint>
+      <!-- RIGHT FINGERTIP -->
+      <link name="egp64_fingertip_right_link">
+        <inertial>
+          <origin xyz="-0.01211 -0.00197 0.00093" rpy="0 0 0" />
+          <mass value="0.001" />
+          <inertia ixx="0.001" ixy="0.0" ixz="0.0" iyy="0.001" iyz="0.0" izz="0.001"/>
+        </inertial>
+        <visual>
+          <geometry>
+            <mesh filename="file://$(find r3mcell_cu_gazebo)/meshes/egp64/egp64_RightFinger.dae" />
+          </geometry>
+          <material name="silver" />
+        </visual>
+        <collision>
+          <geometry>
+            <mesh filename="file://$(find r3mcell_cu_gazebo)/meshes/egp64/egp64_RightFinger.dae" />
+          </geometry>
+          <material name="black"/>
+        </collision>
+      </link>
+      <joint name="egp64_fingertip_right_joint" type="fixed" >
+        <parent link="egp64_finger_right_link" />
+        <child link="egp64_fingertip_right_link" />
+        <origin xyz="-0.01211 -0.00197 0.00093" rpy="0 0 0"/>
+      </joint>
+      <!-- SMALL CUBE FOR GRIPPER PLUGIN -->
+      <link name="EE_egp64">
+        <inertial>
+          <origin xyz="0 0 0" rpy="0 0 0" />
+          <mass value="0.00001" />
+          <inertia ixx="0.001" ixy="0.0" ixz="0.0" iyy="0.001" iyz="0.0" izz="0.001"/>
+        </inertial>
+        <visual>
+          <geometry>
+            <box size= "0.001 0.001 0.001" />
+          </geometry>
+        </visual>
+      </link>
+      <joint name="EE_egp64_joint" type="prismatic" >
+        <parent link="tool0" />
+        <child link="EE_egp64" />
+        <limit effort="10000" lower="0.0" upper="0.0" velocity="0.0"/>
+        <axis xyz="1 0 0" />
+        <origin xyz="0.0 0.0 0.19" rpy="0 0 0"/>
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