Commit message: Adapt r3mcell_cu_gazebo to new HMI (layouts format)(LamStack layout components missing).

File: CranfieldUniversity/r3mcell_cu_gazebo/urdf/irb120_ros2control.xacro (robot description, xacro)
@@ -48,5 +48,5 @@
 -->
 <robot xmlns:xacro="http://www.ros.org/wiki/xacro">
-  <xacro:macro name="irb120_ros2control" params="prefix bringup robot_ip" >
+  <xacro:macro name="irb120_ros2control" params="prefix r3mcell_cu_1 r3mcell_cu_2 bringup robot_ip" >
     <!-- 1. ROS2_CONTROL tag name: -->
     <!-- A. GAZEBO SIMULATION: -->
@@ -60,10 +60,20 @@
     <!-- 2. IF GAZEBO -> Load PLUGIN: -->
     <xacro:unless value="${bringup}">
-      <gazebo>
-        <plugin filename="libgazebo_ros2_control.so" name="gazebo_ros2_control">
-          <robot_sim_type>gazebo_ros2_control/GazeboSystem</robot_sim_type>
-          <parameters>$(find r3mcell_cu_gazebo)/config/irb120egp64_controller.yaml</parameters>
-        </plugin>
-      </gazebo>
+      <xacro:if value="${r3mcell_cu_1}">
+        <gazebo>
+          <plugin filename="libgazebo_ros2_control.so" name="gazebo_ros2_control">
+            <robot_sim_type>gazebo_ros2_control/GazeboSystem</robot_sim_type>
+            <parameters>$(find r3mcell_cu_gazebo)/config/irb120egp64_controller.yaml</parameters>
+          </plugin>
+        </gazebo>
+      </xacro:if>
+      <xacro:if value="${r3mcell_cu_2}">
+        <gazebo>
+          <plugin filename="libgazebo_ros2_control.so" name="gazebo_ros2_control">
+            <robot_sim_type>gazebo_ros2_control/GazeboSystem</robot_sim_type>
+            <parameters>$(find r3mcell_cu_gazebo)/config/irb120_controller.yaml</parameters>
+          </plugin>
+        </gazebo>
+      </xacro:if>
     </xacro:unless>
     <!-- 3. Load ROS2_CONTROL: -->
@@ -176,34 +186,36 @@
       <!-- === SCHUNK EGP-64 GRIPPER === -->
       <xacro:unless value="${bringup}">
-        <!-- egp64_finger_left_joint -->
-        <joint name="egp64_finger_left_joint">
-          <command_interface name="position">
-            <param name="min">-0.001</param>
-            <param name="max">0.04</param>
-          </command_interface>
-          <command_interface name="velocity">
-            <param name="min">-0.2</param>
-            <param name="max">0.2</param>
-          </command_interface>
-          <state_interface name="position">
-            <param name="initial_value">0.0</param>
-          </state_interface>
-          <state_interface name="velocity"/>
-        </joint>
-        <!-- egp64_finger_right_joint -->
-        <joint name="egp64_finger_right_joint">
-          <command_interface name="position">
-            <param name="min">-0.001</param>
-            <param name="max">0.04</param>
-          </command_interface>
-          <command_interface name="velocity">
-            <param name="min">-0.2</param>
-            <param name="max">0.2</param>
-          </command_interface>
-          <state_interface name="position">
-            <param name="initial_value">0.0</param>
-          </state_interface>
-          <state_interface name="velocity"/>
-        </joint>
+        <xacro:if value="${r3mcell_cu_1}">
+          <!-- egp64_finger_left_joint -->
+          <joint name="egp64_finger_left_joint">
+            <command_interface name="position">
+              <param name="min">-0.001</param>
+              <param name="max">0.04</param>
+            </command_interface>
+            <command_interface name="velocity">
+              <param name="min">-0.2</param>
+              <param name="max">0.2</param>
+            </command_interface>
+            <state_interface name="position">
+              <param name="initial_value">0.0</param>
+            </state_interface>
+            <state_interface name="velocity"/>
+          </joint>
+          <!-- egp64_finger_right_joint -->
+          <joint name="egp64_finger_right_joint">
+            <command_interface name="position">
+              <param name="min">-0.001</param>
+              <param name="max">0.04</param>
+            </command_interface>
+            <command_interface name="velocity">
+              <param name="min">-0.2</param>
+              <param name="max">0.2</param>
+            </command_interface>
+            <state_interface name="position">
+              <param name="initial_value">0.0</param>
+            </state_interface>
+            <state_interface name="velocity"/>
+          </joint>
+        </xacro:if>
       </xacro:unless>
       <!-- === SCHUNK EGP-64 GRIPPER === -->
@@ -224,11 +236,22 @@
           <state_interface name="effort"/>
         </joint>
-        <joint name="EE_egp64_joint">
-          <command_interface name="position"/>
-          <command_interface name="velocity"/>
-          <state_interface name="position"/>
-          <state_interface name="velocity"/>
-          <state_interface name="effort"/>
-        </joint>
+        <xacro:if value="${r3mcell_cu_1}">
+          <joint name="EE_egp64_joint">
+            <command_interface name="position"/>
+            <command_interface name="velocity"/>
+            <state_interface name="position"/>
+            <state_interface name="velocity"/>
+            <state_interface name="effort"/>
+          </joint>
+        </xacro:if>
+        <xacro:if value="${r3mcell_cu_2}">
+          <joint name="EE_vgr_joint">
+            <command_interface name="position"/>
+            <command_interface name="velocity"/>
+            <state_interface name="position"/>
+            <state_interface name="velocity"/>
+            <state_interface name="effort"/>
+          </joint>
+        </xacro:if>
       </xacro:unless>
     </ros2_control>
@@ -256,20 +279,29 @@
       </gazebo>
       <!-- === SCHUNK EGP-64 GRIPPER === -->
-      <gazebo reference="egp64_gripper_base_link">
-        <selfCollide>false</selfCollide>
-      </gazebo>
-      <gazebo reference="egp64_finger_left_link">
-        <selfCollide>false</selfCollide>
-      </gazebo>
-      <gazebo reference="egp64_fingertip_left_link">
-        <selfCollide>false</selfCollide>
-      </gazebo>
-      <gazebo reference="egp64_finger_right_link">
-        <selfCollide>false</selfCollide>
-      </gazebo>
-      <gazebo reference="egp64_fingertip_right_link">
-        <selfCollide>false</selfCollide>
-      </gazebo>
+      <xacro:if value="${r3mcell_cu_1}">
+        <gazebo reference="egp64_gripper_base_link">
+          <selfCollide>false</selfCollide>
+        </gazebo>
+        <gazebo reference="egp64_finger_left_link">
+          <selfCollide>false</selfCollide>
+        </gazebo>
+        <gazebo reference="egp64_fingertip_left_link">
+          <selfCollide>false</selfCollide>
+        </gazebo>
+        <gazebo reference="egp64_finger_right_link">
+          <selfCollide>false</selfCollide>
+        </gazebo>
+        <gazebo reference="egp64_fingertip_right_link">
+          <selfCollide>false</selfCollide>
+        </gazebo>
+      </xacro:if>
       <!-- === SCHUNK EGP-64 GRIPPER === -->
+      <!-- === VACUUM GRIPPER === -->
+      <xacro:if value="${r3mcell_cu_2}">
+        <gazebo reference="vgr_link">
+          <selfCollide>false</selfCollide>
+        </gazebo>
+      </xacro:if>
+      <!-- === VACUUM GRIPPER === -->
       <gazebo reference="end_effector_frame_fixed_joint">
         <preserveFixedJoint>true</preserveFixedJoint>

File: CranfieldUniversity/r3mcell_cu_gazebo/urdf/irb120_transmission.xacro (robot description, xacro)
@@ -48,5 +48,5 @@
 -->
 <robot xmlns:xacro="http://wiki.ros.org/xacro">
-  <xacro:macro name="irb120_transmission" params="prefix ">
+  <xacro:macro name="irb120_transmission" params="prefix r3mcell_cu_1 r3mcell_cu_2">
     <transmission name="irb120_joint1_trans">
       <type>transmission_interface/SimpleTransmission</type>
@@ -104,22 +104,24 @@
     </transmission>
     <!-- === SCHUNK EGP-64 GRIPPER === -->
-    <transmission name="egp64_left_finger_trans">
-      <type>transmission_interface/SimpleTransmission</type>
-      <joint name="egp64_finger_left_joint">
-        <hardwareInterface>hardware_interface/PositionJointInterface</hardwareInterface>
-      </joint>
-      <actuator name="egp64_left_finger_motor">
-        <mechanicalReduction>1</mechanicalReduction>
-      </actuator>
-    </transmission>
-    <transmission name="egp64_right_finger_trans">
-      <type>transmission_interface/SimpleTransmission</type>
-      <joint name="egp64_finger_right_joint">
-        <hardwareInterface>hardware_interface/PositionJointInterface</hardwareInterface>
-      </joint>
-      <actuator name="egp64_right_finger_motor">
-        <mechanicalReduction>1</mechanicalReduction>
-      </actuator>
-    </transmission>
+    <xacro:if value="${r3mcell_cu_1}">
+      <transmission name="egp64_left_finger_trans">
+        <type>transmission_interface/SimpleTransmission</type>
+        <joint name="egp64_finger_left_joint">
+          <hardwareInterface>hardware_interface/PositionJointInterface</hardwareInterface>
+        </joint>
+        <actuator name="egp64_left_finger_motor">
+          <mechanicalReduction>1</mechanicalReduction>
+        </actuator>
+      </transmission>
+      <transmission name="egp64_right_finger_trans">
+        <type>transmission_interface/SimpleTransmission</type>
+        <joint name="egp64_finger_right_joint">
+          <hardwareInterface>hardware_interface/PositionJointInterface</hardwareInterface>
+        </joint>
+        <actuator name="egp64_right_finger_motor">
+          <mechanicalReduction>1</mechanicalReduction>
+        </actuator>
+      </transmission>
+    </xacro:if>
     <!-- === SCHUNK EGP-64 GRIPPER === -->
   </xacro:macro>

Commit message: Add: R3M LamStack use-case + adapt moveit.launch to R3M-HMI.

File: CranfieldUniversity/r3mcell_cu_gazebo/urdf/irb120.urdf.xacro (robot description, xacro)
@@ -126,5 +126,50 @@
   </xacro:if>
   <xacro:if value="${r3mcell_cu_2}">
-    <!-- Must add the LamStack layout here! -->
+    <link name="LS_PickingStand">
+      <visual>
+        <origin xyz="0.0 0.0 0.0" rpy="0 0 0" />
+        <geometry>
+          <mesh filename="file://$(find r3mcell_cu_gazebo)/meshes/LamStack_UseCase/R3M_LSPickingStand.dae" scale="1 1 1" />
+        </geometry>
+      </visual>
+      <collision>
+        <origin xyz="0.0 0.0 0.0" rpy="0 0 0" />
+        <geometry>
+          <mesh filename="file://$(find r3mcell_cu_gazebo)/meshes/LamStack_UseCase/R3M_LSPickingStand.dae" scale="1 1 1" />
+        </geometry>
+      </collision>
+      <inertial>
+        <mass value="10.0"/>
+        <inertia ixx="0.0002" ixy="0.0002" ixz="0.0002" iyy="0.0" iyz="0.0" izz="0.0" />
+      </inertial>
+    </link>
+    <joint name="cell-LS_PickingStand-fixed" type="fixed">
+      <parent link="cell"/>
+      <child link="LS_PickingStand"/>
+      <origin xyz="-0.425 0.825 0.8605" rpy="0.0 0.0 0.0" />
+    </joint>
+    <link name="LS_PlacingStand">
+      <visual>
+        <origin xyz="0.0 0.0 0.0" rpy="0 0 0" />
+        <geometry>
+          <mesh filename="file://$(find r3mcell_cu_gazebo)/meshes/LamStack_UseCase/R3M_LSPlacingStand.dae" scale="1 1 1" />
+        </geometry>
+      </visual>
+      <collision>
+        <origin xyz="0.0 0.0 0.0" rpy="0 0 0" />
+        <geometry>
+          <mesh filename="file://$(find r3mcell_cu_gazebo)/meshes/LamStack_UseCase/R3M_LSPlacingStand.dae" scale="1 1 1" />
+        </geometry>
+      </collision>
+      <inertial>
+        <mass value="10.0"/>
+        <inertia ixx="0.0002" ixy="0.0002" ixz="0.0002" iyy="0.0" iyz="0.0" izz="0.0" />
+      </inertial>
+    </link>
+    <joint name="cell-LS_PlacingStand-fixed" type="fixed">
+      <parent link="cell"/>
+      <child link="LS_PlacingStand"/>
+      <origin xyz="-0.525 0.325 0.8605" rpy="0.0 0.0 3.1416" />
+    </joint>
   </xacro:if>
   <!-- CAMERA -->
@@ -186,4 +231,61 @@
       </sensor>
     </gazebo>
+    <!-- CAMERA for R3M-HMI -->
+    <link name="HMI_camera_link">
+      <collision>
+        <origin xyz="0 0 0" rpy="0 0 0"/>
+        <geometry>
+          <box size="0.05 0.05 0.05"/>
+        </geometry>
+      </collision>
+      <visual>
+        <origin xyz="0 0 0" rpy="0 0 0"/>
+        <geometry>
+          <box size="0.05 0.05 0.05"/>
+        </geometry>
+      </visual>
+      <inertial>
+        <mass value="1.0" />
+        <origin xyz="0 0 0" rpy="0 0 0"/>
+        <inertia ixx="0.0" ixy="0.0" ixz="0.0" iyy="0.0" iyz="0.0" izz="0.0" />
+      </inertial>
+    </link>
+    <joint name="HMI_camera_joint" type="fixed">
+      <origin xyz="2.0 1.5 2.0" rpy="0 0.35 -2.6"/>
+      <parent link="world"/>
+      <child link="HMI_camera_link"/>
+    </joint>
+    <gazebo reference="HMI_camera_link">
+      <sensor name="HMI_camera" type="camera">
+        <update_rate>30</update_rate>
+        <camera name="head">
+          <horizontal_fov>1.22</horizontal_fov>
+          <image>
+            <width>1920</width>
+            <height>1080</height>
+            <format>R8G8B8</format>
+          </image>
+          <clip>
+            <near>0.02</near>
+            <far>300</far>
+          </clip>
+          <noise>
+            <type>gaussian</type>
+            <mean>0.0</mean>
+            <stddev>0.007</stddev>
+          </noise>
+        </camera>
+        <plugin filename="libgazebo_ros_camera.so" name="HMI_camera_controller">
+          <robotNamespace/>
+          <alwaysOn>true</alwaysOn>
+          <updateRate>0.0</updateRate>
+          <cameraName>HMI_camera</cameraName>
+          <imageTopicName>HMI_image_raw</imageTopicName>
+          <cameraInfoTopicName>HMI_camera_info</cameraInfoTopicName>
+          <frameName>HMI_camera</frameName>
+          <hackBaseline>0.07</hackBaseline>
+        </plugin>
+      </sensor>
+    </gazebo>
   </xacro:unless>
 </robot>

File: CranfieldUniversity/r3mcell_cu_gazebo/urdf/irb120_macro.urdf.xacro (robot description, xacro)
@@ -582,5 +582,5 @@
         <limit effort="10000" lower="0.0" upper="0.0" velocity="0.0"/>
         <axis xyz="1 0 0" />
-        <origin xyz="0.07 0.0 0.095" rpy="0 0 0"/>
+        <origin xyz="0.065 0.0 0.1" rpy="0 0 0"/>
       </joint>
       <!-- LOAD LinkPose Gazebo (ROS2) PLUGIN: -->

Commit message: Upload: CAN Pick-and-Place Use-Case.

File: CranfieldUniversity/r3mcell_cu_gazebo/urdf/irb120.urdf.xacro (robot description, xacro)
@@ -54,4 +54,13 @@
   <xacro:arg name="r3mcell_cu_2" default="false"/>
   <xacro:property name="r3mcell_cu_2" value="$(arg r3mcell_cu_2)"/>
+  <xacro:arg name="r3mcell_cu_3" default="false"/>
+  <xacro:property name="r3mcell_cu_3" value="$(arg r3mcell_cu_3)"/>
+  <!-- endeffector -->
+  <xacro:arg name="EE_no" default="false"/>
+  <xacro:property name="EE_no" value="$(arg EE_no)"/>
+  <xacro:arg name="EE_egp64" default="false"/>
+  <xacro:property name="EE_egp64" value="$(arg EE_egp64)"/>
+  <xacro:arg name="EE_vgr" default="false"/>
+  <xacro:property name="EE_vgr" value="$(arg EE_vgr)"/>
   <!-- bringup -->
   <xacro:arg name="bringup" default="false"/>
@@ -64,6 +73,7 @@
   <xacro:irb120
     prefix=""
-    r3mcell_cu_1="${r3mcell_cu_1}"
-    r3mcell_cu_2="${r3mcell_cu_2}"
+    EE_no="${EE_no}"
+    EE_egp64="${EE_egp64}"
+    EE_vgr="${EE_vgr}"
     bringup="${bringup}"
     robot_ip="${robot_ip}"/>
@@ -173,4 +183,52 @@
     </joint>
   </xacro:if>
+  <xacro:if value="${r3mcell_cu_3}">
+    <link name="CAN_PickingStand">
+      <visual>
+        <origin xyz="0.0 0.0 0.0" rpy="0 0 0" />
+        <geometry>
+          <mesh filename="file://$(find r3mcell_cu_gazebo)/meshes/canPP/canPicking.dae" scale="1 1 1" />
+        </geometry>
+      </visual>
+      <collision>
+        <origin xyz="0.0 0.0 0.0" rpy="0 0 0" />
+        <geometry>
+          <mesh filename="file://$(find r3mcell_cu_gazebo)/meshes/canPP/canPicking.dae" scale="1 1 1" />
+        </geometry>
+      </collision>
+      <inertial>
+        <mass value="10.0"/>
+        <inertia ixx="0.0002" ixy="0.0002" ixz="0.0002" iyy="0.0" iyz="0.0" izz="0.0" />
+      </inertial>
+    </link>
+    <joint name="cell-CAN_PickingStand-fixed" type="fixed">
+      <parent link="cell"/>
+      <child link="CAN_PickingStand"/>
+      <origin xyz="-0.425 0.825 0.8605" rpy="0.0 0.0 0.0" />
+    </joint>
+    <link name="CAN_PlacingStand">
+      <visual>
+        <origin xyz="0.0 0.0 0.0" rpy="0 0 0" />
+        <geometry>
+          <mesh filename="file://$(find r3mcell_cu_gazebo)/meshes/canPP/canPlacing.dae" scale="1 1 1" />
+        </geometry>
+      </visual>
+      <collision>
+        <origin xyz="0.0 0.0 0.0" rpy="0 0 0" />
+        <geometry>
+          <mesh filename="file://$(find r3mcell_cu_gazebo)/meshes/canPP/canPlacing.dae" scale="1 1 1" />
+        </geometry>
+      </collision>
+      <inertial>
+        <mass value="10.0"/>
+        <inertia ixx="0.0002" ixy="0.0002" ixz="0.0002" iyy="0.0" iyz="0.0" izz="0.0" />
+      </inertial>
+    </link>
+    <joint name="cell-CAN_PlacingStand-fixed" type="fixed">
+      <parent link="cell"/>
+      <child link="CAN_PlacingStand"/>
+      <origin xyz="-0.425 0.225 0.8605" rpy="0.0 0.0 3.1416" />
+    </joint>
+  </xacro:if>
   <!-- CAMERA -->
   <xacro:unless value="${bringup}">

File: CranfieldUniversity/r3mcell_cu_gazebo/urdf/irb120_macro.urdf.xacro (robot description, xacro)
@@ -51,5 +51,5 @@
   <xacro:include filename="$(find r3mcell_cu_gazebo)/urdf/abb_resources/common_materials.xacro"/>
   <!-- XACRO-MACRO of ABB-IRB120: -->
-  <xacro:macro name="irb120" params="prefix r3mcell_cu_1 r3mcell_cu_2 bringup robot_ip">
+  <xacro:macro name="irb120" params="prefix EE_no EE_egp64 EE_vgr bringup robot_ip">
     <!-- ABB-IRB120 + EGP64 TRANSMISSION: -->
     <xacro:unless value="${bringup}">
@@ -57,6 +57,7 @@
       <xacro:irb120_transmission
         prefix=""
-        r3mcell_cu_1="${r3mcell_cu_1}"
-        r3mcell_cu_2="${r3mcell_cu_2}"/>
+        EE_no="${EE_no}"
+        EE_egp64="${EE_egp64}"
+        EE_vgr="${EE_vgr}"/>
     </xacro:unless>
     <!-- ABB-IRB120 + EGP64 GAZEBO - ROS2_CONTROL: -->
@@ -64,6 +65,7 @@
     <xacro:irb120_ros2control
       prefix=""
-      r3mcell_cu_1="${r3mcell_cu_1}"
-      r3mcell_cu_2="${r3mcell_cu_2}"
+      EE_no="${EE_no}"
+      EE_egp64="${EE_egp64}"
+      EE_vgr="${EE_vgr}"
       bringup="${bringup}"
       robot_ip="${robot_ip}"/>
@@ -345,5 +347,5 @@
     <!-- ========== END-EFFECTORS ========== -->
     <!-- === SCHUNK EGP-64 GRIPPER === -->
-    <xacro:if value="${r3mcell_cu_1}">
+    <xacro:if value="${EE_egp64}">
       <!-- Schunk coupler (LINK): -->
       <link name="schunk_coupler">
@@ -540,5 +542,5 @@
     </xacro:if>
     <!-- === CUSTOM R3M VACUUM GRIPPER === -->
-    <xacro:if value="${r3mcell_cu_2}">
+    <xacro:if value="${EE_vgr}">
       <!-- Vacuum Gripper: Body -->
       <link name="vgr_link">

File: CranfieldUniversity/r3mcell_cu_gazebo/urdf/irb120_ros2control.xacro (robot description, xacro)
@@ -48,5 +48,5 @@
 -->
 <robot xmlns:xacro="http://www.ros.org/wiki/xacro">
-  <xacro:macro name="irb120_ros2control" params="prefix r3mcell_cu_1 r3mcell_cu_2 bringup robot_ip" >
+  <xacro:macro name="irb120_ros2control" params="prefix EE_no EE_egp64 EE_vgr bringup robot_ip" >
     <!-- 1. ROS2_CONTROL tag name: -->
     <!-- A. GAZEBO SIMULATION: -->
@@ -60,5 +60,5 @@
     <!-- 2. IF GAZEBO -> Load PLUGIN: -->
     <xacro:unless value="${bringup}">
-      <xacro:if value="${r3mcell_cu_1}">
+      <xacro:if value="${EE_egp64}">
         <gazebo>
           <plugin filename="libgazebo_ros2_control.so" name="gazebo_ros2_control">
@@ -68,5 +68,13 @@
         </gazebo>
       </xacro:if>
-      <xacro:if value="${r3mcell_cu_2}">
+      <xacro:if value="${EE_no}">
+        <gazebo>
+          <plugin filename="libgazebo_ros2_control.so" name="gazebo_ros2_control">
+            <robot_sim_type>gazebo_ros2_control/GazeboSystem</robot_sim_type>
+            <parameters>$(find r3mcell_cu_gazebo)/config/irb120_controller.yaml</parameters>
+          </plugin>
+        </gazebo>
+      </xacro:if>
+      <xacro:if value="${EE_vgr}">
         <gazebo>
           <plugin filename="libgazebo_ros2_control.so" name="gazebo_ros2_control">
@@ -186,5 +194,5 @@
       <!-- === SCHUNK EGP-64 GRIPPER === -->
       <xacro:unless value="${bringup}">
-        <xacro:if value="${r3mcell_cu_1}">
+        <xacro:if value="${EE_egp64}">
           <!-- egp64_finger_left_joint -->
           <joint name="egp64_finger_left_joint">
@@ -236,5 +244,5 @@
           <state_interface name="effort"/>
         </joint>
-        <xacro:if value="${r3mcell_cu_1}">
+        <xacro:if value="${EE_egp64}">
           <joint name="EE_egp64_joint">
             <command_interface name="position"/>
@@ -245,5 +253,5 @@
           </joint>
         </xacro:if>
-        <xacro:if value="${r3mcell_cu_2}">
+        <xacro:if value="${EE_vgr}">
           <joint name="EE_vgr_joint">
             <command_interface name="position"/>
@@ -279,5 +287,5 @@
       </gazebo>
       <!-- === SCHUNK EGP-64 GRIPPER === -->
-      <xacro:if value="${r3mcell_cu_1}">
+      <xacro:if value="${EE_egp64}">
         <gazebo reference="egp64_gripper_base_link">
           <selfCollide>false</selfCollide>
@@ -298,5 +306,5 @@
       <!-- === SCHUNK EGP-64 GRIPPER === -->
       <!-- === VACUUM GRIPPER === -->
-      <xacro:if value="${r3mcell_cu_2}">
+      <xacro:if value="${EE_vgr}">
         <gazebo reference="vgr_link">
           <selfCollide>false</selfCollide>

File: CranfieldUniversity/r3mcell_cu_gazebo/urdf/irb120_transmission.xacro (robot description, xacro)
@@ -48,5 +48,5 @@
 -->
 <robot xmlns:xacro="http://wiki.ros.org/xacro">
-  <xacro:macro name="irb120_transmission" params="prefix r3mcell_cu_1 r3mcell_cu_2">
+  <xacro:macro name="irb120_transmission" params="prefix EE_no EE_egp64 EE_vgr">
     <transmission name="irb120_joint1_trans">
       <type>transmission_interface/SimpleTransmission</type>
@@ -104,5 +104,5 @@
     </transmission>
     <!-- === SCHUNK EGP-64 GRIPPER === -->
-    <xacro:if value="${r3mcell_cu_1}">
+    <xacro:if value="${EE_egp64}">
       <transmission name="egp64_left_finger_trans">
         <type>transmission_interface/SimpleTransmission</type>
