Commit message: Update cubePP use-case.

File: CranfieldUniversity/r3mcell_cu_gazebo/urdf/irb120.urdf.xacro (robot description, xacro)
@@ -109,29 +109,27 @@
   </joint>
   <xacro:if value="${r3mcell_cu_1}">
-    <!-- MUST MODIFY: We need a cirular box rather than a square box to avoid conflict with box detections.
-    <link name="ergobox">
-      <visual>
-        <origin xyz="0.0 0.0 0.0" rpy="0 0 0" />
-        <geometry>
-          <mesh filename="file://$(find r3mcell_cu_gazebo)/meshes/IALab/ergobox.dae" scale="1 1 1" />
-        </geometry>
-      </visual>
-      <collision>
-        <origin xyz="0.0 0.0 0.0" rpy="0 0 0" />
-        <geometry>
-          <mesh filename="file://$(find r3mcell_cu_gazebo)/meshes/IALab/ergobox.dae" scale="1 1 1" />
-        </geometry>
-      </collision>
-      <inertial>
-        <mass value="10.0"/>
-        <inertia ixx="0.0002" ixy="0.0002" ixz="0.0002" iyy="0.0" iyz="0.0" izz="0.0" />
-      </inertial>
-    </link>
-    <joint name="cell-ergobox-fixed" type="fixed">
-      <parent link="cell"/>
-      <child link="ergobox"/>
-      <origin xyz="-0.3 0.32 0.8605" rpy="0.0 0.0 0.0" />
-    </joint>
-    -->
+    <link name="cubePlacing">
+      <visual>
+        <origin xyz="0.0 0.0 0.0" rpy="0 0 0" />
+        <geometry>
+          <mesh filename="file://$(find r3mcell_cu_gazebo)/meshes/cubePP/cubePlacing.dae" scale="1 1 1" />
+        </geometry>
+      </visual>
+      <collision>
+        <origin xyz="0.0 0.0 0.0" rpy="0 0 0" />
+        <geometry>
+          <mesh filename="file://$(find r3mcell_cu_gazebo)/meshes/cubePP/cubePlacing.dae" scale="1 1 1" />
+        </geometry>
+      </collision>
+      <inertial>
+        <mass value="10.0"/>
+        <inertia ixx="0.0002" ixy="0.0002" ixz="0.0002" iyy="0.0" iyz="0.0" izz="0.0" />
+      </inertial>
+    </link>
+    <joint name="cell-cubePlacing-fixed" type="fixed">
+      <parent link="cell"/>
+      <child link="cubePlacing"/>
+      <origin xyz="-0.325 0.325 0.8605" rpy="0.0 0.0 0.0" />
+    </joint>
   </xacro:if>
   <xacro:if value="${r3mcell_cu_2}">

Commit message: Upload: R3M Testing use-case (+adapt current packages).

File: CranfieldUniversity/r3mcell_cu_gazebo/urdf/irb120.urdf.xacro (robot description, xacro)
@@ -56,4 +56,6 @@
   <xacro:arg name="r3mcell_cu_3" default="false"/>
   <xacro:property name="r3mcell_cu_3" value="$(arg r3mcell_cu_3)"/>
+  <xacro:arg name="r3mcell_cu_4" default="false"/>
+  <xacro:property name="r3mcell_cu_4" value="$(arg r3mcell_cu_4)"/>
   <!-- endeffector -->
   <xacro:arg name="EE_no" default="false"/>
@@ -229,4 +231,29 @@
     </joint>
   </xacro:if>
+  <xacro:if value="${r3mcell_cu_4}">
+    <link name="TestingTable">
+      <visual>
+        <origin xyz="0.0 0.0 0.0" rpy="0 0 0" />
+        <geometry>
+          <mesh filename="file://$(find r3mcell_cu_gazebo)/meshes/IALab/TestingTable.dae" scale="1 1 1" />
+        </geometry>
+      </visual>
+      <collision>
+        <origin xyz="0.0 0.0 0.0" rpy="0 0 0" />
+        <geometry>
+          <mesh filename="file://$(find r3mcell_cu_gazebo)/meshes/IALab/TestingTable.dae" scale="1 1 1" />
+        </geometry>
+      </collision>
+      <inertial>
+        <mass value="10.0"/>
+        <inertia ixx="0.0002" ixy="0.0002" ixz="0.0002" iyy="0.0" iyz="0.0" izz="0.0" />
+      </inertial>
+    </link>
+    <joint name="TestingTable_joint" type="fixed">
+      <parent link="cell"/>
+      <child link="TestingTable"/>
+      <origin xyz="0.0 0.0 0.0" rpy="0.0 0.0 0.0" />
+    </joint>
+  </xacro:if>
   <!-- CAMERA -->
   <xacro:unless value="${bringup}">
