Commit message: Add camera to urdf file.

File: CranfieldUniversity/r3mcell_cu_gazebo/urdf/r3mcell_cu_cylinderstacking.urdf.xacro (robot description, xacro)
@@ -121,3 +121,62 @@
     <origin xyz="0.0 0.0 0.0" rpy="0.0 0.0 0.0" />
   </joint>
+  <!-- CAMERA -->
+  <xacro:unless value="${bringup}">
+    <link name="camera_link">
+      <collision>
+        <origin xyz="0 0 0" rpy="0 0 0"/>
+        <geometry>
+          <box size="0.05 0.05 0.05"/>
+        </geometry>
+      </collision>
+      <visual>
+        <origin xyz="0 0 0" rpy="0 0 0"/>
+        <geometry>
+          <box size="0.05 0.05 0.05"/>
+        </geometry>
+      </visual>
+      <inertial>
+        <mass value="1.0" />
+        <origin xyz="0 0 0" rpy="0 0 0"/>
+        <inertia ixx="0.0" ixy="0.0" ixz="0.0" iyy="0.0" iyz="0.0" izz="0.0" />
+      </inertial>
+    </link>
+    <joint name="camera_joint" type="fixed">
+      <origin xyz="0.776 0.526 1.90" rpy="0 1.23 3.1416"/>
+      <parent link="world"/>
+      <child link="camera_link"/>
+    </joint>
+    <gazebo reference="camera_link">
+      <sensor name="camera" type="camera">
+        <update_rate>30</update_rate>
+        <camera name="head">
+          <horizontal_fov>1.22</horizontal_fov>
+          <image>
+            <width>1920</width>
+            <height>1080</height>
+            <format>R8G8B8</format>
+          </image>
+          <clip>
+            <near>0.02</near>
+            <far>300</far>
+          </clip>
+          <noise>
+            <type>gaussian</type>
+            <mean>0.0</mean>
+            <stddev>0.007</stddev>
+          </noise>
+        </camera>
+        <plugin filename="libgazebo_ros_camera.so" name="camera_controller">
+          <robotNamespace/>
+          <alwaysOn>true</alwaysOn>
+          <updateRate>0.0</updateRate>
+          <cameraName>camera</cameraName>
+          <imageTopicName>image_raw</imageTopicName>
+          <cameraInfoTopicName>camera_info</cameraInfoTopicName>
+          <frameName>camera</frameName>
+          <hackBaseline>0.07</hackBaseline>
+        </plugin>
+      </sensor>
+    </gazebo>
+  </xacro:unless>
 </robot>

Commit message: Add aruco tag to r3mcell_cu_15 cell.

File: CranfieldUniversity/r3mcell_cu_gazebo/urdf/r3mcell_cu_cylinderstacking.urdf.xacro (robot description, xacro)
@@ -121,4 +121,30 @@
     <origin xyz="0.0 0.0 0.0" rpy="0.0 0.0 0.0" />
   </joint>
+  <!-- ARUCO TAG -->
+  <xacro:unless value="${bringup}">
+    <link name="aruco100">
+      <visual>
+        <origin xyz="0.0 0.0 0.0" rpy="0 0 0" />
+        <geometry>
+          <mesh filename="file://$(find r3mcell_cu_gazebo)/meshes/CylinderStacking/aruco100.dae" scale="1 1 1" />
+        </geometry>
+      </visual>
+      <collision>
+        <origin xyz="0.0 0.0 0.0" rpy="0 0 0" />
+        <geometry>
+          <mesh filename="file://$(find r3mcell_cu_gazebo)/meshes/CylinderStacking/aruco100.dae" scale="1 1 1" />
+        </geometry>
+      </collision>
+      <inertial>
+        <mass value="10.0"/>
+        <inertia ixx="0.0002" ixy="0.0002" ixz="0.0002" iyy="0.0" iyz="0.0" izz="0.0" />
+      </inertial>
+    </link>
+    <joint name="cell-aruco100-fixed" type="fixed">
+      <parent link="cell"/>
+      <child link="aruco100"/>
+      <origin xyz="-0.05 -0.05 0.0" rpy="0.0 0.0 0.0" />
+    </joint>
+  </xacro:unless>
   <!-- CAMERA -->
   <xacro:unless value="${bringup}">

Commit message: Add ArUco grid to r3mcell_cu_15 urdf.

File: CranfieldUniversity/r3mcell_cu_gazebo/urdf/r3mcell_cu_cylinderstacking.urdf.xacro (robot description, xacro)
@@ -123,4 +123,5 @@
   <!-- ARUCO TAG -->
   <xacro:unless value="${bringup}">
+    <!-- Single ARUCO
     <link name="aruco100">
       <visual>
@@ -147,4 +148,32 @@
     </joint>
     <gazebo reference="cell-aruco100-fixed">
+      <preserveFixedJoint>true</preserveFixedJoint>
+    </gazebo>
+    -->
+    <!-- ARUCO GRID -->
+    <link name="aruco_grid">
+      <visual>
+        <origin xyz="0.0 0.0 0.0" rpy="0 0 0" />
+        <geometry>
+          <mesh filename="file://$(find r3mcell_cu_gazebo)/meshes/CylinderStacking/arucoGrid.dae" scale="1 1 1" />
+        </geometry>
+      </visual>
+      <collision>
+        <origin xyz="0.0 0.0 0.0" rpy="0 0 0" />
+        <geometry>
+          <mesh filename="file://$(find r3mcell_cu_gazebo)/meshes/CylinderStacking/arucoGrid.dae" scale="1 1 1" />
+        </geometry>
+      </collision>
+      <inertial>
+        <mass value="10.0"/>
+        <inertia ixx="0.0002" ixy="0.0002" ixz="0.0002" iyy="0.0" iyz="0.0" izz="0.0" />
+      </inertial>
+    </link>
+    <joint name="cell-aruco_grid-fixed" type="fixed">
+      <parent link="cell"/>
+      <child link="aruco_grid"/>
+      <origin xyz="0.0 0.0 0.0" rpy="0.0 0.0 0.0" />
+    </joint>
+    <gazebo reference="cell-aruco_grid-fixed">
       <preserveFixedJoint>true</preserveFixedJoint>
     </gazebo>
