Commit message: Remove holes in IRB120 enclosure.

File: CranfieldUniversity/r3mcell_cu_gazebo/urdf/r3mcell_cu_cubekitting.urdf.xacro (robot description, xacro)
@@ -73,5 +73,5 @@
       <origin xyz="0.0 0.0 0.0" rpy="0 0 0" />
       <geometry>
-        <mesh filename="file://$(find r3mcell_cu_gazebo)/meshes/IRB120enclosure/IRB120enclosure.dae" scale="1 1 1" />
+        <mesh filename="file://$(find r3mcell_cu_gazebo)/meshes/IRB120enclosure/IRB120enclosure_noholes.dae" scale="1 1 1" />
       </geometry>
     </visual>
@@ -79,5 +79,5 @@
       <origin xyz="0.0 0.0 0.0" rpy="0 0 0" />
       <geometry>
-        <mesh filename="file://$(find r3mcell_cu_gazebo)/meshes/IRB120enclosure/IRB120enclosure.dae" scale="1 1 1" />
+        <mesh filename="file://$(find r3mcell_cu_gazebo)/meshes/IRB120enclosure/IRB120enclosure_noholes.dae" scale="1 1 1" />
       </geometry>
     </collision>

File: CranfieldUniversity/r3mcell_cu_gazebo/urdf/r3mcell_cu_cylinderstacking.urdf.xacro (robot description, xacro)
@@ -73,5 +73,5 @@
       <origin xyz="0.0 0.0 0.0" rpy="0 0 0" />
       <geometry>
-        <mesh filename="file://$(find r3mcell_cu_gazebo)/meshes/IRB120enclosure/IRB120enclosure.dae" scale="1 1 1" />
+        <mesh filename="file://$(find r3mcell_cu_gazebo)/meshes/IRB120enclosure/IRB120enclosure_noholes.dae" scale="1 1 1" />
       </geometry>
     </visual>
@@ -79,5 +79,5 @@
       <origin xyz="0.0 0.0 0.0" rpy="0 0 0" />
       <geometry>
-        <mesh filename="file://$(find r3mcell_cu_gazebo)/meshes/IRB120enclosure/IRB120enclosure.dae" scale="1 1 1" />
+        <mesh filename="file://$(find r3mcell_cu_gazebo)/meshes/IRB120enclosure/IRB120enclosure_noholes.dae" scale="1 1 1" />
       </geometry>
     </collision>

Commit message: Add: ArUco Grid to r3mcell _11 and _12 layouts.

File: CranfieldUniversity/r3mcell_cu_gazebo/urdf/r3mcell_cu_cubekitting.urdf.xacro (robot description, xacro)
@@ -116,5 +116,5 @@
     <parent link="cell"/>
     <child link="KittingTray"/>
-    <origin xyz="-0.6 0.0 0.0" rpy="0.0 0.0 0.0" />
+    <origin xyz="-0.4 0.0 0.0" rpy="0.0 0.0 0.0" />
   </joint>
   <!-- Robot+Cell JOINT -->
@@ -124,4 +124,34 @@
     <origin xyz="-0.6506 0.6489 0.8605" rpy="0.0 0.0 0.0" />
   </joint>
+  <!-- ARUCO TAG -->
+  <xacro:unless value="${bringup}">
+    <!-- ARUCO GRID -->
+    <link name="aruco_grid">
+      <visual>
+        <origin xyz="0.0 0.0 0.0" rpy="0 0 0" />
+        <geometry>
+          <mesh filename="file://$(find r3mcell_cu_gazebo)/meshes/aruco/arucoGrid.dae" scale="1 1 1" />
+        </geometry>
+      </visual>
+      <collision>
+        <origin xyz="0.0 0.0 0.0" rpy="0 0 0" />
+        <geometry>
+          <mesh filename="file://$(find r3mcell_cu_gazebo)/meshes/aruco/arucoGrid.dae" scale="1 1 1" />
+        </geometry>
+      </collision>
+      <inertial>
+        <mass value="10.0"/>
+        <inertia ixx="0.0002" ixy="0.0002" ixz="0.0002" iyy="0.0" iyz="0.0" izz="0.0" />
+      </inertial>
+    </link>
+    <joint name="cell-aruco_grid-fixed" type="fixed">
+      <parent link="cell"/>
+      <child link="aruco_grid"/>
+      <origin xyz="0.0 0.0 0.0" rpy="0.0 0.0 0.0" />
+    </joint>
+    <gazebo reference="cell-aruco_grid-fixed">
+      <preserveFixedJoint>true</preserveFixedJoint>
+    </gazebo>
+  </xacro:unless>
   <!-- CAMERA -->
   <xacro:unless value="${bringup}">

File: CranfieldUniversity/r3mcell_cu_gazebo/urdf/r3mcell_cu_cubestacking.urdf.xacro (robot description, xacro)
@@ -99,4 +99,34 @@
     <origin xyz="-0.6506 0.6489 0.8605" rpy="0.0 0.0 0.0" />
   </joint>
+  <!-- ARUCO TAG -->
+  <xacro:unless value="${bringup}">
+    <!-- ARUCO GRID -->
+    <link name="aruco_grid">
+      <visual>
+        <origin xyz="0.0 0.0 0.0" rpy="0 0 0" />
+        <geometry>
+          <mesh filename="file://$(find r3mcell_cu_gazebo)/meshes/aruco/arucoGrid.dae" scale="1 1 1" />
+        </geometry>
+      </visual>
+      <collision>
+        <origin xyz="0.0 0.0 0.0" rpy="0 0 0" />
+        <geometry>
+          <mesh filename="file://$(find r3mcell_cu_gazebo)/meshes/aruco/arucoGrid.dae" scale="1 1 1" />
+        </geometry>
+      </collision>
+      <inertial>
+        <mass value="10.0"/>
+        <inertia ixx="0.0002" ixy="0.0002" ixz="0.0002" iyy="0.0" iyz="0.0" izz="0.0" />
+      </inertial>
+    </link>
+    <joint name="cell-aruco_grid-fixed" type="fixed">
+      <parent link="cell"/>
+      <child link="aruco_grid"/>
+      <origin xyz="0.0 0.0 0.0" rpy="0.0 0.0 0.0" />
+    </joint>
+    <gazebo reference="cell-aruco_grid-fixed">
+      <preserveFixedJoint>true</preserveFixedJoint>
+    </gazebo>
+  </xacro:unless>
   <!-- CAMERA -->
   <xacro:unless value="${bringup}">
