Commit message: Adapt: r3mcell_cu_ur3 cell to include ArUco markers.

File: CranfieldUniversity/r3mcell_cu_gazebo/urdf/r3mcell_cu_CSTur.urdf.xacro (robot description, xacro)
@@ -109,29 +109,4 @@
     <origin xyz="0.0 0.0 0.85" rpy="0.0 0.0 0.0" />
   </joint>
-  <!-- Kitting Tray -->
-  <link name="KittingTray">
-    <visual>
-      <origin xyz="0.0 0.0 0.0" rpy="0 0 0" />
-      <geometry>
-        <mesh filename="file://$(find r3mcell_cu_gazebo)/meshes/CubeKitting/KittingTray_UR.dae" scale="1 1 1" />
-      </geometry>
-    </visual>
-    <collision>
-      <origin xyz="0.0 0.0 0.0" rpy="0 0 0" />
-      <geometry>
-        <mesh filename="file://$(find r3mcell_cu_gazebo)/meshes/CubeKitting/KittingTray_UR.dae" scale="1 1 1" />
-      </geometry>
-    </collision>
-    <inertial>
-      <mass value="10.0"/>
-      <inertia ixx="500.0" ixy="500.0" ixz="500.0" iyy="500.0" iyz="500.0" izz="500.0" />
-    </inertial>
-  </link>
-  <!-- Kitting Tray: FIXED JOINT -->
-  <joint name="tray-cell-fixed" type="fixed">
-    <parent link="ur3_stand"/>
-    <child link="KittingTray"/>
-    <origin xyz="0.02 -0.16 0.0" rpy="0.0 0.0 0.0" />
-  </joint>
   <!-- ARUCO TAG -->
   <xacro:unless value="${bringup}">

File: CranfieldUniversity/r3mcell_cu_gazebo/urdf/r3mcell_cu_CSur.urdf.xacro (robot description, xacro)
@@ -135,32 +135,4 @@
   <!-- ARUCO TAG -->
   <xacro:unless value="${bringup}">
-    <!-- Single ARUCO
-    <link name="aruco100">
-      <visual>
-        <origin xyz="0.0 0.0 0.0" rpy="0 0 0" />
-        <geometry>
-          <mesh filename="file://$(find r3mcell_cu_gazebo)/meshes/aruco/aruco100_UR.dae" scale="1 1 1" />
-        </geometry>
-      </visual>
-      <collision>
-        <origin xyz="0.0 0.0 0.0" rpy="0 0 0" />
-        <geometry>
-          <mesh filename="file://$(find r3mcell_cu_gazebo)/meshes/aruco/aruco100_UR.dae" scale="1 1 1" />
-        </geometry>
-      </collision>
-      <inertial>
-        <mass value="10.0"/>
-        <inertia ixx="0.0002" ixy="0.0002" ixz="0.0002" iyy="0.0" iyz="0.0" izz="0.0" />
-      </inertial>
-    </link>
-    <joint name="ur3_stand-aruco100-fixed" type="fixed">
-      <parent link="ur3_stand"/>
-      <child link="aruco100_UR"/>
-      <origin xyz="-0.05 -0.05 0.0" rpy="0.0 0.0 0.0" />
-    </joint>
-    <gazebo reference="cell-aruco100-fixed">
-      <preserveFixedJoint>true</preserveFixedJoint>
-    </gazebo>
-    -->
     <!-- ARUCO GRID -->
     <link name="aruco_grid">
