Commit message: Move BD fixture x=0.05m.

File: CranfieldUniversity/r3mcell_cu_gazebo/urdf/r3mcell_cu_BD.urdf.xacro (robot description, xacro)
@@ -121,5 +121,5 @@
     <parent link="cell"/>
     <child link="BD_Fixture"/>
-    <origin xyz="0.0 0.0 0.0" rpy="0.0 0.0 0.0" />
+    <origin xyz="0.05 0.0 0.0" rpy="0.0 0.0 0.0" />
   </joint>
   <!-- R3M Cranfield Uni Cell: BD -> ERGOBOX -->
