Commit message: Re-structure R3MCell: APG Section (liaison missing).

File: CranfieldUniversity/r3mcell_cu_gazebo/urdf/objects/Cube.urdf (robot description, URDF)
Before this commit: robot can, 1 links, 0 joints
Links:
- removed link can
- added link ${name}, mass 0.1; collision mesh filename=file://$(find r3mcell_cu_gazebo)/meshes/objects/${name}.dae; visual mesh filename=file://$(find r3mcell_cu_gazebo)/meshes/objects/${name}.dae
