Commit message: Fix UseCase configurations (urdf + mesh files).

File: CranfieldUniversity/r3mcell_cu_gazebo/urdf/objects/BaseCylinder.urdf (robot description, URDF)
Before this commit: robot LamSheet, 1 links, 0 joints
Links:
- removed link LamSheet
- added link BaseCylinder, mass 0.1; collision mesh filename=file://$(find r3mcell_cu_gazebo)/meshes/CylinderStacking/Ba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; visual mesh filename=file://$(find r3mcell_cu_gazebo)/meshes/CylinderStacking/Ba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

File: CranfieldUniversity/r3mcell_cu_gazebo/urdf/objects/Battery.urdf (robot description, URDF)
Before this commit: robot LamSheet, 1 links, 0 joints
Links:
- removed link LamSheet
- added link Battery, mass 0.1; collision mesh filename=file://$(find r3mcell_cu_gazebo)/meshes/BatteryDisassembly/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; visual mesh filename=file://$(find r3mcell_cu_gazebo)/meshes/BatteryDisassembly/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

File: CranfieldUniversity/r3mcell_cu_gazebo/urdf/objects/BlueCube.urdf (robot description, URDF)
Before this commit: robot LamSheet, 1 links, 0 joints
Links:
- removed link LamSheet
- added link RedCube, mass 0.1; collision mesh filename=file://$(find r3mcell_cu_gazebo)/meshes/CubeKitting/BlueCub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; visual mesh filename=file://$(find r3mcell_cu_gazebo)/meshes/CubeKitting/BlueCub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

File: CranfieldUniversity/r3mcell_cu_gazebo/urdf/objects/BottomCube.urdf (robot description, URDF)
Before this commit: robot LamSheet, 1 links, 0 joints
Links:
- removed link LamSheet
- added link BottomCube, mass 0.1; collision mesh filename=file://$(find r3mcell_cu_gazebo)/meshes/CubeStacking/Bottom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; visual mesh filename=file://$(find r3mcell_cu_gazebo)/meshes/CubeStacking/Bottom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

File: CranfieldUniversity/r3mcell_cu_gazebo/urdf/objects/Can.urdf (robot description, URDF)
Before this commit: robot assembly, 1 links, 0 joints
Links:
- removed link ${name}
- added link Can, mass 0.1; collision mesh filename=file://$(find r3mcell_cu_gazebo)/meshes/canPP/Can.dae; visual mesh filename=file://$(find r3mcell_cu_gazebo)/meshes/canPP/Can.dae

File: CranfieldUniversity/r3mcell_cu_gazebo/urdf/objects/EmptyAssembly.urdf (robot description, URDF)
Before this commit: robot cube, 1 links, 0 joints
Links:
- removed link ${name}
- added link EmptyAssembly, mass 1.0; collision mesh filename=file://$(find r3mcell_cu_gazebo)/meshes/CylinderStacking/Em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; visual mesh filename=file://$(find r3mcell_cu_gazebo)/meshes/CylinderStacking/Em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

File: CranfieldUniversity/r3mcell_cu_gazebo/urdf/objects/FullAssembly.urdf (robot description, URDF)
Before this commit: robot LamSheet, 1 links, 0 joints
Links:
- removed link LamSheet
- added link FullAssembly, mass 1.0; collision mesh filename=file://$(find r3mcell_cu_gazebo)/meshes/CylinderStacking/Fu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; visual mesh filename=file://$(find r3mcell_cu_gazebo)/meshes/CylinderStacking/Fu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

File: CranfieldUniversity/r3mcell_cu_gazebo/urdf/objects/GreenCube.urdf (robot description, URDF)
Before this commit: robot can, 1 links, 0 joints
Links:
- removed link can
- added link GreenCube, mass 0.1; collision mesh filename=file://$(find r3mcell_cu_gazebo)/meshes/CubeKitting/GreenCu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; visual mesh filename=file://$(find r3mcell_cu_gazebo)/meshes/CubeKitting/GreenCu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

File: CranfieldUniversity/r3mcell_cu_gazebo/urdf/objects/MidAssembly.urdf (robot description, URDF)
Before this commit: robot LamSheet, 1 links, 0 joints
Links:
- removed link LamSheet
- added link MidAssembly, mass 1.0; collision mesh filename=file://$(find r3mcell_cu_gazebo)/meshes/CylinderStacking/Mi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; visual mesh filename=file://$(find r3mcell_cu_gazebo)/meshes/CylinderStacking/Mi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

File: CranfieldUniversity/r3mcell_cu_gazebo/urdf/objects/RedCube.urdf (robot description, URDF)
Before this commit: robot LamSheet, 1 links, 0 joints
Links:
- removed link LamSheet
- added link RedCube, mass 0.1; collision mesh filename=file://$(find r3mcell_cu_gazebo)/meshes/CubeKitting/RedCube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; visual mesh filename=file://$(find r3mcell_cu_gazebo)/meshes/CubeKitting/RedCube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

File: CranfieldUniversity/r3mcell_cu_gazebo/urdf/objects/TopCube.urdf (robot description, URDF)
Before this commit: robot cube, 1 links, 0 joints
Links:
- removed link ${name}
- added link TopCube, mass 0.1; collision mesh filename=file://$(find r3mcell_cu_gazebo)/meshes/CubeStacking/TopCub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; visual mesh filename=file://$(find r3mcell_cu_gazebo)/meshes/CubeStacking/TopCub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

File: CranfieldUniversity/r3mcell_cu_gazebo/urdf/objects/TopCylinder.urdf (robot description, URDF)
Before this commit: robot LamSheet, 1 links, 0 joints
Links:
- removed link LamSheet
- added link TopCylinder, mass 0.1; collision mesh filename=file://$(find r3mcell_cu_gazebo)/meshes/CylinderStacking/To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; visual mesh filename=file://$(find r3mcell_cu_gazebo)/meshes/CylinderStacking/To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

File: CranfieldUniversity/r3mcell_cu_gazebo/urdf/objects/WhiteCube.urdf (robot description, URDF)
Before this commit: robot LamSheet, 1 links, 0 joints
Links:
- removed link LamSheet
- added link WhiteCube, mass 0.1; collision mesh filename=file://$(find r3mcell_cu_gazebo)/meshes/CubeKitting/WhiteCu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; visual mesh filename=file://$(find r3mcell_cu_gazebo)/meshes/CubeKitting/WhiteCu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

File: CranfieldUniversity/r3mcell_cu_gazebo/urdf/r3mcell_cu_1.urdf.xacro (robot description, xacro)
@@ -32,4 +32,6 @@
   <xacro:arg name="bringup" default="false"/>
   <xacro:property name="bringup" value="$(arg bringup)"/>
+  <xacro:arg name="hmi" default="false"/>
+  <xacro:property name="hmi" value="$(arg hmi)"/>
   <xacro:arg name="robot_ip" default="0.0.0.0"/>
   <xacro:property name="robot_ip" value="$(arg robot_ip)"/>
@@ -156,3 +158,15 @@
     </gazebo>
   </xacro:unless>
+  <!-- ros2srrc_HMI CAMERA -->
+  <xacro:if value="${hmi}">
+    <xacro:include filename="$(find ros2srrc_hmi)/urdf/hmicamera.urdf.xacro"/>
+    <xacro:HMI_camera
+      x="2.0"
+      y="1.25"
+      z="1.85"
+      roll="0.0"
+      pitch="0.35"
+      yaw="-2.6"
+    />
+  </xacro:if>
 </robot>

File: CranfieldUniversity/r3mcell_cu_gazebo/urdf/r3mcell_cu_2.urdf.xacro (robot description, xacro)
@@ -32,4 +32,6 @@
   <xacro:arg name="bringup" default="false"/>
   <xacro:property name="bringup" value="$(arg bringup)"/>
+  <xacro:arg name="hmi" default="false"/>
+  <xacro:property name="hmi" value="$(arg hmi)"/>
   <xacro:arg name="robot_ip" default="0.0.0.0"/>
   <xacro:property name="robot_ip" value="$(arg robot_ip)"/>
@@ -166,3 +168,15 @@
     </gazebo>
   </xacro:unless>
+  <!-- ros2srrc_HMI CAMERA -->
+  <xacro:if value="${hmi}">
+    <xacro:include filename="$(find ros2srrc_hmi)/urdf/hmicamera.urdf.xacro"/>
+    <xacro:HMI_camera
+      x="2.0"
+      y="1.25"
+      z="1.70"
+      roll="0.0"
+      pitch="0.35"
+      yaw="-2.6"
+    />
+  </xacro:if>
 </robot>

File: CranfieldUniversity/r3mcell_cu_gazebo/urdf/r3mcell_cu_BD.urdf.xacro (robot description, xacro)
@@ -48,4 +48,10 @@
     EE_name="${EE_name}"
   />
+  <!-- Include XACRO-MACRO file of the EGP64: -->
+  <xacro:include filename="$(find ros2srrc_endeffectors)/egp64/urdf/egp64v3_macro.urdf.xacro"/>
+  <xacro:egp64
+    bringup="${bringup}"
+    parent_link="tool0"
+  />
   <!-- Load ROS 2 Gazebo Plugin -->
   <xacro:unless value="${bringup}">
@@ -55,4 +61,6 @@
         <!-- IRB120 Controller -->
         <parameters>$(find ros2srrc_robots)/irb120/config/controller.yaml</parameters>
+        <!-- End-Effector Controller (if needed) -->
+        <parameters>$(find ros2srrc_endeffectors)/${EE_name}/config/controller.yaml</parameters>
       </plugin>
     </gazebo>
@@ -91,10 +99,10 @@
     <origin xyz="-0.6506 0.6489 0.8605" rpy="0.0 0.0 0.0" />
   </joint>
-  <!-- PERCEPTION TESTING: TABLE -->
-  <link name="TestingTable">
+  <!-- R3M Cranfield Uni Cell: BD -> Fixture -->
+  <link name="BD_Fixture">
     <visual>
       <origin xyz="0.0 0.0 0.0" rpy="0 0 0" />
       <geometry>
-        <mesh filename="file://$(find r3mcell_cu_gazebo)/meshes/PerceptionTest/TestingTable.dae" scale="1 1 1" />
+        <mesh filename="file://$(find r3mcell_cu_gazebo)/meshes/BatteryDisassembly/BD_TopBottom.dae" scale="1 1 1" />
       </geometry>
     </visual>
@@ -102,5 +110,5 @@
       <origin xyz="0.0 0.0 0.0" rpy="0 0 0" />
       <geometry>
-        <mesh filename="file://$(find r3mcell_cu_gazebo)/meshes/PerceptionTest/TestingTable.dae" scale="1 1 1" />
+        <mesh filename="file://$(find r3mcell_cu_gazebo)/meshes/BatteryDisassembly/BD_TopBottom.dae.dae" scale="1 1 1" />
       </geometry>
     </collision>
@@ -110,7 +118,7 @@
     </inertial>
   </link>
-  <joint name="TestingTable_joint" type="fixed">
+  <joint name="cell-BD_Fixture-fixed" type="fixed">
     <parent link="cell"/>
-    <child link="TestingTable"/>
+    <child link="BD_Fixture"/>
     <origin xyz="0.0 0.0 0.0" rpy="0.0 0.0 0.0" />
   </joint>
@@ -141,6 +149,9 @@
       <child link="camera_link"/>
     </joint>
+    <gazebo reference="camera_joint">
+      <preserveFixedJoint>true</preserveFixedJoint>
+    </gazebo>
     <gazebo reference="camera_link">
-      <sensor name="lenovoFHD_gazebo" type="camera">
+      <sensor name="camera" type="camera">
         <update_rate>30</update_rate>
         <camera name="head">
@@ -165,5 +176,5 @@
           <alwaysOn>true</alwaysOn>
           <updateRate>0.0</updateRate>
-          <cameraName>lenovoFHD_gazebo</cameraName>
+          <cameraName>camera</cameraName>
           <imageTopicName>image_raw</imageTopicName>
           <cameraInfoTopicName>camera_info</cameraInfoTopicName>

File: CranfieldUniversity/r3mcell_cu_gazebo/urdf/r3mcell_cu_CKur.urdf.xacro (robot description, xacro)
@@ -28,5 +28,5 @@
 # IFRA-Cranfield (2023) ROS 2 Sim-to-Real Robot Control. URL: https://github.com/IFRA-Cranfield/ros2_SimRealRobotControl.
 -->
-<robot name="irb120" xmlns:xacro="http://ros.org/wiki/xacro">
+<robot name="ur3" xmlns:xacro="http://ros.org/wiki/xacro">
   <!-- PASS ARGUMENTS: -->
   <xacro:arg name="bringup" default="false"/>
@@ -36,15 +36,31 @@
   <xacro:arg name="robot_ip" default="0.0.0.0"/>
   <xacro:property name="robot_ip" value="$(arg robot_ip)"/>
-  <xacro:arg name="EE" default="true"/>
+  <xacro:arg name="EE" default="false"/>
   <xacro:property name="EE" value="$(arg EE)"/>
   <xacro:arg name="EE_name" default="none"/>
   <xacro:property name="EE_name" value="$(arg EE_name)"/>
-  <!-- Include XACRO-MACRO file of the IRB120: -->
-  <xacro:include filename="$(find ros2srrc_robots)/irb120/urdf/irb120_macro.urdf.xacro"/>
-  <xacro:irb120
+  <!-- UR3 Control ARGUMENTS -->
+  <xacro:arg name="script_filename" default="none"/>
+  <xacro:property name="script_filename" value="$(arg script_filename)"/>
+  <xacro:arg name="input_recipe_filename" default="none"/>
+  <xacro:property name="input_recipe_filename" value="$(arg input_recipe_filename)"/>
+  <xacro:arg name="output_recipe_filename" default="none"/>
+  <xacro:property name="output_recipe_filename" value="$(arg output_recipe_filename)"/>
+  <!-- Include XACRO-MACRO file of the UR3: -->
+  <xacro:include filename="$(find ros2srrc_robots)/ur3/urdf/ur3_macro.urdf.xacro"/>
+  <xacro:ur3
     bringup="${bringup}"
     robot_ip="${robot_ip}"
     EE="${EE}"
     EE_name="${EE_name}"
+    script_filename="${script_filename}"
+    input_recipe_filename="${input_recipe_filename}"
+    output_recipe_filename="${output_recipe_filename}"
+  />
+  <!-- Include XACRO-MACRO file of the Robotiq 2f-85: -->
+  <xacro:include filename="$(find ros2srrc_endeffectors)/robotiq_hande/urdf/robotiq_hande_macro.urdf.xacro"/>
+  <xacro:robotiq_hande
+    bringup="${bringup}"
+    parent_link="tool0"
   />
   <!-- Load ROS 2 Gazebo Plugin -->
@@ -53,6 +69,8 @@
       <plugin filename="libgazebo_ros2_control.so" name="gazebo_ros2_control">
         <robot_sim_type>gazebo_ros2_control/GazeboSystem</robot_sim_type>
-        <!-- IRB120 Controller -->
-        <parameters>$(find ros2srrc_robots)/irb120/config/controller.yaml</parameters>
+        <!-- UR3 Controller -->
+        <parameters>$(find ros2srrc_robots)/ur3/config/controller.yaml</parameters>
+        <!-- End-Effector Controller (if needed) -->
+        <parameters>$(find ros2srrc_endeffectors)/${EE_name}/config/controller.yaml</parameters>
       </plugin>
     </gazebo>
@@ -60,10 +78,10 @@
   <!-- World: LINK -->
   <link name="world"/>
-  <!-- ABB IRB-120 ENCLOSURE -->
-  <link name="cell">
+  <!-- Robot Stand: LINK -->
+  <link name='ur3_stand'>
     <visual>
       <origin xyz="0.0 0.0 0.0" rpy="0 0 0" />
       <geometry>
-        <mesh filename="file://$(find r3mcell_cu_gazebo)/meshes/IRB120enclosure/IRB120enclosure.dae" scale="1 1 1" />
+        <mesh filename="file://$(find r3mcell_cu_gazebo)/meshes/UR3stand/ur3stand_complete.dae" scale="1 1 1" />
       </geometry>
     </visual>
@@ -71,5 +89,5 @@
       <origin xyz="0.0 0.0 0.0" rpy="0 0 0" />
       <geometry>
-        <mesh filename="file://$(find r3mcell_cu_gazebo)/meshes/IRB120enclosure/IRB120enclosure.dae" scale="1 1 1" />
+        <mesh filename="file://$(find r3mcell_cu_gazebo)/meshes/UR3stand/ur3stand_complete.dae" scale="1 1 1" />
       </geometry>
     </collision>
@@ -79,22 +97,22 @@
     </inertial>
   </link>
-  <!-- Robot Cell: FIXED JOINT -->
-  <joint name="world-cell-fixed" type="fixed">
-    <parent link="world"/>
-    <child link="cell"/>
-    <origin xyz="0.926 -0.124 0.0" rpy="0.0 0.0 0.0" />
+  <!-- Robot Stand: FIXED JOINT -->
+  <joint name="world_joint" type="fixed">
+    <parent link="world" />
+    <child link = "ur3_stand" />
+    <origin xyz="0.0 0.0 0.0" rpy="0.0 0.0 0.0" />
   </joint>
-  <!-- Robot+Cell JOINT -->
-  <joint name="cell-base_link-fixed" type="fixed">
-    <parent link="cell"/>
-    <child link="base_link"/>
-    <origin xyz="-0.6506 0.6489 0.8605" rpy="0.0 0.0 0.0" />
+  <!-- Robot Stand: Robot+Stand JOINT -->
+  <joint name="ur_joint" type="fixed">
+    <parent link="ur3_stand" />
+    <child link = "base_link" />
+    <origin xyz="0.0 0.0 0.85" rpy="0.0 0.0 0.0" />
   </joint>
-  <!-- PERCEPTION TESTING: TABLE -->
-  <link name="TestingTable">
+  <!-- Kitting Tray -->
+  <link name="KittingTray">
     <visual>
       <origin xyz="0.0 0.0 0.0" rpy="0 0 0" />
       <geometry>
-        <mesh filename="file://$(find r3mcell_cu_gazebo)/meshes/PerceptionTest/TestingTable.dae" scale="1 1 1" />
+        <mesh filename="file://$(find r3mcell_cu_gazebo)/meshes/CubeKitting/KittingTray_UR.dae" scale="1 1 1" />
       </geometry>
     </visual>
@@ -102,15 +120,16 @@
       <origin xyz="0.0 0.0 0.0" rpy="0 0 0" />
       <geometry>
-        <mesh filename="file://$(find r3mcell_cu_gazebo)/meshes/PerceptionTest/TestingTable.dae" scale="1 1 1" />
+        <mesh filename="file://$(find r3mcell_cu_gazebo)/meshes/CubeKitting/KittingTray_UR.dae" scale="1 1 1" />
       </geometry>
     </collision>
     <inertial>
       <mass value="10.0"/>
-      <inertia ixx="0.0002" ixy="0.0002" ixz="0.0002" iyy="0.0" iyz="0.0" izz="0.0" />
+      <inertia ixx="500.0" ixy="500.0" ixz="500.0" iyy="500.0" iyz="500.0" izz="500.0" />
     </inertial>
   </link>
-  <joint name="TestingTable_joint" type="fixed">
-    <parent link="cell"/>
-    <child link="TestingTable"/>
+  <!-- Kitting Tray: FIXED JOINT -->
+  <joint name="tray-cell-fixed" type="fixed">
+    <parent link="ur3_stand"/>
+    <child link="KittingTray"/>
     <origin xyz="0.0 0.0 0.0" rpy="0.0 0.0 0.0" />
   </joint>
@@ -137,10 +156,10 @@
     </link>
     <joint name="camera_joint" type="fixed">
-      <origin xyz="0.776 0.526 1.90" rpy="0 1.23 3.1416"/>
+      <origin xyz="0.0 0.32 2.09" rpy="0.0 1.5708 1.5708"/>
       <parent link="world"/>
       <child link="camera_link"/>
     </joint>
     <gazebo reference="camera_link">
-      <sensor name="lenovoFHD_gazebo" type="camera">
+      <sensor name="camera" type="camera">
         <update_rate>30</update_rate>
         <camera name="head">
@@ -165,5 +184,5 @@
           <alwaysOn>true</alwaysOn>
           <updateRate>0.0</updateRate>
-          <cameraName>lenovoFHD_gazebo</cameraName>
+          <cameraName>camera</cameraName>
           <imageTopicName>image_raw</imageTopicName>
           <cameraInfoTopicName>camera_info</cameraInfoTopicName>
@@ -180,5 +199,5 @@
       x="2.0"
       y="1.25"
-      z="1.85"
+      z="1.70"
       roll="0.0"
       pitch="0.35"

File: CranfieldUniversity/r3mcell_cu_gazebo/urdf/r3mcell_cu_LamStack.urdf.xacro (robot description, xacro)
@@ -32,4 +32,6 @@
   <xacro:arg name="bringup" default="false"/>
   <xacro:property name="bringup" value="$(arg bringup)"/>
+  <xacro:arg name="hmi" default="false"/>
+  <xacro:property name="hmi" value="$(arg hmi)"/>
   <xacro:arg name="robot_ip" default="0.0.0.0"/>
   <xacro:property name="robot_ip" value="$(arg robot_ip)"/>
@@ -144,3 +146,74 @@
     <origin xyz="-0.525 0.325 0.8605" rpy="0.0 0.0 3.1416" />
   </joint>
+  <!-- CAMERA -->
+  <xacro:unless value="${bringup}">
+    <link name="camera_link">
+      <collision>
+        <origin xyz="0 0 0" rpy="0 0 0"/>
+        <geometry>
+          <box size="0.05 0.05 0.05"/>
+        </geometry>
+      </collision>
+      <visual>
+        <origin xyz="0 0 0" rpy="0 0 0"/>
+        <geometry>
+          <box size="0.05 0.05 0.05"/>
+        </geometry>
+      </visual>
+      <inertial>
+        <mass value="1.0" />
+        <origin xyz="0 0 0" rpy="0 0 0"/>
+        <inertia ixx="0.0" ixy="0.0" ixz="0.0" iyy="0.0" iyz="0.0" izz="0.0" />
+      </inertial>
+    </link>
+    <joint name="camera_joint" type="fixed">
+      <origin xyz="0.776 0.526 1.90" rpy="0 1.23 3.1416"/>
+      <parent link="world"/>
+      <child link="camera_link"/>
+    </joint>
+    <gazebo reference="camera_link">
+      <sensor name="camera" type="camera">
+        <update_rate>30</update_rate>
+        <camera name="head">
+          <horizontal_fov>1.22</horizontal_fov>
+          <image>
+            <width>1920</width>
+            <height>1080</height>
+            <format>R8G8B8</format>
+          </image>
+          <clip>
+            <near>0.02</near>
+            <far>300</far>
+          </clip>
+          <noise>
+            <type>gaussian</type>
+            <mean>0.0</mean>
+            <stddev>0.007</stddev>
+          </noise>
+        </camera>
+        <plugin filename="libgazebo_ros_camera.so" name="camera_controller">
+          <robotNamespace/>
+          <alwaysOn>true</alwaysOn>
+          <updateRate>0.0</updateRate>
+          <cameraName>camera</cameraName>
+          <imageTopicName>image_raw</imageTopicName>
+          <cameraInfoTopicName>camera_info</cameraInfoTopicName>
+          <frameName>camera</frameName>
+          <hackBaseline>0.07</hackBaseline>
+        </plugin>
+      </sensor>
+    </gazebo>
+  </xacro:unless>
+  <!-- ros2srrc_HMI CAMERA -->
+  <xacro:if value="${hmi}">
+    <xacro:include filename="$(find ros2srrc_hmi)/urdf/hmicamera.urdf.xacro"/>
+    <xacro:HMI_camera
+      x="2.0"
+      y="1.25"
+      z="1.85"
+      roll="0.0"
+      pitch="0.35"
+      yaw="-2.6"
+    />
+  </xacro:if>
 </robot>

File: CranfieldUniversity/r3mcell_cu_gazebo/urdf/r3mcell_cu_canPP.urdf.xacro (robot description, xacro)
@@ -32,4 +32,6 @@
   <xacro:arg name="bringup" default="false"/>
   <xacro:property name="bringup" value="$(arg bringup)"/>
+  <xacro:arg name="hmi" default="false"/>
+  <xacro:property name="hmi" value="$(arg hmi)"/>
   <xacro:arg name="robot_ip" default="0.0.0.0"/>
   <xacro:property name="robot_ip" value="$(arg robot_ip)"/>
@@ -144,3 +146,74 @@
     <origin xyz="-0.425 0.225 0.8605" rpy="0.0 0.0 3.1416" />
   </joint>
+  <!-- CAMERA -->
+  <xacro:unless value="${bringup}">
+    <link name="camera_link">
+      <collision>
+        <origin xyz="0 0 0" rpy="0 0 0"/>
+        <geometry>
+          <box size="0.05 0.05 0.05"/>
+        </geometry>
+      </collision>
+      <visual>
+        <origin xyz="0 0 0" rpy="0 0 0"/>
+        <geometry>
+          <box size="0.05 0.05 0.05"/>
+        </geometry>
+      </visual>
+      <inertial>
+        <mass value="1.0" />
+        <origin xyz="0 0 0" rpy="0 0 0"/>
+        <inertia ixx="0.0" ixy="0.0" ixz="0.0" iyy="0.0" iyz="0.0" izz="0.0" />
+      </inertial>
+    </link>
+    <joint name="camera_joint" type="fixed">
+      <origin xyz="0.776 0.526 1.90" rpy="0 1.23 3.1416"/>
+      <parent link="world"/>
+      <child link="camera_link"/>
+    </joint>
+    <gazebo reference="camera_link">
+      <sensor name="camera" type="camera">
+        <update_rate>30</update_rate>
+        <camera name="head">
+          <horizontal_fov>1.22</horizontal_fov>
+          <image>
+            <width>1920</width>
+            <height>1080</height>
+            <format>R8G8B8</format>
+          </image>
+          <clip>
+            <near>0.02</near>
+            <far>300</far>
+          </clip>
+          <noise>
+            <type>gaussian</type>
+            <mean>0.0</mean>
+            <stddev>0.007</stddev>
+          </noise>
+        </camera>
+        <plugin filename="libgazebo_ros_camera.so" name="camera_controller">
+          <robotNamespace/>
+          <alwaysOn>true</alwaysOn>
+          <updateRate>0.0</updateRate>
+          <cameraName>camera</cameraName>
+          <imageTopicName>image_raw</imageTopicName>
+          <cameraInfoTopicName>camera_info</cameraInfoTopicName>
+          <frameName>camera</frameName>
+          <hackBaseline>0.07</hackBaseline>
+        </plugin>
+      </sensor>
+    </gazebo>
+  </xacro:unless>
+  <!-- ros2srrc_HMI CAMERA -->
+  <xacro:if value="${hmi}">
+    <xacro:include filename="$(find ros2srrc_hmi)/urdf/hmicamera.urdf.xacro"/>
+    <xacro:HMI_camera
+      x="2.0"
+      y="1.25"
+      z="1.85"
+      roll="0.0"
+      pitch="0.35"
+      yaw="-2.6"
+    />
+  </xacro:if>
 </robot>
