Commit message: R3M use-cases update (18-12-2024).

File: CranfieldUniversity/r3mcell_cu_gazebo/urdf/objects/BlueCube.urdf (robot description, URDF)
Before this commit: robot BlueCube, 1 links, 0 joints
Links:
- removed link RedCube
- added link BlueCube, mass 0.1; collision mesh filename=file://$(find r3mcell_cu_gazebo)/meshes/CubeKitting/BlueCub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; visual mesh filename=file://$(find r3mcell_cu_gazebo)/meshes/CubeKitting/BlueCub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

File: CranfieldUniversity/r3mcell_cu_gazebo/urdf/r3mcell_cu_BD.urdf.xacro (robot description, xacro)
@@ -110,5 +110,5 @@
       <origin xyz="0.0 0.0 0.0" rpy="0 0 0" />
       <geometry>
-        <mesh filename="file://$(find r3mcell_cu_gazebo)/meshes/BatteryDisassembly/BD_TopBottom.dae.dae" scale="1 1 1" />
+        <mesh filename="file://$(find r3mcell_cu_gazebo)/meshes/BatteryDisassembly/BD_TopBottom.dae" scale="1 1 1" />
       </geometry>
     </collision>

File: CranfieldUniversity/r3mcell_cu_gazebo/urdf/r3mcell_cu_cubekitting.urdf.xacro (robot description, xacro)
@@ -116,5 +116,5 @@
     <parent link="cell"/>
     <child link="KittingTray"/>
-    <origin xyz="0.0 0.0 0.0" rpy="0.0 0.0 0.0" />
+    <origin xyz="-0.6 0.0 0.0" rpy="0.0 0.0 0.0" />
   </joint>
   <!-- Robot+Cell JOINT -->
