Commit message: Modify battery (urdf and dae files).

File: CranfieldUniversity/r3mcell_cu_gazebo/urdf/objects/Battery.urdf (robot description, URDF)
Before this commit: robot Battery, 1 links, 0 joints
Links:
- removed link Battery
- added link ${name}, mass 0.1; collision mesh filename=file://$(find r3mcell_cu_gazebo)/meshes/BatteryDisassembly/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; visual mesh filename=file://$(find r3mcell_cu_gazebo)/meshes/BatteryDisassembly/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
