Commit message: Upload: TallMount to AMRC Cell.

File: AMRC/r3mcell_amrc_gazebo/urdf/r3mcell_amrc_CubeKitting.urdf.xacro (robot description, xacro)
@@ -113,4 +113,28 @@
     <origin xyz="0.0 0.0 0.0" rpy="0.0 0.0 0.0" />
   </joint>
+  <!-- ReconCell: TallMount -->
+  <link name="TallMount">
+    <visual>
+      <origin xyz="0.0 0.0 0.0" rpy="0 0 0" />
+      <geometry>
+        <mesh filename="file://$(find r3mcell_amrc_gazebo)/meshes/ReconCell/TallMount.dae" scale="1 1 1" />
+      </geometry>
+    </visual>
+    <collision>
+      <origin xyz="0.0 0.0 0.0" rpy="0 0 0" />
+      <geometry>
+        <mesh filename="file://$(find r3mcell_amrc_gazebo)/meshes/ReconCell/TallMount.dae" scale="1 1 1" />
+      </geometry>
+    </collision>
+    <inertial>
+      <mass value="1000.0"/>
+      <inertia ixx="500.0" ixy="500.0" ixz="500.0" iyy="500.0" iyz="500.0" izz="500.0" />
+    </inertial>
+  </link>
+  <joint name="world-TallMount-fixed" type="fixed">
+    <parent link="world"/>
+    <child link="TallMount"/>
+    <origin xyz="0.0 0.0 0.0" rpy="0.0 0.0 0.0" />
+  </joint>
   <!-- IRB1200 - Adapter Plate -->
   <link name="adapter_plate">
