Commit message: R3M use-cases update (19-12-2024).

File: AMRC/r3mcell_amrc_gazebo/urdf/r3mcell_amrc_2.urdf.xacro (robot description, xacro)
@@ -32,4 +32,6 @@
   <xacro:arg name="bringup" default="false"/>
   <xacro:property name="bringup" value="$(arg bringup)"/>
+  <xacro:arg name="hmi" default="false"/>
+  <xacro:property name="hmi" value="$(arg hmi)"/>
   <xacro:arg name="robot_ip" default="0.0.0.0"/>
   <xacro:property name="robot_ip" value="$(arg robot_ip)"/>
@@ -114,3 +116,15 @@
     <origin xyz="0.0 0.0 0.0" rpy="0.0 0.0 0.0" />
   </joint>
+  <!-- ros2srrc_HMI CAMERA -->
+  <xacro:if value="${hmi}">
+    <xacro:include filename="$(find ros2srrc_hmi)/urdf/hmicamera.urdf.xacro"/>
+    <xacro:HMI_camera
+      x="3.5"
+      y="3.5"
+      z="2.5"
+      roll="0.0"
+      pitch="0.35"
+      yaw="-2.5"
+    />
+  </xacro:if>
 </robot>

File: AMRC/r3mcell_amrc_gazebo/urdf/r3mcell_amrc_BD.urdf.xacro (robot description, xacro)
@@ -32,4 +32,6 @@
   <xacro:arg name="bringup" default="false"/>
   <xacro:property name="bringup" value="$(arg bringup)"/>
+  <xacro:arg name="hmi" default="false"/>
+  <xacro:property name="hmi" value="$(arg hmi)"/>
   <xacro:arg name="robot_ip" default="0.0.0.0"/>
   <xacro:property name="robot_ip" value="$(arg robot_ip)"/>
@@ -274,3 +276,15 @@
     <material>Gazebo/Grey</material>
   </gazebo>
+  <!-- ros2srrc_HMI CAMERA -->
+  <xacro:if value="${hmi}">
+    <xacro:include filename="$(find ros2srrc_hmi)/urdf/hmicamera.urdf.xacro"/>
+    <xacro:HMI_camera
+      x="1.5"
+      y="4.0"
+      z="2.5"
+      roll="0.0"
+      pitch="0.35"
+      yaw="-1.75"
+    />
+  </xacro:if>
 </robot>

File: AMRC/r3mcell_amrc_gazebo/urdf/r3mcell_amrc_CK_1200.urdf.xacro (robot description, xacro)
@@ -48,4 +48,33 @@
     EE_name="${EE_name}"
   />
+  <!-- Include: IRB1200/GPP5010NC ADAPTER -->
+  <link name="adapter">
+    <visual>
+      <geometry>
+        <mesh filename="file://$(find ros2srrc_endeffectors)/gpp5010nc/meshes/gpp5010nc_irb1200_Adapter.dae" />
+      </geometry>
+    </visual>
+    <collision>
+      <geometry>
+        <mesh filename="file://$(find ros2srrc_endeffectors)/gpp5010nc/meshes/gpp5010nc_irb1200_Adapter.dae" />
+      </geometry>
+    </collision>
+    <inertial>
+      <origin xyz="0 0 0" rpy="0 0 0" />
+      <mass value="0.001" />
+      <inertia ixx="0.001" ixy="0.0" ixz="0.0" iyy="0.001" iyz="0.0" izz="0.001"/>
+    </inertial>
+  </link>
+  <joint name="adapter_joint" type="fixed">
+    <origin xyz="0.0 0.0 0.0125" rpy="0 1.5708 3.1416" />
+    <parent link="tool0"/>
+    <child link="adapter"/>
+  </joint>
+  <!-- Include XACRO-MACRO file of the GPP5010NC: -->
+  <xacro:include filename="$(find ros2srrc_endeffectors)/gpp5010nc/urdf/gpp5010ncv2_macro.urdf.xacro"/>
+  <xacro:gpp5010nc
+    bringup="${bringup}"
+    parent_link="adapter"
+  />
   <!-- Load ROS 2 Gazebo Plugin -->
   <xacro:unless value="${bringup}">
@@ -55,4 +84,6 @@
         <!-- IRB1200 Controller -->
         <parameters>$(find ros2srrc_robots)/irb1200/config/controller.yaml</parameters>
+        <!-- End-Effector Controller (if needed) -->
+        <parameters>$(find ros2srrc_endeffectors)/${EE_name}/config/controller.yaml</parameters>
       </plugin>
     </gazebo>
@@ -168,7 +199,7 @@
     <xacro:include filename="$(find ros2srrc_hmi)/urdf/hmicamera.urdf.xacro"/>
     <xacro:HMI_camera
-      x="3.00"
-      y="1.50"
-      z="1.70"
+      x="2.0"
+      y="1.10"
+      z="1.25"
       roll="0.0"
       pitch="0.35"

File: AMRC/r3mcell_amrc_gazebo/urdf/r3mcell_amrc_CyS_1200.urdf.xacro (robot description, xacro)
@@ -32,4 +32,6 @@
   <xacro:arg name="bringup" default="false"/>
   <xacro:property name="bringup" value="$(arg bringup)"/>
+  <xacro:arg name="hmi" default="false"/>
+  <xacro:property name="hmi" value="$(arg hmi)"/>
   <xacro:arg name="robot_ip" default="0.0.0.0"/>
   <xacro:property name="robot_ip" value="$(arg robot_ip)"/>
@@ -70,5 +72,5 @@
   </joint>
   <!-- Include XACRO-MACRO file of the GPP5010NC: -->
-  <xacro:include filename="$(find ros2srrc_endeffectors)/gpp5010nc/urdf/gpp5010ncv2_macro.urdf.xacro"/>
+  <xacro:include filename="$(find ros2srrc_endeffectors)/gpp5010nc/urdf/gpp5010nc_macro.urdf.xacro"/>
   <xacro:gpp5010nc
     bringup="${bringup}"
@@ -193,3 +195,15 @@
     <origin xyz="0.0 0.0 0.0" rpy="0.0 0.0 0.0" />
   </joint>
+  <!-- ros2srrc_HMI CAMERA -->
+  <xacro:if value="${hmi}">
+    <xacro:include filename="$(find ros2srrc_hmi)/urdf/hmicamera.urdf.xacro"/>
+    <xacro:HMI_camera
+      x="2.0"
+      y="1.10"
+      z="1.25"
+      roll="0.0"
+      pitch="0.35"
+      yaw="-2.6"
+    />
+  </xacro:if>
 </robot>

File: AMRC/r3mcell_amrc_gazebo/urdf/r3mcell_amrc_LamStack.urdf.xacro (robot description, xacro)
@@ -32,4 +32,6 @@
   <xacro:arg name="bringup" default="false"/>
   <xacro:property name="bringup" value="$(arg bringup)"/>
+  <xacro:arg name="hmi" default="false"/>
+  <xacro:property name="hmi" value="$(arg hmi)"/>
   <xacro:arg name="robot_ip" default="0.0.0.0"/>
   <xacro:property name="robot_ip" value="$(arg robot_ip)"/>
@@ -214,3 +216,15 @@
     <origin xyz="0.0 0.0 0.139" rpy="0.0 0.0 0.0" />
   </joint>
+  <!-- ros2srrc_HMI CAMERA -->
+  <xacro:if value="${hmi}">
+    <xacro:include filename="$(find ros2srrc_hmi)/urdf/hmicamera.urdf.xacro"/>
+    <xacro:HMI_camera
+      x="2.0"
+      y="2.0"
+      z="1.50"
+      roll="0.0"
+      pitch="0.35"
+      yaw="-2.6"
+    />
+  </xacro:if>
 </robot>
