Commit message: R3M use-cases update (14-01-2025).

File: AMRC/r3mcell_amrc_gazebo/urdf/r3mcell_amrc_CK_6640.urdf.xacro (robot description, xacro)
@@ -28,5 +28,5 @@
 # IFRA-Cranfield (2023) ROS 2 Sim-to-Real Robot Control. URL: https://github.com/IFRA-Cranfield/ros2_SimRealRobotControl.
 -->
-<robot name="irb1200" xmlns:xacro="http://ros.org/wiki/xacro">
+<robot name="irb6640" xmlns:xacro="http://ros.org/wiki/xacro">
   <!-- PASS ARGUMENTS: -->
   <xacro:arg name="bringup" default="false"/>
@@ -40,7 +40,7 @@
   <xacro:arg name="EE_name" default="none"/>
   <xacro:property name="EE_name" value="$(arg EE_name)"/>
-  <!-- Include XACRO-MACRO file of the IRB1200: -->
-  <xacro:include filename="$(find ros2srrc_robots)/irb1200/urdf/irb1200_macro.urdf.xacro"/>
-  <xacro:irb1200
+  <!-- Include XACRO-MACRO file of the IRB6640: -->
+  <xacro:include filename="$(find ros2srrc_robots)/irb6640/urdf/irb6640_macro.urdf.xacro"/>
+  <xacro:irb6640
     bringup="${bringup}"
     robot_ip="${robot_ip}"
@@ -48,14 +48,14 @@
     EE_name="${EE_name}"
   />
-  <!-- Include: IRB1200/GPP5010NC ADAPTER -->
+  <!-- Include: IRB6640/GPP5010NC ADAPTER -->
   <link name="adapter">
     <visual>
       <geometry>
-        <mesh filename="file://$(find ros2srrc_endeffectors)/gpp5010nc/meshes/gpp5010nc_irb1200_Adapter.dae" />
+        <mesh filename="file://$(find ros2srrc_endeffectors)/gpp5010nc/meshes/gpp5010nc_irb6640_Adapter.dae" />
       </geometry>
     </visual>
     <collision>
       <geometry>
-        <mesh filename="file://$(find ros2srrc_endeffectors)/gpp5010nc/meshes/gpp5010nc_irb1200_Adapter.dae" />
+        <mesh filename="file://$(find ros2srrc_endeffectors)/gpp5010nc/meshes/gpp5010nc_irb6640_Adapter.dae" />
       </geometry>
     </collision>
@@ -67,14 +67,16 @@
   </link>
   <joint name="adapter_joint" type="fixed">
-    <origin xyz="0.0 0.0 0.0125" rpy="0 1.5708 3.1416" />
+    <origin xyz="0.0 0 0.023" rpy="0 ${pi/2} ${pi}" />
     <parent link="tool0"/>
     <child link="adapter"/>
   </joint>
   <!-- Include XACRO-MACRO file of the GPP5010NC: -->
-  <xacro:include filename="$(find ros2srrc_endeffectors)/gpp5010nc/urdf/gpp5010ncv2_macro.urdf.xacro"/>
-  <xacro:gpp5010nc
-    bringup="${bringup}"
-    parent_link="adapter"
-  />
+  <xacro:if value="${EE}">
+    <xacro:include filename="$(find ros2srrc_endeffectors)/gpp5010nc/urdf/gpp5010ncv2_macro.urdf.xacro"/>
+    <xacro:gpp5010nc
+      bringup="${bringup}"
+      parent_link="adapter"
+    />
+  </xacro:if>
   <!-- Load ROS 2 Gazebo Plugin -->
   <xacro:unless value="${bringup}">
@@ -82,8 +84,10 @@
       <plugin filename="libgazebo_ros2_control.so" name="gazebo_ros2_control">
         <robot_sim_type>gazebo_ros2_control/GazeboSystem</robot_sim_type>
-        <!-- IRB1200 Controller -->
-        <parameters>$(find ros2srrc_robots)/irb1200/config/controller.yaml</parameters>
+        <!-- IRB6640 Controller -->
+        <parameters>$(find ros2srrc_robots)/irb6640/config/controller.yaml</parameters>
         <!-- End-Effector Controller (if needed) -->
-        <parameters>$(find ros2srrc_endeffectors)/${EE_name}/config/controller.yaml</parameters>
+        <xacro:if value="${EE}">
+          <parameters>$(find ros2srrc_endeffectors)/${EE_name}/config/controller.yaml</parameters>
+        </xacro:if>
       </plugin>
     </gazebo>
@@ -96,5 +100,5 @@
       <origin xyz="0.0 0.0 0.0" rpy="0 0 0" />
       <geometry>
-        <mesh filename="file://$(find r3mcell_amrc_gazebo)/meshes/ReconCell/floor_irb1200.dae" scale="1 1 1" />
+        <mesh filename="file://$(find r3mcell_amrc_gazebo)/meshes/ReconCell/floor_irb6640.dae" scale="1 1 1" />
       </geometry>
     </visual>
@@ -102,5 +106,5 @@
       <origin xyz="0.0 0.0 0.0" rpy="0 0 0" />
       <geometry>
-        <mesh filename="file://$(find r3mcell_amrc_gazebo)/meshes/ReconCell/floor_irb1200.dae" scale="1 1 1" />
+        <mesh filename="file://$(find r3mcell_amrc_gazebo)/meshes/ReconCell/floor_irb6640.dae" scale="1 1 1" />
       </geometry>
     </collision>
@@ -110,4 +114,5 @@
     </inertial>
   </link>
+  <!-- FLOOR: FIXED JOINT -->
   <joint name="world-floor-fixed" type="fixed">
     <parent link="world"/>
@@ -115,58 +120,9 @@
     <origin xyz="0.0 0.0 0.0" rpy="0.0 0.0 0.0" />
   </joint>
-  <!-- ReconCell: TallMount -->
-  <link name="TallMount">
-    <visual>
-      <origin xyz="0.0 0.0 0.0" rpy="0 0 0" />
-      <geometry>
-        <mesh filename="file://$(find r3mcell_amrc_gazebo)/meshes/ReconCell/TallMount.dae" scale="1 1 1" />
-      </geometry>
-    </visual>
-    <collision>
-      <origin xyz="0.0 0.0 0.0" rpy="0 0 0" />
-      <geometry>
-        <mesh filename="file://$(find r3mcell_amrc_gazebo)/meshes/ReconCell/TallMount.dae" scale="1 1 1" />
-      </geometry>
-    </collision>
-    <inertial>
-      <mass value="1000.0"/>
-      <inertia ixx="500.0" ixy="500.0" ixz="500.0" iyy="500.0" iyz="500.0" izz="500.0" />
-    </inertial>
-  </link>
-  <joint name="world-TallMount-fixed" type="fixed">
-    <parent link="world"/>
-    <child link="TallMount"/>
-    <origin xyz="0.0 0.0 0.0" rpy="0.0 0.0 0.0" />
-  </joint>
-  <!-- IRB1200 - Adapter Plate -->
-  <link name="adapter_plate">
-    <visual>
-      <origin xyz="0.0 0.0 0.0" rpy="0 0 0" />
-      <geometry>
-        <mesh filename="file://$(find r3mcell_amrc_gazebo)/meshes/ReconCell/irb1200_FloorAdapter.dae" scale="1 1 1" />
-      </geometry>
-    </visual>
-    <collision>
-      <origin xyz="0.0 0.0 0.0" rpy="0 0 0" />
-      <geometry>
-        <mesh filename="file://$(find r3mcell_amrc_gazebo)/meshes/ReconCell/irb1200_FloorAdapter.dae" scale="1 1 1" />
-      </geometry>
-    </collision>
-    <inertial>
-      <mass value="1000.0"/>
-      <inertia ixx="500.0" ixy="500.0" ixz="500.0" iyy="500.0" iyz="500.0" izz="500.0" />
-    </inertial>
-  </link>
-  <!-- Floor+Adapter JOINT -->
-  <joint name="floor-adapter-fixed" type="fixed">
+  <!-- Robot+Floor JOINT -->
+  <joint name="floor-base_link-fixed" type="fixed">
     <parent link="floor"/>
-    <child link="adapter_plate"/>
-    <origin xyz="0.0 0.0 0.0" rpy="0.0 0.0 0.0" />
-  </joint>
-  <!-- Robot+Adapter JOINT -->
-  <joint name="adapter-base_link-fixed" type="fixed">
-    <parent link="adapter_plate"/>
     <child link="base_link"/>
-    <origin xyz="0.0 0.0 0.139" rpy="0.0 0.0 0.0" />
+    <origin xyz="0.0 0.0 0.148" rpy="0.0 0.0 0.0" />
   </joint>
   <!-- ReconCell: WALLS -->
@@ -175,5 +131,5 @@
       <origin xyz="0.0 0.0 0.0" rpy="0 0 0" />
       <geometry>
-        <mesh filename="file://$(find r3mcell_amrc_gazebo)/meshes/ReconCell/walls_1200.dae" scale="1 1 1" />
+        <mesh filename="file://$(find r3mcell_amrc_gazebo)/meshes/ReconCell/walls_6640.dae" scale="1 1 1" />
       </geometry>
     </visual>
@@ -181,5 +137,5 @@
       <origin xyz="0.0 0.0 0.0" rpy="0 0 0" />
       <geometry>
-        <mesh filename="file://$(find r3mcell_amrc_gazebo)/meshes/ReconCell/walls_1200.dae" scale="1 1 1" />
+        <mesh filename="file://$(find r3mcell_amrc_gazebo)/meshes/ReconCell/walls_6640.dae" scale="1 1 1" />
       </geometry>
     </collision>
@@ -218,5 +174,5 @@
     <parent link="floor"/>
     <child link="KittingTray"/>
-    <origin xyz="0.0 0.0 0.0" rpy="0.0 0.0 0.0" />
+    <origin xyz="-0.75 2.9 0.0" rpy="0.0 0.0 0.0" />
   </joint>
   <!-- ros2srrc_HMI CAMERA -->
@@ -224,10 +180,10 @@
     <xacro:include filename="$(find ros2srrc_hmi)/urdf/hmicamera.urdf.xacro"/>
     <xacro:HMI_camera
-      x="2.0"
-      y="1.10"
-      z="1.25"
+      x="3.5"
+      y="3.5"
+      z="2.5"
       roll="0.0"
       pitch="0.35"
-      yaw="-2.6"
+      yaw="-2.5"
     />
   </xacro:if>

File: AMRC/r3mcell_amrc_gazebo/urdf/r3mcell_amrc_CuS_6640.urdf.xacro (robot description, xacro)
@@ -28,5 +28,5 @@
 # IFRA-Cranfield (2023) ROS 2 Sim-to-Real Robot Control. URL: https://github.com/IFRA-Cranfield/ros2_SimRealRobotControl.
 -->
-<robot name="irb1200" xmlns:xacro="http://ros.org/wiki/xacro">
+<robot name="irb6640" xmlns:xacro="http://ros.org/wiki/xacro">
   <!-- PASS ARGUMENTS: -->
   <xacro:arg name="bringup" default="false"/>
@@ -40,7 +40,7 @@
   <xacro:arg name="EE_name" default="none"/>
   <xacro:property name="EE_name" value="$(arg EE_name)"/>
-  <!-- Include XACRO-MACRO file of the IRB1200: -->
-  <xacro:include filename="$(find ros2srrc_robots)/irb1200/urdf/irb1200_macro.urdf.xacro"/>
-  <xacro:irb1200
+  <!-- Include XACRO-MACRO file of the IRB6640: -->
+  <xacro:include filename="$(find ros2srrc_robots)/irb6640/urdf/irb6640_macro.urdf.xacro"/>
+  <xacro:irb6640
     bringup="${bringup}"
     robot_ip="${robot_ip}"
@@ -48,14 +48,14 @@
     EE_name="${EE_name}"
   />
-  <!-- Include: IRB1200/GPP5010NC ADAPTER -->
+  <!-- Include: IRB6640/GPP5010NC ADAPTER -->
   <link name="adapter">
     <visual>
       <geometry>
-        <mesh filename="file://$(find ros2srrc_endeffectors)/gpp5010nc/meshes/gpp5010nc_irb1200_Adapter.dae" />
+        <mesh filename="file://$(find ros2srrc_endeffectors)/gpp5010nc/meshes/gpp5010nc_irb6640_Adapter.dae" />
       </geometry>
     </visual>
     <collision>
       <geometry>
-        <mesh filename="file://$(find ros2srrc_endeffectors)/gpp5010nc/meshes/gpp5010nc_irb1200_Adapter.dae" />
+        <mesh filename="file://$(find ros2srrc_endeffectors)/gpp5010nc/meshes/gpp5010nc_irb6640_Adapter.dae" />
       </geometry>
     </collision>
@@ -67,14 +67,16 @@
   </link>
   <joint name="adapter_joint" type="fixed">
-    <origin xyz="0.0 0.0 0.0125" rpy="0 1.5708 3.1416" />
+    <origin xyz="0.0 0 0.023" rpy="0 ${pi/2} ${pi}" />
     <parent link="tool0"/>
     <child link="adapter"/>
   </joint>
   <!-- Include XACRO-MACRO file of the GPP5010NC: -->
-  <xacro:include filename="$(find ros2srrc_endeffectors)/gpp5010nc/urdf/gpp5010ncv2_macro.urdf.xacro"/>
-  <xacro:gpp5010nc
-    bringup="${bringup}"
-    parent_link="adapter"
-  />
+  <xacro:if value="${EE}">
+    <xacro:include filename="$(find ros2srrc_endeffectors)/gpp5010nc/urdf/gpp5010ncv2_macro.urdf.xacro"/>
+    <xacro:gpp5010nc
+      bringup="${bringup}"
+      parent_link="adapter"
+    />
+  </xacro:if>
   <!-- Load ROS 2 Gazebo Plugin -->
   <xacro:unless value="${bringup}">
@@ -82,8 +84,10 @@
       <plugin filename="libgazebo_ros2_control.so" name="gazebo_ros2_control">
         <robot_sim_type>gazebo_ros2_control/GazeboSystem</robot_sim_type>
-        <!-- IRB1200 Controller -->
-        <parameters>$(find ros2srrc_robots)/irb1200/config/controller.yaml</parameters>
+        <!-- IRB6640 Controller -->
+        <parameters>$(find ros2srrc_robots)/irb6640/config/controller.yaml</parameters>
         <!-- End-Effector Controller (if needed) -->
-        <parameters>$(find ros2srrc_endeffectors)/${EE_name}/config/controller.yaml</parameters>
+        <xacro:if value="${EE}">
+          <parameters>$(find ros2srrc_endeffectors)/${EE_name}/config/controller.yaml</parameters>
+        </xacro:if>
       </plugin>
     </gazebo>
@@ -96,5 +100,5 @@
       <origin xyz="0.0 0.0 0.0" rpy="0 0 0" />
       <geometry>
-        <mesh filename="file://$(find r3mcell_amrc_gazebo)/meshes/ReconCell/floor_irb1200.dae" scale="1 1 1" />
+        <mesh filename="file://$(find r3mcell_amrc_gazebo)/meshes/ReconCell/floor_irb6640.dae" scale="1 1 1" />
       </geometry>
     </visual>
@@ -102,5 +106,5 @@
       <origin xyz="0.0 0.0 0.0" rpy="0 0 0" />
       <geometry>
-        <mesh filename="file://$(find r3mcell_amrc_gazebo)/meshes/ReconCell/floor_irb1200.dae" scale="1 1 1" />
+        <mesh filename="file://$(find r3mcell_amrc_gazebo)/meshes/ReconCell/floor_irb6640.dae" scale="1 1 1" />
       </geometry>
     </collision>
@@ -110,4 +114,5 @@
     </inertial>
   </link>
+  <!-- FLOOR: FIXED JOINT -->
   <joint name="world-floor-fixed" type="fixed">
     <parent link="world"/>
@@ -115,58 +120,9 @@
     <origin xyz="0.0 0.0 0.0" rpy="0.0 0.0 0.0" />
   </joint>
-  <!-- ReconCell: TallMount -->
-  <link name="TallMount">
-    <visual>
-      <origin xyz="0.0 0.0 0.0" rpy="0 0 0" />
-      <geometry>
-        <mesh filename="file://$(find r3mcell_amrc_gazebo)/meshes/ReconCell/TallMount.dae" scale="1 1 1" />
-      </geometry>
-    </visual>
-    <collision>
-      <origin xyz="0.0 0.0 0.0" rpy="0 0 0" />
-      <geometry>
-        <mesh filename="file://$(find r3mcell_amrc_gazebo)/meshes/ReconCell/TallMount.dae" scale="1 1 1" />
-      </geometry>
-    </collision>
-    <inertial>
-      <mass value="1000.0"/>
-      <inertia ixx="500.0" ixy="500.0" ixz="500.0" iyy="500.0" iyz="500.0" izz="500.0" />
-    </inertial>
-  </link>
-  <joint name="world-TallMount-fixed" type="fixed">
-    <parent link="world"/>
-    <child link="TallMount"/>
-    <origin xyz="0.0 0.0 0.0" rpy="0.0 0.0 0.0" />
-  </joint>
-  <!-- IRB1200 - Adapter Plate -->
-  <link name="adapter_plate">
-    <visual>
-      <origin xyz="0.0 0.0 0.0" rpy="0 0 0" />
-      <geometry>
-        <mesh filename="file://$(find r3mcell_amrc_gazebo)/meshes/ReconCell/irb1200_FloorAdapter.dae" scale="1 1 1" />
-      </geometry>
-    </visual>
-    <collision>
-      <origin xyz="0.0 0.0 0.0" rpy="0 0 0" />
-      <geometry>
-        <mesh filename="file://$(find r3mcell_amrc_gazebo)/meshes/ReconCell/irb1200_FloorAdapter.dae" scale="1 1 1" />
-      </geometry>
-    </collision>
-    <inertial>
-      <mass value="1000.0"/>
-      <inertia ixx="500.0" ixy="500.0" ixz="500.0" iyy="500.0" iyz="500.0" izz="500.0" />
-    </inertial>
-  </link>
-  <!-- Floor+Adapter JOINT -->
-  <joint name="floor-adapter-fixed" type="fixed">
+  <!-- Robot+Floor JOINT -->
+  <joint name="floor-base_link-fixed" type="fixed">
     <parent link="floor"/>
-    <child link="adapter_plate"/>
-    <origin xyz="0.0 0.0 0.0" rpy="0.0 0.0 0.0" />
-  </joint>
-  <!-- Robot+Adapter JOINT -->
-  <joint name="adapter-base_link-fixed" type="fixed">
-    <parent link="adapter_plate"/>
     <child link="base_link"/>
-    <origin xyz="0.0 0.0 0.139" rpy="0.0 0.0 0.0" />
+    <origin xyz="0.0 0.0 0.148" rpy="0.0 0.0 0.0" />
   </joint>
   <!-- ReconCell: WALLS -->
@@ -175,5 +131,5 @@
       <origin xyz="0.0 0.0 0.0" rpy="0 0 0" />
       <geometry>
-        <mesh filename="file://$(find r3mcell_amrc_gazebo)/meshes/ReconCell/walls_1200.dae" scale="1 1 1" />
+        <mesh filename="file://$(find r3mcell_amrc_gazebo)/meshes/ReconCell/walls_6640.dae" scale="1 1 1" />
       </geometry>
     </visual>
@@ -181,5 +137,5 @@
       <origin xyz="0.0 0.0 0.0" rpy="0 0 0" />
       <geometry>
-        <mesh filename="file://$(find r3mcell_amrc_gazebo)/meshes/ReconCell/walls_1200.dae" scale="1 1 1" />
+        <mesh filename="file://$(find r3mcell_amrc_gazebo)/meshes/ReconCell/walls_6640.dae" scale="1 1 1" />
       </geometry>
     </collision>
@@ -195,39 +151,14 @@
     <origin xyz="0.0 0.0 0.0" rpy="0.0 0.0 0.0" />
   </joint>
-  <!-- Kitting Tray -->
-  <link name="KittingTray">
-    <visual>
-      <origin xyz="0.0 0.0 0.0" rpy="0 0 0" />
-      <geometry>
-        <mesh filename="file://$(find r3mcell_amrc_gazebo)/meshes/CubeKitting/KittingTray.dae" scale="1 1 1" />
-      </geometry>
-    </visual>
-    <collision>
-      <origin xyz="0.0 0.0 0.0" rpy="0 0 0" />
-      <geometry>
-        <mesh filename="file://$(find r3mcell_amrc_gazebo)/meshes/CubeKitting/KittingTray.dae" scale="1 1 1" />
-      </geometry>
-    </collision>
-    <inertial>
-      <mass value="10.0"/>
-      <inertia ixx="500.0" ixy="500.0" ixz="500.0" iyy="500.0" iyz="500.0" izz="500.0" />
-    </inertial>
-  </link>
-  <!-- Kitting Tray: FIXED JOINT -->
-  <joint name="tray-floor-fixed" type="fixed">
-    <parent link="floor"/>
-    <child link="KittingTray"/>
-    <origin xyz="0.0 0.0 0.0" rpy="0.0 0.0 0.0" />
-  </joint>
   <!-- ros2srrc_HMI CAMERA -->
   <xacro:if value="${hmi}">
     <xacro:include filename="$(find ros2srrc_hmi)/urdf/hmicamera.urdf.xacro"/>
     <xacro:HMI_camera
-      x="2.0"
-      y="1.10"
-      z="1.25"
+      x="3.5"
+      y="3.5"
+      z="2.5"
       roll="0.0"
       pitch="0.35"
-      yaw="-2.6"
+      yaw="-2.5"
     />
   </xacro:if>
