Commit message: Upload: AMRC-BD Use-Case (not ready).

File: AMRC/r3mcell_amrc_gazebo/urdf/r3mcell_amrc_BD.urdf.xacro (robot description, xacro)
@@ -46,4 +46,33 @@
     EE_name="${EE_name}"
   />
+  <!-- Include: IRB6640/GPP5010NC ADAPTER -->
+  <link name="adapter">
+    <visual>
+      <geometry>
+        <mesh filename="file://$(find ros2srrc_endeffectors)/gpp5010nc/meshes/gpp5010nc_irb6640_Adapter.dae" />
+      </geometry>
+    </visual>
+    <collision>
+      <geometry>
+        <mesh filename="file://$(find ros2srrc_endeffectors)/gpp5010nc/meshes/gpp5010nc_irb6640_Adapter.dae" />
+      </geometry>
+    </collision>
+    <inertial>
+      <origin xyz="0 0 0" rpy="0 0 0" />
+      <mass value="0.001" />
+      <inertia ixx="0.001" ixy="0.0" ixz="0.0" iyy="0.001" iyz="0.0" izz="0.001"/>
+    </inertial>
+  </link>
+  <joint name="adapter_joint" type="fixed">
+    <origin xyz="0.0 0 0.023" rpy="0 ${pi/2} ${pi}" />
+    <parent link="tool0"/>
+    <child link="adapter"/>
+  </joint>
+  <!-- Include XACRO-MACRO file of the GPP5010NC: -->
+  <xacro:include filename="$(find ros2srrc_endeffectors)/gpp5010nc/urdf/gpp5010nc_macro.urdf.xacro"/>
+  <xacro:gpp5010nc
+    bringup="${bringup}"
+    parent_link="adapter"
+  />
   <!-- Load ROS 2 Gazebo Plugin -->
   <xacro:unless value="${bringup}">
@@ -53,4 +82,6 @@
         <!-- IRB6640 Controller -->
         <parameters>$(find ros2srrc_robots)/irb6640/config/controller.yaml</parameters>
+        <!-- End-Effector Controller (if needed) -->
+        <parameters>$(find ros2srrc_endeffectors)/${EE_name}/config/controller.yaml</parameters>
       </plugin>
     </gazebo>
@@ -89,3 +120,76 @@
     <origin xyz="0.0 0.0 0.148" rpy="0.0 0.0 0.0" />
   </joint>
+  <!-- BATTERY DISASSEMBLY USE-CASE -->
+  <link name="BD_fixture">
+    <visual>
+      <origin xyz="0.0 0.0 0.0" rpy="0 0 0" />
+      <geometry>
+        <mesh filename="file://$(find r3mcell_amrc_gazebo)/meshes/BatteryDisassembly/BD_Fixture.dae" scale="1 1 1" />
+      </geometry>
+    </visual>
+    <collision>
+      <origin xyz="0.0 0.0 0.0" rpy="0 0 0" />
+      <geometry>
+        <mesh filename="file://$(find r3mcell_amrc_gazebo)/meshes/BatteryDisassembly/BD_Fixture.dae" scale="1 1 1" />
+      </geometry>
+    </collision>
+    <inertial>
+      <mass value="1000.0"/>
+      <inertia ixx="500.0" ixy="500.0" ixz="500.0" iyy="500.0" iyz="500.0" izz="500.0" />
+    </inertial>
+  </link>
+  <joint name="fixture-floor-fixed" type="fixed">
+    <parent link="floor"/>
+    <child link="BD_fixture"/>
+    <origin xyz="0.0 0.0 0.0" rpy="0.0 0.0 0.0" />
+  </joint>
+  <link name="BD_PlasticBin">
+    <visual>
+      <origin xyz="0.0 0.0 0.0" rpy="0 0 0" />
+      <geometry>
+        <mesh filename="file://$(find r3mcell_amrc_gazebo)/meshes/BatteryDisassembly/BD_PlasticBin.dae" scale="1 1 1" />
+      </geometry>
+    </visual>
+    <collision>
+      <origin xyz="0.0 0.0 0.0" rpy="0 0 0" />
+      <geometry>
+        <mesh filename="file://$(find r3mcell_amrc_gazebo)/meshes/BatteryDisassembly/BD_PlasticBin.dae" scale="1 1 1" />
+      </geometry>
+    </collision>
+    <inertial>
+      <mass value="1000.0"/>
+      <inertia ixx="500.0" ixy="500.0" ixz="500.0" iyy="500.0" iyz="500.0" izz="500.0" />
+    </inertial>
+  </link>
+  <joint name="PlasticBin-floor-fixed" type="fixed">
+    <parent link="floor"/>
+    <child link="BD_PlasticBin"/>
+    <origin xyz="0.0 0.0 0.0" rpy="0.0 0.0 0.0" />
+  </joint>
+  <link name="BD_CaseBottom">
+    <visual>
+      <origin xyz="0.0 0.0 0.0" rpy="0 0 0" />
+      <geometry>
+        <mesh filename="file://$(find r3mcell_amrc_gazebo)/meshes/BatteryDisassembly/BD_CaseBottom.dae" scale="1 1 1" />
+      </geometry>
+    </visual>
+    <collision>
+      <origin xyz="0.0 0.0 0.0" rpy="0 0 0" />
+      <geometry>
+        <mesh filename="file://$(find r3mcell_amrc_gazebo)/meshes/BatteryDisassembly/BD_CaseBottom_collisions.dae" scale="1 1 1" />
+      </geometry>
+    </collision>
+    <inertial>
+      <mass value="1000.0"/>
+      <inertia ixx="500.0" ixy="500.0" ixz="500.0" iyy="500.0" iyz="500.0" izz="500.0" />
+    </inertial>
+  </link>
+  <joint name="CaseBottom-floor-fixed" type="fixed">
+    <parent link="floor"/>
+    <child link="BD_CaseBottom"/>
+    <origin xyz="0.0 0.0 0.0" rpy="0.0 0.0 0.0" />
+  </joint>
+  <gazebo reference="BD_CaseBottom">
+    <material>Gazebo/Grey</material>
+  </gazebo>
 </robot>

Commit message: Update: R3M Cell (24-01-2025).

File: AMRC/r3mcell_amrc_gazebo/urdf/r3mcell_amrc_BD.urdf.xacro (robot description, xacro)
@@ -219,51 +219,5 @@
     <parent link="floor"/>
     <child link="BD_CaseBottom"/>
-    <origin xyz="0.0 0.0 0.0" rpy="0.0 0.0 0.0" />
-  </joint>
-  <link name="BD_CaseSideL">
-    <visual>
-      <origin xyz="0.0 0.0 0.0" rpy="0 0 0" />
-      <geometry>
-        <mesh filename="file://$(find r3mcell_amrc_gazebo)/meshes/BatteryDisassembly/BD_CaseSide.dae" scale="1 1 1" />
-      </geometry>
-    </visual>
-    <collision>
-      <origin xyz="0.0 0.0 0.0" rpy="0 0 0" />
-      <geometry>
-        <mesh filename="file://$(find r3mcell_amrc_gazebo)/meshes/BatteryDisassembly/BD_CaseSide.dae" scale="1 1 1" />
-      </geometry>
-    </collision>
-    <inertial>
-      <mass value="1000.0"/>
-      <inertia ixx="500.0" ixy="500.0" ixz="500.0" iyy="500.0" iyz="500.0" izz="500.0" />
-    </inertial>
-  </link>
-  <joint name="CaseSideL-floor-fixed" type="fixed">
-    <parent link="floor"/>
-    <child link="BD_CaseSideL"/>
-    <origin xyz="2.005 0.0315 0.232" rpy="0.0 0.0 0.0" />
-  </joint>
-  <link name="BD_CaseSideR">
-    <visual>
-      <origin xyz="0.0 0.0 0.0" rpy="0 0 0" />
-      <geometry>
-        <mesh filename="file://$(find r3mcell_amrc_gazebo)/meshes/BatteryDisassembly/BD_CaseSide.dae" scale="1 1 1" />
-      </geometry>
-    </visual>
-    <collision>
-      <origin xyz="0.0 0.0 0.0" rpy="0 0 0" />
-      <geometry>
-        <mesh filename="file://$(find r3mcell_amrc_gazebo)/meshes/BatteryDisassembly/BD_CaseSide.dae" scale="1 1 1" />
-      </geometry>
-    </collision>
-    <inertial>
-      <mass value="1000.0"/>
-      <inertia ixx="500.0" ixy="500.0" ixz="500.0" iyy="500.0" iyz="500.0" izz="500.0" />
-    </inertial>
-  </link>
-  <joint name="CaseSideR-floor-fixed" type="fixed">
-    <parent link="floor"/>
-    <child link="BD_CaseSideR"/>
-    <origin xyz="2.255 0.1215 0.232" rpy="0.0 0.0 3.1416" />
+    <origin xyz="0.0 0.0 0.005" rpy="0.0 0.0 0.0" />
   </joint>
   <gazebo reference="BD_CaseBottom">

File: AMRC/r3mcell_amrc_gazebo/urdf/r3mcell_amrc_CyS_1200.urdf.xacro (robot description, xacro)
@@ -72,5 +72,5 @@
   </joint>
   <!-- Include XACRO-MACRO file of the GPP5010NC: -->
-  <xacro:include filename="$(find ros2srrc_endeffectors)/gpp5010nc/urdf/gpp5010nc_macro.urdf.xacro"/>
+  <xacro:include filename="$(find ros2srrc_endeffectors)/gpp5010nc/urdf/gpp5010ncv3_macro.urdf.xacro"/>
   <xacro:gpp5010nc
     bringup="${bringup}"
@@ -193,4 +193,28 @@
     <parent link="world"/>
     <child link="walls"/>
+    <origin xyz="0.0 0.0 0.0" rpy="0.0 0.0 0.0" />
+  </joint>
+  <!-- R3M AMRC Cell: Cylinder Stacking -> Fixture -->
+  <link name="CS_Fixture">
+    <visual>
+      <origin xyz="0.0 0.0 0.0" rpy="0 0 0" />
+      <geometry>
+        <mesh filename="file://$(find r3mcell_amrc_gazebo)/meshes/CylinderStacking/CylinderStacking_Fixture.dae" scale="1 1 1" />
+      </geometry>
+    </visual>
+    <collision>
+      <origin xyz="0.0 0.0 0.0" rpy="0 0 0" />
+      <geometry>
+        <mesh filename="file://$(find r3mcell_amrc_gazebo)/meshes/CylinderStacking/CylinderStacking_Fixture.dae" scale="1 1 1" />
+      </geometry>
+    </collision>
+    <inertial>
+      <mass value="10.0"/>
+      <inertia ixx="0.0002" ixy="0.0002" ixz="0.0002" iyy="0.0" iyz="0.0" izz="0.0" />
+    </inertial>
+  </link>
+  <joint name="floor-CS_Fixture-fixed" type="fixed">
+    <parent link="floor"/>
+    <child link="CS_Fixture"/>
     <origin xyz="0.0 0.0 0.0" rpy="0.0 0.0 0.0" />
   </joint>

File: AMRC/r3mcell_amrc_gazebo/urdf/r3mcell_amrc_CyS_6640.urdf.xacro (robot description, xacro)
@@ -73,5 +73,5 @@
   <!-- Include XACRO-MACRO file of the GPP5010NC: -->
   <xacro:if value="${EE}">
-    <xacro:include filename="$(find ros2srrc_endeffectors)/gpp5010nc/urdf/gpp5010ncv2_macro.urdf.xacro"/>
+    <xacro:include filename="$(find ros2srrc_endeffectors)/gpp5010nc/urdf/gpp5010ncv3_macro.urdf.xacro"/>
     <xacro:gpp5010nc
       bringup="${bringup}"
@@ -151,10 +151,10 @@
     <origin xyz="0.0 0.0 0.0" rpy="0.0 0.0 0.0" />
   </joint>
-  <!-- Kitting Tray -->
-  <link name="KittingTray">
+  <!-- R3M AMRC Cell: Cylinder Stacking -> Fixture -->
+  <link name="CS_Fixture">
     <visual>
       <origin xyz="0.0 0.0 0.0" rpy="0 0 0" />
       <geometry>
-        <mesh filename="file://$(find r3mcell_amrc_gazebo)/meshes/CubeKitting/KittingTray_irb6640.dae" scale="1 1 1" />
+        <mesh filename="file://$(find r3mcell_amrc_gazebo)/meshes/CylinderStacking/CylinderStacking_Fixture_irb6640.dae" scale="1 1 1" />
       </geometry>
     </visual>
@@ -162,16 +162,15 @@
       <origin xyz="0.0 0.0 0.0" rpy="0 0 0" />
       <geometry>
-        <mesh filename="file://$(find r3mcell_amrc_gazebo)/meshes/CubeKitting/KittingTray_irb6640.dae" scale="1 1 1" />
+        <mesh filename="file://$(find r3mcell_amrc_gazebo)/meshes/CylinderStacking/CylinderStacking_Fixture_irb6640.dae" scale="1 1 1" />
       </geometry>
     </collision>
     <inertial>
       <mass value="10.0"/>
-      <inertia ixx="500.0" ixy="500.0" ixz="500.0" iyy="500.0" iyz="500.0" izz="500.0" />
+      <inertia ixx="0.0002" ixy="0.0002" ixz="0.0002" iyy="0.0" iyz="0.0" izz="0.0" />
     </inertial>
   </link>
-  <!-- Kitting Tray: FIXED JOINT -->
-  <joint name="tray-floor-fixed" type="fixed">
+  <joint name="floor-CS_Fixture-fixed" type="fixed">
     <parent link="floor"/>
-    <child link="KittingTray"/>
+    <child link="CS_Fixture"/>
     <origin xyz="0.0 0.0 0.0" rpy="0.0 0.0 0.0" />
   </joint>

File: CranfieldUniversity/r3mcell_cu_gazebo/urdf/r3mcell_cu_CSur.urdf.xacro (robot description, xacro)
@@ -59,5 +59,5 @@
   />
   <!-- Include XACRO-MACRO file of the Robotiq 2f-85: -->
-  <xacro:include filename="$(find ros2srrc_endeffectors)/robotiq_hande/urdf/robotiq_hande_macro.urdf.xacro"/>
+  <xacro:include filename="$(find ros2srrc_endeffectors)/robotiq_hande/urdf/robotiq_handev2_macro.urdf.xacro"/>
   <xacro:robotiq_hande
     bringup="${bringup}"

Commit message: Add collision walls to IRB6640 floor.

File: AMRC/r3mcell_amrc_gazebo/urdf/r3mcell_amrc_BD.urdf.xacro (robot description, xacro)
@@ -106,5 +106,5 @@
       <origin xyz="0.0 0.0 0.0" rpy="0 0 0" />
       <geometry>
-        <mesh filename="file://$(find r3mcell_amrc_gazebo)/meshes/ReconCell/floor_irb6640.dae" scale="1 1 1" />
+        <mesh filename="file://$(find r3mcell_amrc_gazebo)/meshes/ReconCell/floor_irb6640_collision.dae" scale="1 1 1" />
       </geometry>
     </collision>
