Commit message: Update URDF+Config: LamStack (AMRC) VcGripper.

File: AMRC/r3mcell_amrc_gazebo/urdf/r3mcell_amrc_1.urdf.xacro (robot description, xacro)
@@ -63,5 +63,5 @@
       <origin xyz="0.0 0.0 0.0" rpy="0 0 0" />
       <geometry>
-        <mesh filename="file://$(find r3mcell_amrc_gazebo)/meshes/ReconCell/floor_simplified.dae" scale="1 1 1" />
+        <mesh filename="file://$(find r3mcell_amrc_gazebo)/meshes/ReconCell/floor.dae" scale="1 1 1" />
       </geometry>
     </visual>
@@ -69,5 +69,5 @@
       <origin xyz="0.0 0.0 0.0" rpy="0 0 0" />
       <geometry>
-        <mesh filename="file://$(find r3mcell_amrc_gazebo)/meshes/ReconCell/floor_simplified.dae" scale="1 1 1" />
+        <mesh filename="file://$(find r3mcell_amrc_gazebo)/meshes/ReconCell/floor.dae" scale="1 1 1" />
       </geometry>
     </collision>

File: AMRC/r3mcell_amrc_gazebo/urdf/r3mcell_amrc_LamStack.urdf.xacro (robot description, xacro)
@@ -28,5 +28,5 @@
 # IFRA-Cranfield (2023) ROS 2 Sim-to-Real Robot Control. URL: https://github.com/IFRA-Cranfield/ros2_SimRealRobotControl.
 -->
-<robot name="irb6640" xmlns:xacro="http://ros.org/wiki/xacro">
+<robot name="irb1200" xmlns:xacro="http://ros.org/wiki/xacro">
   <!-- PASS ARGUMENTS: -->
   <xacro:arg name="bringup" default="false"/>
@@ -38,11 +38,17 @@
   <xacro:arg name="EE_name" default="none"/>
   <xacro:property name="EE_name" value="$(arg EE_name)"/>
-  <!-- Include XACRO-MACRO file of the IRB6640: -->
-  <xacro:include filename="$(find ros2srrc_robots)/irb6640/urdf/irb6640_macro.urdf.xacro"/>
-  <xacro:irb6640
+  <!-- Include XACRO-MACRO file of the IRB1200: -->
+  <xacro:include filename="$(find ros2srrc_robots)/irb1200/urdf/irb1200_macro.urdf.xacro"/>
+  <xacro:irb1200
     bringup="${bringup}"
     robot_ip="${robot_ip}"
     EE="${EE}"
     EE_name="${EE_name}"
+  />
+  <!-- Include XACRO-MACRO file of the LS-VGR: -->
+  <xacro:include filename="$(find ros2srrc_endeffectors)/ls_vgr_amrc/urdf/ls_vgr_amrc_macro.urdf.xacro"/>
+  <xacro:ls_vgr_amrc
+    bringup="${bringup}"
+    parent_link="tool0"
   />
   <!-- Load ROS 2 Gazebo Plugin -->
@@ -51,6 +57,6 @@
       <plugin filename="libgazebo_ros2_control.so" name="gazebo_ros2_control">
         <robot_sim_type>gazebo_ros2_control/GazeboSystem</robot_sim_type>
-        <!-- IRB6640 Controller -->
-        <parameters>$(find ros2srrc_robots)/irb6640/config/controller.yaml</parameters>
+        <!-- IRB1200 Controller -->
+        <parameters>$(find ros2srrc_robots)/irb1200/config/controller.yaml</parameters>
       </plugin>
     </gazebo>
@@ -77,4 +83,23 @@
     </inertial>
   </link>
+  <!-- IRB1200 - Adapter Plate -->
+  <link name="adapter_plate">
+    <visual>
+      <origin xyz="0.0 0.0 0.0" rpy="0 0 0" />
+      <geometry>
+        <mesh filename="file://$(find r3mcell_amrc_gazebo)/meshes/ReconCell/irb1200_FloorAdapter.dae" scale="1 1 1" />
+      </geometry>
+    </visual>
+    <collision>
+      <origin xyz="0.0 0.0 0.0" rpy="0 0 0" />
+      <geometry>
+        <mesh filename="file://$(find r3mcell_amrc_gazebo)/meshes/ReconCell/irb1200_FloorAdapter.dae" scale="1 1 1" />
+      </geometry>
+    </collision>
+    <inertial>
+      <mass value="1000.0"/>
+      <inertia ixx="500.0" ixy="500.0" ixz="500.0" iyy="500.0" iyz="500.0" izz="500.0" />
+    </inertial>
+  </link>
   <!-- FLOOR: FIXED JOINT -->
   <joint name="world-floor-fixed" type="fixed">
@@ -83,9 +108,15 @@
     <origin xyz="0.0 0.0 0.0" rpy="0.0 0.0 0.0" />
   </joint>
-  <!-- Robot+Floor JOINT -->
-  <joint name="floor-base_link-fixed" type="fixed">
+  <!-- Floor+Adapter JOINT -->
+  <joint name="floor-adapter-fixed" type="fixed">
     <parent link="floor"/>
+    <child link="adapter_plate"/>
+    <origin xyz="0.0 0.0 0.0" rpy="0.0 0.0 0.0" />
+  </joint>
+  <!-- Robot+Adapter JOINT -->
+  <joint name="adapter-base_link-fixed" type="fixed">
+    <parent link="adapter_plate"/>
     <child link="base_link"/>
-    <origin xyz="1.65 0.65 0.148" rpy="0.0 0.0 0.0" />
+    <origin xyz="2.55 4.4 0.139" rpy="0.0 0.0 -1.571" />
   </joint>
 </robot>

Commit message: Update: AMRC ReconCell CAD.

File: AMRC/r3mcell_amrc_gazebo/urdf/r3mcell_amrc_1.urdf.xacro (robot description, xacro)
@@ -63,5 +63,5 @@
       <origin xyz="0.0 0.0 0.0" rpy="0 0 0" />
       <geometry>
-        <mesh filename="file://$(find r3mcell_amrc_gazebo)/meshes/ReconCell/floor.dae" scale="1 1 1" />
+        <mesh filename="file://$(find r3mcell_amrc_gazebo)/meshes/ReconCell/floor_irb1200.dae" scale="1 1 1" />
       </geometry>
     </visual>
@@ -69,5 +69,5 @@
       <origin xyz="0.0 0.0 0.0" rpy="0 0 0" />
       <geometry>
-        <mesh filename="file://$(find r3mcell_amrc_gazebo)/meshes/ReconCell/floor.dae" scale="1 1 1" />
+        <mesh filename="file://$(find r3mcell_amrc_gazebo)/meshes/ReconCell/floor_irb1200.dae" scale="1 1 1" />
       </geometry>
     </collision>
@@ -77,4 +77,9 @@
     </inertial>
   </link>
+  <joint name="world-floor-fixed" type="fixed">
+    <parent link="world"/>
+    <child link="floor"/>
+    <origin xyz="0.0 0.0 0.0" rpy="0.0 0.0 0.0" />
+  </joint>
   <!-- IRB1200 - Adapter Plate -->
   <link name="adapter_plate">
@@ -96,10 +101,4 @@
     </inertial>
   </link>
-  <!-- FLOOR: FIXED JOINT -->
-  <joint name="world-floor-fixed" type="fixed">
-    <parent link="world"/>
-    <child link="floor"/>
-    <origin xyz="0.0 0.0 0.0" rpy="0.0 0.0 0.0" />
-  </joint>
   <!-- Floor+Adapter JOINT -->
   <joint name="floor-adapter-fixed" type="fixed">
@@ -112,5 +111,30 @@
     <parent link="adapter_plate"/>
     <child link="base_link"/>
-    <origin xyz="2.55 4.4 0.139" rpy="0.0 0.0 -1.571" />
+    <origin xyz="0.0 0.0 0.139" rpy="0.0 0.0 0.0" />
+  </joint>
+  <!-- ReconCell: WALLS -->
+  <link name="walls">
+    <visual>
+      <origin xyz="0.0 0.0 0.0" rpy="0 0 0" />
+      <geometry>
+        <mesh filename="file://$(find r3mcell_amrc_gazebo)/meshes/ReconCell/walls_1200.dae" scale="1 1 1" />
+      </geometry>
+    </visual>
+    <collision>
+      <origin xyz="0.0 0.0 0.0" rpy="0 0 0" />
+      <geometry>
+        <mesh filename="file://$(find r3mcell_amrc_gazebo)/meshes/ReconCell/walls_1200.dae" scale="1 1 1" />
+      </geometry>
+    </collision>
+    <inertial>
+      <mass value="1000.0"/>
+      <inertia ixx="500.0" ixy="500.0" ixz="500.0" iyy="500.0" iyz="500.0" izz="500.0" />
+    </inertial>
+  </link>
+  <!-- WALLS: FIXED JOINT -->
+  <joint name="world-walls-fixed" type="fixed">
+    <parent link="world"/>
+    <child link="walls"/>
+    <origin xyz="0.0 0.0 0.0" rpy="0.0 0.0 0.0" />
   </joint>
 </robot>

File: AMRC/r3mcell_amrc_gazebo/urdf/r3mcell_amrc_2.urdf.xacro (robot description, xacro)
@@ -89,3 +89,28 @@
     <origin xyz="0.0 0.0 0.148" rpy="0.0 0.0 0.0" />
   </joint>
+  <!-- ReconCell: WALLS -->
+  <link name="walls">
+    <visual>
+      <origin xyz="0.0 0.0 0.0" rpy="0 0 0" />
+      <geometry>
+        <mesh filename="file://$(find r3mcell_amrc_gazebo)/meshes/ReconCell/walls_6640.dae" scale="1 1 1" />
+      </geometry>
+    </visual>
+    <collision>
+      <origin xyz="0.0 0.0 0.0" rpy="0 0 0" />
+      <geometry>
+        <mesh filename="file://$(find r3mcell_amrc_gazebo)/meshes/ReconCell/walls_6640.dae" scale="1 1 1" />
+      </geometry>
+    </collision>
+    <inertial>
+      <mass value="1000.0"/>
+      <inertia ixx="500.0" ixy="500.0" ixz="500.0" iyy="500.0" iyz="500.0" izz="500.0" />
+    </inertial>
+  </link>
+  <!-- WALLS: FIXED JOINT -->
+  <joint name="world-walls-fixed" type="fixed">
+    <parent link="world"/>
+    <child link="walls"/>
+    <origin xyz="0.0 0.0 0.0" rpy="0.0 0.0 0.0" />
+  </joint>
 </robot>

File: AMRC/r3mcell_amrc_gazebo/urdf/r3mcell_amrc_BD.urdf.xacro (robot description, xacro)
@@ -120,4 +120,29 @@
     <origin xyz="0.0 0.0 0.148" rpy="0.0 0.0 0.0" />
   </joint>
+  <!-- ReconCell: WALLS -->
+  <link name="walls">
+    <visual>
+      <origin xyz="0.0 0.0 0.0" rpy="0 0 0" />
+      <geometry>
+        <mesh filename="file://$(find r3mcell_amrc_gazebo)/meshes/ReconCell/walls_6640.dae" scale="1 1 1" />
+      </geometry>
+    </visual>
+    <collision>
+      <origin xyz="0.0 0.0 0.0" rpy="0 0 0" />
+      <geometry>
+        <mesh filename="file://$(find r3mcell_amrc_gazebo)/meshes/ReconCell/walls_6640.dae" scale="1 1 1" />
+      </geometry>
+    </collision>
+    <inertial>
+      <mass value="1000.0"/>
+      <inertia ixx="500.0" ixy="500.0" ixz="500.0" iyy="500.0" iyz="500.0" izz="500.0" />
+    </inertial>
+  </link>
+  <!-- WALLS: FIXED JOINT -->
+  <joint name="world-walls-fixed" type="fixed">
+    <parent link="world"/>
+    <child link="walls"/>
+    <origin xyz="0.0 0.0 0.0" rpy="0.0 0.0 0.0" />
+  </joint>
   <!-- BATTERY DISASSEMBLY USE-CASE -->
   <link name="BD_fixture">
@@ -189,7 +214,59 @@
     <child link="BD_CaseBottom"/>
     <origin xyz="0.0 0.0 0.0" rpy="0.0 0.0 0.0" />
+  </joint>
+  <link name="BD_CaseSideL">
+    <visual>
+      <origin xyz="0.0 0.0 0.0" rpy="0 0 0" />
+      <geometry>
+        <mesh filename="file://$(find r3mcell_amrc_gazebo)/meshes/BatteryDisassembly/BD_CaseSide.dae" scale="1 1 1" />
+      </geometry>
+    </visual>
+    <collision>
+      <origin xyz="0.0 0.0 0.0" rpy="0 0 0" />
+      <geometry>
+        <mesh filename="file://$(find r3mcell_amrc_gazebo)/meshes/BatteryDisassembly/BD_CaseSide.dae" scale="1 1 1" />
+      </geometry>
+    </collision>
+    <inertial>
+      <mass value="1000.0"/>
+      <inertia ixx="500.0" ixy="500.0" ixz="500.0" iyy="500.0" iyz="500.0" izz="500.0" />
+    </inertial>
+  </link>
+  <joint name="CaseSideL-floor-fixed" type="fixed">
+    <parent link="floor"/>
+    <child link="BD_CaseSideL"/>
+    <origin xyz="2.005 0.0315 0.232" rpy="0.0 0.0 0.0" />
+  </joint>
+  <link name="BD_CaseSideR">
+    <visual>
+      <origin xyz="0.0 0.0 0.0" rpy="0 0 0" />
+      <geometry>
+        <mesh filename="file://$(find r3mcell_amrc_gazebo)/meshes/BatteryDisassembly/BD_CaseSide.dae" scale="1 1 1" />
+      </geometry>
+    </visual>
+    <collision>
+      <origin xyz="0.0 0.0 0.0" rpy="0 0 0" />
+      <geometry>
+        <mesh filename="file://$(find r3mcell_amrc_gazebo)/meshes/BatteryDisassembly/BD_CaseSide.dae" scale="1 1 1" />
+      </geometry>
+    </collision>
+    <inertial>
+      <mass value="1000.0"/>
+      <inertia ixx="500.0" ixy="500.0" ixz="500.0" iyy="500.0" iyz="500.0" izz="500.0" />
+    </inertial>
+  </link>
+  <joint name="CaseSideR-floor-fixed" type="fixed">
+    <parent link="floor"/>
+    <child link="BD_CaseSideR"/>
+    <origin xyz="2.255 0.1215 0.232" rpy="0.0 0.0 3.1416" />
   </joint>
   <gazebo reference="BD_CaseBottom">
     <material>Gazebo/Grey</material>
   </gazebo>
+  <gazebo reference="BD_CaseSideL">
+    <material>Gazebo/Grey</material>
+  </gazebo>
+  <gazebo reference="BD_CaseSideR">
+    <material>Gazebo/Grey</material>
+  </gazebo>
 </robot>

File: AMRC/r3mcell_amrc_gazebo/urdf/r3mcell_amrc_LamStack.urdf.xacro (robot description, xacro)
@@ -88,4 +88,29 @@
     <origin xyz="0.0 0.0 0.0" rpy="0.0 0.0 0.0" />
   </joint>
+  <!-- ReconCell: WALLS -->
+  <link name="walls">
+    <visual>
+      <origin xyz="0.0 0.0 0.0" rpy="0 0 0" />
+      <geometry>
+        <mesh filename="file://$(find r3mcell_amrc_gazebo)/meshes/ReconCell/walls_1200.dae" scale="1 1 1" />
+      </geometry>
+    </visual>
+    <collision>
+      <origin xyz="0.0 0.0 0.0" rpy="0 0 0" />
+      <geometry>
+        <mesh filename="file://$(find r3mcell_amrc_gazebo)/meshes/ReconCell/walls_1200.dae" scale="1 1 1" />
+      </geometry>
+    </collision>
+    <inertial>
+      <mass value="1000.0"/>
+      <inertia ixx="500.0" ixy="500.0" ixz="500.0" iyy="500.0" iyz="500.0" izz="500.0" />
+    </inertial>
+  </link>
+  <!-- WALLS: FIXED JOINT -->
+  <joint name="world-walls-fixed" type="fixed">
+    <parent link="world"/>
+    <child link="walls"/>
+    <origin xyz="0.0 0.0 0.0" rpy="0.0 0.0 0.0" />
+  </joint>
   <!-- IRB1200 - Adapter Plate -->
   <link name="adapter_plate">

Commit message: Add TallMount to AMRC Cell (all IRB1200-related urdfs).

File: AMRC/r3mcell_amrc_gazebo/urdf/r3mcell_amrc_1.urdf.xacro (robot description, xacro)
@@ -82,4 +82,28 @@
     <origin xyz="0.0 0.0 0.0" rpy="0.0 0.0 0.0" />
   </joint>
+  <!-- ReconCell: TallMount -->
+  <link name="TallMount">
+    <visual>
+      <origin xyz="0.0 0.0 0.0" rpy="0 0 0" />
+      <geometry>
+        <mesh filename="file://$(find r3mcell_amrc_gazebo)/meshes/ReconCell/TallMount.dae" scale="1 1 1" />
+      </geometry>
+    </visual>
+    <collision>
+      <origin xyz="0.0 0.0 0.0" rpy="0 0 0" />
+      <geometry>
+        <mesh filename="file://$(find r3mcell_amrc_gazebo)/meshes/ReconCell/TallMount.dae" scale="1 1 1" />
+      </geometry>
+    </collision>
+    <inertial>
+      <mass value="1000.0"/>
+      <inertia ixx="500.0" ixy="500.0" ixz="500.0" iyy="500.0" iyz="500.0" izz="500.0" />
+    </inertial>
+  </link>
+  <joint name="world-TallMount-fixed" type="fixed">
+    <parent link="world"/>
+    <child link="TallMount"/>
+    <origin xyz="0.0 0.0 0.0" rpy="0.0 0.0 0.0" />
+  </joint>
   <!-- IRB1200 - Adapter Plate -->
   <link name="adapter_plate">

File: AMRC/r3mcell_amrc_gazebo/urdf/r3mcell_amrc_LamStack.urdf.xacro (robot description, xacro)
@@ -88,4 +88,28 @@
     <origin xyz="0.0 0.0 0.0" rpy="0.0 0.0 0.0" />
   </joint>
+  <!-- ReconCell: TallMount -->
+  <link name="TallMount">
+    <visual>
+      <origin xyz="0.0 0.0 0.0" rpy="0 0 0" />
+      <geometry>
+        <mesh filename="file://$(find r3mcell_amrc_gazebo)/meshes/ReconCell/TallMount.dae" scale="1 1 1" />
+      </geometry>
+    </visual>
+    <collision>
+      <origin xyz="0.0 0.0 0.0" rpy="0 0 0" />
+      <geometry>
+        <mesh filename="file://$(find r3mcell_amrc_gazebo)/meshes/ReconCell/TallMount.dae" scale="1 1 1" />
+      </geometry>
+    </collision>
+    <inertial>
+      <mass value="1000.0"/>
+      <inertia ixx="500.0" ixy="500.0" ixz="500.0" iyy="500.0" iyz="500.0" izz="500.0" />
+    </inertial>
+  </link>
+  <joint name="world-TallMount-fixed" type="fixed">
+    <parent link="world"/>
+    <child link="TallMount"/>
+    <origin xyz="0.0 0.0 0.0" rpy="0.0 0.0 0.0" />
+  </joint>
   <!-- ReconCell: WALLS -->
   <link name="walls">

Commit message: R3M-Cell update (AMRC, 05-02-2025).

File: AMRC/r3mcell_amrc_gazebo/urdf/r3mcell_amrc_1.urdf.xacro (robot description, xacro)
@@ -71,5 +71,5 @@
       <origin xyz="0.0 0.0 0.0" rpy="0 0 0" />
       <geometry>
-        <mesh filename="file://$(find r3mcell_amrc_gazebo)/meshes/ReconCell/floor_irb1200.dae" scale="1 1 1" />
+        <mesh filename="file://$(find r3mcell_amrc_gazebo)/meshes/ReconCell/floor_irb1200_collision.dae" scale="1 1 1" />
       </geometry>
     </collision>

File: AMRC/r3mcell_amrc_gazebo/urdf/r3mcell_amrc_2.urdf.xacro (robot description, xacro)
@@ -48,4 +48,28 @@
     EE_name="${EE_name}"
   />
+  <!-- Include Link6's extension (CABLE HOLDER): -->
+  <link name="link_6_ext">
+    <visual>
+      <origin xyz="0.0 0.0 0.0" rpy="0 0 0" />
+      <geometry>
+        <mesh filename="file://$(find r3mcell_amrc_gazebo)/meshes/ReconCell/irb6640_AMRC_link6.dae" scale="1 1 1" />
+      </geometry>
+    </visual>
+    <collision>
+      <origin xyz="0.0 0.0 0.0" rpy="0 0 0" />
+      <geometry>
+        <mesh filename="file://$(find r3mcell_amrc_gazebo)/meshes/ReconCell/irb6640_AMRC_link6.dae" scale="1 1 1" />
+      </geometry>
+    </collision>
+    <inertial>
+      <mass value="10.0"/>
+      <inertia ixx="500.0" ixy="500.0" ixz="500.0" iyy="500.0" iyz="500.0" izz="500.0" />
+    </inertial>
+  </link>
+  <joint name="link6_ext_fixedjoint" type="fixed">
+    <parent link="link_6"/>
+    <child link="link_6_ext"/>
+    <origin xyz="0.0 0.0 0.0" rpy="0.0 0.0 0.0" />
+  </joint>
   <!-- Load ROS 2 Gazebo Plugin -->
   <xacro:unless value="${bringup}">

File: AMRC/r3mcell_amrc_gazebo/urdf/r3mcell_amrc_BD.urdf.xacro (robot description, xacro)
@@ -79,4 +79,28 @@
     />
   </xacro:if>
+  <!-- Include Link6's extension (CABLE HOLDER): -->
+  <link name="link_6_ext">
+    <visual>
+      <origin xyz="0.0 0.0 0.0" rpy="0 0 0" />
+      <geometry>
+        <mesh filename="file://$(find r3mcell_amrc_gazebo)/meshes/ReconCell/irb6640_AMRC_link6.dae" scale="1 1 1" />
+      </geometry>
+    </visual>
+    <collision>
+      <origin xyz="0.0 0.0 0.0" rpy="0 0 0" />
+      <geometry>
+        <mesh filename="file://$(find r3mcell_amrc_gazebo)/meshes/ReconCell/irb6640_AMRC_link6.dae" scale="1 1 1" />
+      </geometry>
+    </collision>
+    <inertial>
+      <mass value="10.0"/>
+      <inertia ixx="500.0" ixy="500.0" ixz="500.0" iyy="500.0" iyz="500.0" izz="500.0" />
+    </inertial>
+  </link>
+  <joint name="link6_ext_fixedjoint" type="fixed">
+    <parent link="link_6"/>
+    <child link="link_6_ext"/>
+    <origin xyz="0.0 0.0 0.0" rpy="0.0 0.0 0.0" />
+  </joint>
   <!-- Load ROS 2 Gazebo Plugin -->
   <xacro:unless value="${bringup}">

File: AMRC/r3mcell_amrc_gazebo/urdf/r3mcell_amrc_CK_1200.urdf.xacro (robot description, xacro)
@@ -102,5 +102,5 @@
       <origin xyz="0.0 0.0 0.0" rpy="0 0 0" />
       <geometry>
-        <mesh filename="file://$(find r3mcell_amrc_gazebo)/meshes/ReconCell/floor_irb1200.dae" scale="1 1 1" />
+        <mesh filename="file://$(find r3mcell_amrc_gazebo)/meshes/ReconCell/floor_irb1200_collision.dae" scale="1 1 1" />
       </geometry>
     </collision>

File: AMRC/r3mcell_amrc_gazebo/urdf/r3mcell_amrc_CK_6640.urdf.xacro (robot description, xacro)
@@ -48,4 +48,28 @@
     EE_name="${EE_name}"
   />
+  <!-- Include Link6's extension (CABLE HOLDER): -->
+  <link name="link_6_ext">
+    <visual>
+      <origin xyz="0.0 0.0 0.0" rpy="0 0 0" />
+      <geometry>
+        <mesh filename="file://$(find r3mcell_amrc_gazebo)/meshes/ReconCell/irb6640_AMRC_link6.dae" scale="1 1 1" />
+      </geometry>
+    </visual>
+    <collision>
+      <origin xyz="0.0 0.0 0.0" rpy="0 0 0" />
+      <geometry>
+        <mesh filename="file://$(find r3mcell_amrc_gazebo)/meshes/ReconCell/irb6640_AMRC_link6.dae" scale="1 1 1" />
+      </geometry>
+    </collision>
+    <inertial>
+      <mass value="10.0"/>
+      <inertia ixx="500.0" ixy="500.0" ixz="500.0" iyy="500.0" iyz="500.0" izz="500.0" />
+    </inertial>
+  </link>
+  <joint name="link6_ext_fixedjoint" type="fixed">
+    <parent link="link_6"/>
+    <child link="link_6_ext"/>
+    <origin xyz="0.0 0.0 0.0" rpy="0.0 0.0 0.0" />
+  </joint>
   <!-- Include: IRB6640/GPP5010NC ADAPTER -->
   <link name="adapter">

File: AMRC/r3mcell_amrc_gazebo/urdf/r3mcell_amrc_CuS_1200.urdf.xacro (robot description, xacro)
@@ -102,5 +102,5 @@
       <origin xyz="0.0 0.0 0.0" rpy="0 0 0" />
       <geometry>
-        <mesh filename="file://$(find r3mcell_amrc_gazebo)/meshes/ReconCell/floor_irb1200.dae" scale="1 1 1" />
+        <mesh filename="file://$(find r3mcell_amrc_gazebo)/meshes/ReconCell/floor_irb1200_collision.dae" scale="1 1 1" />
       </geometry>
     </collision>

File: AMRC/r3mcell_amrc_gazebo/urdf/r3mcell_amrc_CuS_6640.urdf.xacro (robot description, xacro)
@@ -48,4 +48,28 @@
     EE_name="${EE_name}"
   />
+  <!-- Include Link6's extension (CABLE HOLDER): -->
+  <link name="link_6_ext">
+    <visual>
+      <origin xyz="0.0 0.0 0.0" rpy="0 0 0" />
+      <geometry>
+        <mesh filename="file://$(find r3mcell_amrc_gazebo)/meshes/ReconCell/irb6640_AMRC_link6.dae" scale="1 1 1" />
+      </geometry>
+    </visual>
+    <collision>
+      <origin xyz="0.0 0.0 0.0" rpy="0 0 0" />
+      <geometry>
+        <mesh filename="file://$(find r3mcell_amrc_gazebo)/meshes/ReconCell/irb6640_AMRC_link6.dae" scale="1 1 1" />
+      </geometry>
+    </collision>
+    <inertial>
+      <mass value="10.0"/>
+      <inertia ixx="500.0" ixy="500.0" ixz="500.0" iyy="500.0" iyz="500.0" izz="500.0" />
+    </inertial>
+  </link>
+  <joint name="link6_ext_fixedjoint" type="fixed">
+    <parent link="link_6"/>
+    <child link="link_6_ext"/>
+    <origin xyz="0.0 0.0 0.0" rpy="0.0 0.0 0.0" />
+  </joint>
   <!-- Include: IRB6640/GPP5010NC ADAPTER -->
   <link name="adapter">

File: AMRC/r3mcell_amrc_gazebo/urdf/r3mcell_amrc_CyS_1200.urdf.xacro (robot description, xacro)
@@ -102,5 +102,5 @@
       <origin xyz="0.0 0.0 0.0" rpy="0 0 0" />
       <geometry>
-        <mesh filename="file://$(find r3mcell_amrc_gazebo)/meshes/ReconCell/floor_irb1200.dae" scale="1 1 1" />
+        <mesh filename="file://$(find r3mcell_amrc_gazebo)/meshes/ReconCell/floor_irb1200_collision.dae" scale="1 1 1" />
       </geometry>
     </collision>

File: AMRC/r3mcell_amrc_gazebo/urdf/r3mcell_amrc_CyS_6640.urdf.xacro (robot description, xacro)
@@ -48,4 +48,28 @@
     EE_name="${EE_name}"
   />
+  <!-- Include Link6's extension (CABLE HOLDER): -->
+  <link name="link_6_ext">
+    <visual>
+      <origin xyz="0.0 0.0 0.0" rpy="0 0 0" />
+      <geometry>
+        <mesh filename="file://$(find r3mcell_amrc_gazebo)/meshes/ReconCell/irb6640_AMRC_link6.dae" scale="1 1 1" />
+      </geometry>
+    </visual>
+    <collision>
+      <origin xyz="0.0 0.0 0.0" rpy="0 0 0" />
+      <geometry>
+        <mesh filename="file://$(find r3mcell_amrc_gazebo)/meshes/ReconCell/irb6640_AMRC_link6.dae" scale="1 1 1" />
+      </geometry>
+    </collision>
+    <inertial>
+      <mass value="10.0"/>
+      <inertia ixx="500.0" ixy="500.0" ixz="500.0" iyy="500.0" iyz="500.0" izz="500.0" />
+    </inertial>
+  </link>
+  <joint name="link6_ext_fixedjoint" type="fixed">
+    <parent link="link_6"/>
+    <child link="link_6_ext"/>
+    <origin xyz="0.0 0.0 0.0" rpy="0.0 0.0 0.0" />
+  </joint>
   <!-- Include: IRB6640/GPP5010NC ADAPTER -->
   <link name="adapter">

File: AMRC/r3mcell_amrc_gazebo/urdf/r3mcell_amrc_LamStack.urdf.xacro (robot description, xacro)
@@ -77,5 +77,5 @@
       <origin xyz="0.0 0.0 0.0" rpy="0 0 0" />
       <geometry>
-        <mesh filename="file://$(find r3mcell_amrc_gazebo)/meshes/ReconCell/floor_irb1200.dae" scale="1 1 1" />
+        <mesh filename="file://$(find r3mcell_amrc_gazebo)/meshes/ReconCell/floor_irb1200_collision.dae" scale="1 1 1" />
       </geometry>
     </collision>
