Commit message: Adapt: IRB1200 set-up for r3mcell_amrc_12 use-case.

File: AMRC/r3mcell_amrc_gazebo/urdf/r3mcell_amrc_CK_1200.urdf.xacro (robot description, xacro)
@@ -220,4 +220,34 @@
     <origin xyz="0.0 0.0 0.0" rpy="0.0 0.0 0.0" />
   </joint>
+  <!-- ARUCO TAG -->
+  <xacro:unless value="${bringup}">
+    <!-- ARUCO GRID -->
+    <link name="aruco_grid">
+      <visual>
+        <origin xyz="0.0 0.0 0.0" rpy="0 0 0" />
+        <geometry>
+          <mesh filename="file://$(find r3mcell_amrc_gazebo)/meshes/aruco/arucoGrid_irb1200.dae" scale="1 1 1" />
+        </geometry>
+      </visual>
+      <collision>
+        <origin xyz="0.0 0.0 0.0" rpy="0 0 0" />
+        <geometry>
+          <mesh filename="file://$(find r3mcell_amrc_gazebo)/meshes/aruco/arucoGrid_irb1200.dae" scale="1 1 1" />
+        </geometry>
+      </collision>
+      <inertial>
+        <mass value="10.0"/>
+        <inertia ixx="0.0002" ixy="0.0002" ixz="0.0002" iyy="0.0" iyz="0.0" izz="0.0" />
+      </inertial>
+    </link>
+    <joint name="floor-aruco_grid-fixed" type="fixed">
+      <parent link="floor"/>
+      <child link="aruco_grid"/>
+      <origin xyz="0.0 0.0 0.0" rpy="0.0 0.0 0.0" />
+    </joint>
+    <gazebo reference="floor-aruco_grid-fixed">
+      <preserveFixedJoint>true</preserveFixedJoint>
+    </gazebo>
+  </xacro:unless>
   <!-- ros2srrc_HMI CAMERA -->
   <xacro:if value="${hmi}">

Commit message: Adapt R3M Cell (AMRC-IRB1200) to use-cases.

File: AMRC/r3mcell_amrc_gazebo/urdf/r3mcell_amrc_CK_1200.urdf.xacro (robot description, xacro)
@@ -262,3 +262,62 @@
     />
   </xacro:if>
+  <!-- CAMERA -->
+  <xacro:unless value="${bringup}">
+    <link name="camera_link">
+      <collision>
+        <origin xyz="0 0 0" rpy="0 0 0"/>
+        <geometry>
+          <box size="0.05 0.05 0.05"/>
+        </geometry>
+      </collision>
+      <visual>
+        <origin xyz="0 0 0" rpy="0 0 0"/>
+        <geometry>
+          <box size="0.05 0.05 0.05"/>
+        </geometry>
+      </visual>
+      <inertial>
+        <mass value="1.0" />
+        <origin xyz="0 0 0" rpy="0 0 0"/>
+        <inertia ixx="0.0" ixy="0.0" ixz="0.0" iyy="0.0" iyz="0.0" izz="0.0" />
+      </inertial>
+    </link>
+    <joint name="camera_joint" type="fixed">
+      <origin xyz="1.60 0.10 1.20" rpy="0 0.95 3.1416"/>
+      <parent link="world"/>
+      <child link="camera_link"/>
+    </joint>
+    <gazebo reference="camera_link">
+      <sensor name="camera" type="camera">
+        <update_rate>30</update_rate>
+        <camera name="head">
+          <horizontal_fov>1.22</horizontal_fov>
+          <image>
+            <width>1920</width>
+            <height>1080</height>
+            <format>R8G8B8</format>
+          </image>
+          <clip>
+            <near>0.02</near>
+            <far>300</far>
+          </clip>
+          <noise>
+            <type>gaussian</type>
+            <mean>0.0</mean>
+            <stddev>0.007</stddev>
+          </noise>
+        </camera>
+        <plugin filename="libgazebo_ros_camera.so" name="camera_controller">
+          <robotNamespace/>
+          <alwaysOn>true</alwaysOn>
+          <updateRate>0.0</updateRate>
+          <cameraName>camera</cameraName>
+          <imageTopicName>image_raw</imageTopicName>
+          <cameraInfoTopicName>camera_info</cameraInfoTopicName>
+          <frameName>camera</frameName>
+          <hackBaseline>0.07</hackBaseline>
+        </plugin>
+      </sensor>
+    </gazebo>
+  </xacro:unless>
 </robot>

File: AMRC/r3mcell_amrc_gazebo/urdf/r3mcell_amrc_CuS_1200.urdf.xacro (robot description, xacro)
@@ -195,4 +195,34 @@
     <origin xyz="0.0 0.0 0.0" rpy="0.0 0.0 0.0" />
   </joint>
+  <!-- ARUCO TAG -->
+  <xacro:unless value="${bringup}">
+    <!-- ARUCO GRID -->
+    <link name="aruco_grid">
+      <visual>
+        <origin xyz="0.0 0.0 0.0" rpy="0 0 0" />
+        <geometry>
+          <mesh filename="file://$(find r3mcell_amrc_gazebo)/meshes/aruco/arucoGrid_irb1200.dae" scale="1 1 1" />
+        </geometry>
+      </visual>
+      <collision>
+        <origin xyz="0.0 0.0 0.0" rpy="0 0 0" />
+        <geometry>
+          <mesh filename="file://$(find r3mcell_amrc_gazebo)/meshes/aruco/arucoGrid_irb1200.dae" scale="1 1 1" />
+        </geometry>
+      </collision>
+      <inertial>
+        <mass value="10.0"/>
+        <inertia ixx="0.0002" ixy="0.0002" ixz="0.0002" iyy="0.0" iyz="0.0" izz="0.0" />
+      </inertial>
+    </link>
+    <joint name="floor-aruco_grid-fixed" type="fixed">
+      <parent link="floor"/>
+      <child link="aruco_grid"/>
+      <origin xyz="0.0 0.0 0.0" rpy="0.0 0.0 0.0" />
+    </joint>
+    <gazebo reference="floor-aruco_grid-fixed">
+      <preserveFixedJoint>true</preserveFixedJoint>
+    </gazebo>
+  </xacro:unless>
   <!-- ros2srrc_HMI CAMERA -->
   <xacro:if value="${hmi}">
@@ -207,3 +237,62 @@
     />
   </xacro:if>
+  <!-- CAMERA -->
+  <xacro:unless value="${bringup}">
+    <link name="camera_link">
+      <collision>
+        <origin xyz="0 0 0" rpy="0 0 0"/>
+        <geometry>
+          <box size="0.05 0.05 0.05"/>
+        </geometry>
+      </collision>
+      <visual>
+        <origin xyz="0 0 0" rpy="0 0 0"/>
+        <geometry>
+          <box size="0.05 0.05 0.05"/>
+        </geometry>
+      </visual>
+      <inertial>
+        <mass value="1.0" />
+        <origin xyz="0 0 0" rpy="0 0 0"/>
+        <inertia ixx="0.0" ixy="0.0" ixz="0.0" iyy="0.0" iyz="0.0" izz="0.0" />
+      </inertial>
+    </link>
+    <joint name="camera_joint" type="fixed">
+      <origin xyz="1.60 0.10 1.20" rpy="0 0.95 3.1416"/>
+      <parent link="world"/>
+      <child link="camera_link"/>
+    </joint>
+    <gazebo reference="camera_link">
+      <sensor name="camera" type="camera">
+        <update_rate>30</update_rate>
+        <camera name="head">
+          <horizontal_fov>1.22</horizontal_fov>
+          <image>
+            <width>1920</width>
+            <height>1080</height>
+            <format>R8G8B8</format>
+          </image>
+          <clip>
+            <near>0.02</near>
+            <far>300</far>
+          </clip>
+          <noise>
+            <type>gaussian</type>
+            <mean>0.0</mean>
+            <stddev>0.007</stddev>
+          </noise>
+        </camera>
+        <plugin filename="libgazebo_ros_camera.so" name="camera_controller">
+          <robotNamespace/>
+          <alwaysOn>true</alwaysOn>
+          <updateRate>0.0</updateRate>
+          <cameraName>camera</cameraName>
+          <imageTopicName>image_raw</imageTopicName>
+          <cameraInfoTopicName>camera_info</cameraInfoTopicName>
+          <frameName>camera</frameName>
+          <hackBaseline>0.07</hackBaseline>
+        </plugin>
+      </sensor>
+    </gazebo>
+  </xacro:unless>
 </robot>

File: AMRC/r3mcell_amrc_gazebo/urdf/r3mcell_amrc_CyS_1200.urdf.xacro (robot description, xacro)
@@ -195,4 +195,34 @@
     <origin xyz="0.0 0.0 0.0" rpy="0.0 0.0 0.0" />
   </joint>
+  <!-- ARUCO TAG -->
+  <xacro:unless value="${bringup}">
+    <!-- ARUCO GRID -->
+    <link name="aruco_grid">
+      <visual>
+        <origin xyz="0.0 0.0 0.0" rpy="0 0 0" />
+        <geometry>
+          <mesh filename="file://$(find r3mcell_amrc_gazebo)/meshes/aruco/arucoGrid_irb1200.dae" scale="1 1 1" />
+        </geometry>
+      </visual>
+      <collision>
+        <origin xyz="0.0 0.0 0.0" rpy="0 0 0" />
+        <geometry>
+          <mesh filename="file://$(find r3mcell_amrc_gazebo)/meshes/aruco/arucoGrid_irb1200.dae" scale="1 1 1" />
+        </geometry>
+      </collision>
+      <inertial>
+        <mass value="10.0"/>
+        <inertia ixx="0.0002" ixy="0.0002" ixz="0.0002" iyy="0.0" iyz="0.0" izz="0.0" />
+      </inertial>
+    </link>
+    <joint name="floor-aruco_grid-fixed" type="fixed">
+      <parent link="floor"/>
+      <child link="aruco_grid"/>
+      <origin xyz="0.0 0.0 0.0" rpy="0.0 0.0 0.0" />
+    </joint>
+    <gazebo reference="floor-aruco_grid-fixed">
+      <preserveFixedJoint>true</preserveFixedJoint>
+    </gazebo>
+  </xacro:unless>
   <!-- ros2srrc_HMI CAMERA -->
   <xacro:if value="${hmi}">
@@ -207,3 +237,62 @@
     />
   </xacro:if>
+  <!-- CAMERA -->
+  <xacro:unless value="${bringup}">
+    <link name="camera_link">
+      <collision>
+        <origin xyz="0 0 0" rpy="0 0 0"/>
+        <geometry>
+          <box size="0.05 0.05 0.05"/>
+        </geometry>
+      </collision>
+      <visual>
+        <origin xyz="0 0 0" rpy="0 0 0"/>
+        <geometry>
+          <box size="0.05 0.05 0.05"/>
+        </geometry>
+      </visual>
+      <inertial>
+        <mass value="1.0" />
+        <origin xyz="0 0 0" rpy="0 0 0"/>
+        <inertia ixx="0.0" ixy="0.0" ixz="0.0" iyy="0.0" iyz="0.0" izz="0.0" />
+      </inertial>
+    </link>
+    <joint name="camera_joint" type="fixed">
+      <origin xyz="1.60 0.10 1.20" rpy="0 0.95 3.1416"/>
+      <parent link="world"/>
+      <child link="camera_link"/>
+    </joint>
+    <gazebo reference="camera_link">
+      <sensor name="camera" type="camera">
+        <update_rate>30</update_rate>
+        <camera name="head">
+          <horizontal_fov>1.22</horizontal_fov>
+          <image>
+            <width>1920</width>
+            <height>1080</height>
+            <format>R8G8B8</format>
+          </image>
+          <clip>
+            <near>0.02</near>
+            <far>300</far>
+          </clip>
+          <noise>
+            <type>gaussian</type>
+            <mean>0.0</mean>
+            <stddev>0.007</stddev>
+          </noise>
+        </camera>
+        <plugin filename="libgazebo_ros_camera.so" name="camera_controller">
+          <robotNamespace/>
+          <alwaysOn>true</alwaysOn>
+          <updateRate>0.0</updateRate>
+          <cameraName>camera</cameraName>
+          <imageTopicName>image_raw</imageTopicName>
+          <cameraInfoTopicName>camera_info</cameraInfoTopicName>
+          <frameName>camera</frameName>
+          <hackBaseline>0.07</hackBaseline>
+        </plugin>
+      </sensor>
+    </gazebo>
+  </xacro:unless>
 </robot>

Commit message: R3M-Cell update for R3M Demo day.

File: AMRC/r3mcell_amrc_gazebo/urdf/r3mcell_amrc_CK_1200.urdf.xacro (robot description, xacro)
@@ -168,5 +168,5 @@
     <parent link="adapter_plate"/>
     <child link="base_link"/>
-    <origin xyz="0.0 0.0 0.139" rpy="0.0 0.0 0.0" />
+    <origin xyz="0.0 0.0 0.15" rpy="0.0 0.0 0.0" />
   </joint>
   <!-- ReconCell: WALLS -->

File: AMRC/r3mcell_amrc_gazebo/urdf/r3mcell_amrc_CyS_1200.urdf.xacro (robot description, xacro)
@@ -168,5 +168,5 @@
     <parent link="adapter_plate"/>
     <child link="base_link"/>
-    <origin xyz="0.0 0.0 0.139" rpy="0.0 0.0 0.0" />
+    <origin xyz="0.0 0.0 0.16" rpy="0.0 0.0 0.0" />
   </joint>
   <!-- ReconCell: WALLS -->
