Commit message: R3M use-cases update (20-12-2024).

File: AMRC/r3mcell_amrc_gazebo/urdf/objects/BaseCylinder.urdf (robot description, URDF)
Before this commit: robot LamSheet, 1 links, 0 joints
Links:
- removed link LamSheet
- added link BaseCylinder, mass 0.1; collision mesh filename=file://$(find r3mcell_amrc_gazebo)/meshes/CylinderStacking/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; visual mesh filename=file://$(find r3mcell_amrc_gazebo)/meshes/CylinderStacking/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

File: AMRC/r3mcell_amrc_gazebo/urdf/objects/Battery.urdf (robot description, URDF)
Before this commit: robot LamSheet, 1 links, 0 joints
Links:
- removed link LamSheet
- added link Battery, mass 0.1; collision mesh filename=file://$(find r3mcell_amrc_gazebo)/meshes/BatteryDisassembl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; visual mesh filename=file://$(find r3mcell_amrc_gazebo)/meshes/BatteryDisassembl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

File: AMRC/r3mcell_amrc_gazebo/urdf/objects/BlueCube.urdf (robot description, URDF)
Before this commit: robot LamSheet, 1 links, 0 joints
Links:
- removed link LamSheet
- added link BlueCube, mass 0.1; collision mesh filename=file://$(find r3mcell_amrc_gazebo)/meshes/CubeKitting/BlueC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; visual mesh filename=file://$(find r3mcell_amrc_gazebo)/meshes/CubeKitting/BlueC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

File: AMRC/r3mcell_amrc_gazebo/urdf/objects/BottomCube.urdf (robot description, URDF)
Before this commit: robot LamSheet, 1 links, 0 joints
Links:
- removed link LamSheet
- added link BottomCube, mass 0.1; collision mesh filename=file://$(find r3mcell_amrc_gazebo)/meshes/CubeStacking/Bott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; visual mesh filename=file://$(find r3mcell_amrc_gazebo)/meshes/CubeStacking/Bott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

File: AMRC/r3mcell_amrc_gazebo/urdf/objects/EmptyAssembly.urdf (robot description, URDF)
Before this commit: robot LamSheet, 1 links, 0 joints
Links:
- removed link LamSheet
- added link EmptyAssembly, mass 1.0; collision mesh filename=file://$(find r3mcell_amrc_gazebo)/meshes/CylinderStacking/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; visual mesh filename=file://$(find r3mcell_amrc_gazebo)/meshes/CylinderStacking/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

File: AMRC/r3mcell_amrc_gazebo/urdf/objects/FullAssembly.urdf (robot description, URDF)
Before this commit: robot LamSheet, 1 links, 0 joints
Links:
- removed link LamSheet
- added link FullAssembly, mass 1.0; collision mesh filename=file://$(find r3mcell_amrc_gazebo)/meshes/CylinderStacking/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; visual mesh filename=file://$(find r3mcell_amrc_gazebo)/meshes/CylinderStacking/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

File: AMRC/r3mcell_amrc_gazebo/urdf/objects/GreenCube.urdf (robot description, URDF)
Before this commit: robot LamSheet, 1 links, 0 joints
Links:
- removed link LamSheet
- added link GreenCube, mass 0.1; collision mesh filename=file://$(find r3mcell_amrc_gazebo)/meshes/CubeKitting/Green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; visual mesh filename=file://$(find r3mcell_amrc_gazebo)/meshes/CubeKitting/Green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

File: AMRC/r3mcell_amrc_gazebo/urdf/objects/MidAssembly.urdf (robot description, URDF)
Before this commit: robot LamSheet, 1 links, 0 joints
Links:
- removed link LamSheet
- added link MidAssembly, mass 1.0; collision mesh filename=file://$(find r3mcell_amrc_gazebo)/meshes/CylinderStacking/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; visual mesh filename=file://$(find r3mcell_amrc_gazebo)/meshes/CylinderStacking/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

File: AMRC/r3mcell_amrc_gazebo/urdf/objects/RedCube.urdf (robot description, URDF)
Before this commit: robot LamSheet, 1 links, 0 joints
Links:
- removed link LamSheet
- added link RedCube, mass 0.1; collision mesh filename=file://$(find r3mcell_amrc_gazebo)/meshes/CubeKitting/RedCu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; visual mesh filename=file://$(find r3mcell_amrc_gazebo)/meshes/CubeKitting/RedCu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

File: AMRC/r3mcell_amrc_gazebo/urdf/objects/TopCube.urdf (robot description, URDF)
Before this commit: robot LamSheet, 1 links, 0 joints
Links:
- removed link LamSheet
- added link TopCube, mass 0.1; collision mesh filename=file://$(find r3mcell_amrc_gazebo)/meshes/CubeStacking/TopC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; visual mesh filename=file://$(find r3mcell_amrc_gazebo)/meshes/CubeStacking/TopC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

File: AMRC/r3mcell_amrc_gazebo/urdf/objects/TopCylinder.urdf (robot description, URDF)
Before this commit: robot LamSheet, 1 links, 0 joints
Links:
- removed link LamSheet
- added link TopCylinder, mass 0.1; collision mesh filename=file://$(find r3mcell_amrc_gazebo)/meshes/CylinderStacking/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; visual mesh filename=file://$(find r3mcell_amrc_gazebo)/meshes/CylinderStacking/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

File: AMRC/r3mcell_amrc_gazebo/urdf/objects/WhiteCube.urdf (robot description, URDF)
Before this commit: robot LamSheet, 1 links, 0 joints
Links:
- removed link LamSheet
- added link WhiteCube, mass 0.1; collision mesh filename=file://$(find r3mcell_amrc_gazebo)/meshes/CubeKitting/White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; visual mesh filename=file://$(find r3mcell_amrc_gazebo)/meshes/CubeKitting/White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

File: CranfieldUniversity/r3mcell_cu_gazebo/urdf/objects/SideCase_L.urdf (robot description, URDF)
Before this commit: robot LamSheet, 1 links, 0 joints
Links:
- removed link LamSheet
- added link SideCase_L, mass 0.1; collision mesh filename=file://$(find r3mcell_cu_gazebo)/meshes/BatteryDisassembly/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; visual mesh filename=file://$(find r3mcell_cu_gazebo)/meshes/BatteryDisassembly/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

File: CranfieldUniversity/r3mcell_cu_gazebo/urdf/objects/SideCase_R.urdf (robot description, URDF)
Before this commit: robot LamSheet, 1 links, 0 joints
Links:
- removed link LamSheet
- added link SideCase_R, mass 0.1; collision mesh filename=file://$(find r3mcell_cu_gazebo)/meshes/BatteryDisassembly/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; visual mesh filename=file://$(find r3mcell_cu_gazebo)/meshes/BatteryDisassembly/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

File: CranfieldUniversity/r3mcell_cu_gazebo/urdf/objects/TopCase.urdf (robot description, URDF)
Before this commit: robot LamSheet, 1 links, 0 joints
Links:
- removed link LamSheet
- added link TopCase, mass 0.1; collision mesh filename=file://$(find r3mcell_cu_gazebo)/meshes/BatteryDisassembly/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; visual mesh filename=file://$(find r3mcell_cu_gazebo)/meshes/BatteryDisassembly/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

File: CranfieldUniversity/r3mcell_cu_gazebo/urdf/r3mcell_cu_BD.urdf.xacro (robot description, xacro)
@@ -104,5 +104,5 @@
       <origin xyz="0.0 0.0 0.0" rpy="0 0 0" />
       <geometry>
-        <mesh filename="file://$(find r3mcell_cu_gazebo)/meshes/BatteryDisassembly/BD_TopBottom.dae" scale="1 1 1" />
+        <mesh filename="file://$(find r3mcell_cu_gazebo)/meshes/BatteryDisassembly/BD_Bottom.dae" scale="1 1 1" />
       </geometry>
     </visual>
@@ -110,5 +110,5 @@
       <origin xyz="0.0 0.0 0.0" rpy="0 0 0" />
       <geometry>
-        <mesh filename="file://$(find r3mcell_cu_gazebo)/meshes/BatteryDisassembly/BD_TopBottom.dae" scale="1 1 1" />
+        <mesh filename="file://$(find r3mcell_cu_gazebo)/meshes/BatteryDisassembly/BD_Bottom.dae" scale="1 1 1" />
       </geometry>
     </collision>
@@ -121,4 +121,28 @@
     <parent link="cell"/>
     <child link="BD_Fixture"/>
+    <origin xyz="0.0 0.0 0.0" rpy="0.0 0.0 0.0" />
+  </joint>
+  <!-- R3M Cranfield Uni Cell: BD -> ERGOBOX -->
+  <link name="ergobox">
+    <visual>
+      <origin xyz="0.0 0.0 0.0" rpy="0 0 0" />
+      <geometry>
+        <mesh filename="file://$(find r3mcell_cu_gazebo)/meshes/BatteryDisassembly/ergobox.dae" scale="1 1 1" />
+      </geometry>
+    </visual>
+    <collision>
+      <origin xyz="0.0 0.0 0.0" rpy="0 0 0" />
+      <geometry>
+        <mesh filename="file://$(find r3mcell_cu_gazebo)/meshes/BatteryDisassembly/ergobox.dae" scale="1 1 1" />
+      </geometry>
+    </collision>
+    <inertial>
+      <mass value="10.0"/>
+      <inertia ixx="0.0002" ixy="0.0002" ixz="0.0002" iyy="0.0" iyz="0.0" izz="0.0" />
+    </inertial>
+  </link>
+  <joint name="cell-ergobox-fixed" type="fixed">
+    <parent link="cell"/>
+    <child link="ergobox"/>
     <origin xyz="0.0 0.0 0.0" rpy="0.0 0.0 0.0" />
   </joint>

File: CranfieldUniversity/r3mcell_cu_gazebo/urdf/r3mcell_cu_CSur.urdf.xacro (robot description, xacro)
@@ -140,5 +140,5 @@
         <origin xyz="0.0 0.0 0.0" rpy="0 0 0" />
         <geometry>
-          <mesh filename="file://$(find r3mcell_cu_gazebo)/meshes/CylinderStacking/aruco100_UR.dae" scale="1 1 1" />
+          <mesh filename="file://$(find r3mcell_cu_gazebo)/meshes/aruco/aruco100_UR.dae" scale="1 1 1" />
         </geometry>
       </visual>
@@ -146,5 +146,5 @@
         <origin xyz="0.0 0.0 0.0" rpy="0 0 0" />
         <geometry>
-          <mesh filename="file://$(find r3mcell_cu_gazebo)/meshes/CylinderStacking/aruco100_UR.dae" scale="1 1 1" />
+          <mesh filename="file://$(find r3mcell_cu_gazebo)/meshes/aruco/aruco100_UR.dae" scale="1 1 1" />
         </geometry>
       </collision>
@@ -168,5 +168,5 @@
         <origin xyz="0.0 0.0 0.0" rpy="0 0 0" />
         <geometry>
-          <mesh filename="file://$(find r3mcell_cu_gazebo)/meshes/CylinderStacking/arucoGrid_UR.dae" scale="1 1 1" />
+          <mesh filename="file://$(find r3mcell_cu_gazebo)/meshes/aruco/arucoGrid_UR.dae" scale="1 1 1" />
         </geometry>
       </visual>
@@ -174,5 +174,5 @@
         <origin xyz="0.0 0.0 0.0" rpy="0 0 0" />
         <geometry>
-          <mesh filename="file://$(find r3mcell_cu_gazebo)/meshes/CylinderStacking/arucoGrid_UR.dae" scale="1 1 1" />
+          <mesh filename="file://$(find r3mcell_cu_gazebo)/meshes/aruco/arucoGrid_UR.dae" scale="1 1 1" />
         </geometry>
       </collision>

File: CranfieldUniversity/r3mcell_cu_gazebo/urdf/r3mcell_cu_cylinderstacking.urdf.xacro (robot description, xacro)
@@ -130,5 +130,5 @@
         <origin xyz="0.0 0.0 0.0" rpy="0 0 0" />
         <geometry>
-          <mesh filename="file://$(find r3mcell_cu_gazebo)/meshes/CylinderStacking/aruco100.dae" scale="1 1 1" />
+          <mesh filename="file://$(find r3mcell_cu_gazebo)/meshes/aruco/aruco100.dae" scale="1 1 1" />
         </geometry>
       </visual>
@@ -136,5 +136,5 @@
         <origin xyz="0.0 0.0 0.0" rpy="0 0 0" />
         <geometry>
-          <mesh filename="file://$(find r3mcell_cu_gazebo)/meshes/CylinderStacking/aruco100.dae" scale="1 1 1" />
+          <mesh filename="file://$(find r3mcell_cu_gazebo)/meshes/aruco/aruco100.dae" scale="1 1 1" />
         </geometry>
       </collision>
@@ -158,5 +158,5 @@
         <origin xyz="0.0 0.0 0.0" rpy="0 0 0" />
         <geometry>
-          <mesh filename="file://$(find r3mcell_cu_gazebo)/meshes/CylinderStacking/arucoGrid.dae" scale="1 1 1" />
+          <mesh filename="file://$(find r3mcell_cu_gazebo)/meshes/aruco/arucoGrid.dae" scale="1 1 1" />
         </geometry>
       </visual>
@@ -164,5 +164,5 @@
         <origin xyz="0.0 0.0 0.0" rpy="0 0 0" />
         <geometry>
-          <mesh filename="file://$(find r3mcell_cu_gazebo)/meshes/CylinderStacking/arucoGrid.dae" scale="1 1 1" />
+          <mesh filename="file://$(find r3mcell_cu_gazebo)/meshes/aruco/arucoGrid.dae" scale="1 1 1" />
         </geometry>
       </collision>
