Commit message: Fix: BD fixture height + Battery urdf.

File: AMRC/r3mcell_amrc_gazebo/urdf/objects/Battery.urdf (robot description, URDF)
Before this commit: robot Battery, 1 links, 0 joints
Links:
- removed link Battery
- added link ${name}, mass 0.1; collision mesh filename=file://$(find r3mcell_amrc_gazebo)/meshes/BatteryDisassembl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; visual mesh filename=file://$(find r3mcell_amrc_gazebo)/meshes/BatteryDisassembl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

File: AMRC/r3mcell_amrc_gazebo/urdf/r3mcell_amrc_BD.urdf.xacro (robot description, xacro)
@@ -173,5 +173,5 @@
     <parent link="floor"/>
     <child link="BD_fixture"/>
-    <origin xyz="0.0 0.0 0.0" rpy="0.0 0.0 0.0" />
+    <origin xyz="0.0 0.0 0.005" rpy="0.0 0.0 0.0" />
   </joint>
   <link name="BD_PlasticBin">
@@ -196,5 +196,5 @@
     <parent link="floor"/>
     <child link="BD_PlasticBin"/>
-    <origin xyz="0.0 0.0 0.0" rpy="0.0 0.0 0.0" />
+    <origin xyz="0.0 0.0 0.005" rpy="0.0 0.0 0.0" />
   </joint>
   <link name="BD_CaseBottom">
